File: radio.kicad_sch (KiCad schematic)
At the start: 0 parts

Commit message: wen branch and pr
Other:
- title: Diagram -> (none)
Changed lines of the file:
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@@
 	(paper "A4")
 	(title_block
-		(title "Diagram")
 		(date "2025-12-13")
 		(rev "1.0")
