File: mcu_power.kicad_sch (KiCad schematic)
At the start: 1 part, among them U1 STM32H743ZITx

Commit message: more passives work
Parts:
- added C1, C10, C11, C2, C3, C4, C5, C6, C7, C8, C9: 100n, 0_capacitor_smd:C_0402_1005Metric, symbol Device:C
- added C12: 4u7, 0_capacitor_smd:C_0603_1608Metric, symbol Device:C
- added C13, C14: 2u2, 0_capacitor_smd:C_0603_1608Metric, symbol Device:C
Connections:
- net at U1.106 (VCAP): now also C14.1
- net GND: now reaches U1.107 (VSS)
- net GND: now also U1.120 (VSS), U1.130 (VSS), U1.16 (VSS), U1.31 (VSSA), U1.38 (VSS), U1.51 (VSS), U1.61 (VSS), U1.83 (VSS), U1.94 (VSS), C1.2, C10.2, C11.2, C12.2, C13.2, C14.2, C2.2, C3.2, C4.2, C5.2, C6.2, C7.2, C8.2, C9.2
- net +3V3: now reaches U1.108 (VDD)
- net +3V3: now also U1.121 (VDD), U1.131 (VDD), U1.144 (VDD), U1.17 (VDD), U1.30 (VDD), U1.39 (VDD), U1.52 (VDD), U1.6 (VBAT), U1.62 (VDD), U1.72 (VDD), U1.84 (VDD), U1.95 (VDD33_USB), C1.1, C10.1, C11.1, C12.1, C2.1, C3.1, C4.1, C5.1, C6.1, C7.1, C8.1, C9.1
- net at U1.71 (VCAP): now also C13.1
Other:
- moved on the sheet: U1A

Commit message: sensors done, mcu worked on
Parts:
- added C15, C17: 100n, 0_capacitor_smd:C_0402_1005Metric, symbol Device:C
- added C16, C18, C19: 1u, 0_capacitor_smd:C_0603_1608Metric, symbol Device:C
- added L1: 600R@100MHz, symbol Device:L_Ferrite
Connections:
- net +3V3: now also U1.143 (PDR_ON), C19.1, L1.1
- net GND: now also C15.2, C16.2, C17.2, C18.2, C19.2
- net at U1.32 (VREF+): now also U1.33 (VDDA), C15.1, C16.1, C17.1, C18.1, L1.2
Other:
- title: Hoppen FC -> MCU Power
- moved on the sheet: C1, C10, C11, C12, C13, C14, C2, C3, C4, C5, C6, C7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

Commit message: rs232,can,ind,storage,usb v01
Parts:
- renumbered C12 to C1, C4 to C10, C3 to C11, C16 to C12, C18 to C13, C2 to C14, C17 to C16, C1 to C17, C13 to C18, C14 to C19, C11 to C2, C10 to C3, C9 to C4, C8 to C5, C7 to C6, C6 to C7, C19 to C8, C5 to C9
Other:
- moved on the sheet: C13, C16

Commit message: yeah
Connections:
- net +3V3: no longer C8.1, L1.1
- net MCU_VDDA: now reaches C12.1, C13.1, C15.1, C16.1, L1.2, U1.32 (VREF+), U1.33 (VDDA)
- net MCU_VCAP2: now reaches C19.1, U1.106 (VCAP)
- net MCU_VCAP1: now reaches C18.1, U1.71 (VCAP)
- new net +3V3A: C8.1, L1.1
Changed lines of the file:
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@@
 		(company "Hoppen")
+	)
+	(rectangle
+		(start 25.4 38.1)
+		(end 266.7 139.7)
+		(stroke
+			(width 0.254)
+			(type dash)
+		)
+		(fill
+			(type none)
+		)
 	)
 	(text_box "[${#}] ${TITLE}"
@@
 			(width 0)
 			(type default)
+		)
+	)
+	(label "MCU_VREF"
+		(at 133.35 115.57 0)
+		(effects
+			(font
+				(size 1.27 1.27)
+			)
+			(justify left bottom)
+		)
+	)
+	(label "MCU_VCAP1"
+		(at 220.98 58.42 0)
+		(effects
+			(font
+				(size 1.27 1.27)
+			)
+			(justify left bottom)
+		)
+	)
+	(label "MCU_VDDA"
+		(at 133.35 91.44 0)
+		(effects
+			(font
+				(size 1.27 1.27)
+			)
+			(justify left bottom)
+		)
+	)
+	(label "MCU_VCAP2"
+		(at 220.98 55.88 0)
+		(effects
+			(font
+				(size 1.27 1.27)
+			)
+			(justify left bottom)
 		)
 	)
@@
 			)
 		)
-		(property "Value" "+3V3"
-			(at 110.49 86.36 0)
-			(effects
-				(font
-					(size 1.27 1.27)
-				)
-			)
-		)
+		(property "Value" "+3V3A"
+			(at 113.03 90.1699 0)
+			(effects
+				(font
+					(size 1.27 1.27)
+				)
+				(justify left)
+			)
+		)

Commit message: wen branch and pr
Changed lines of the file:
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@@
-		)
-	)
-	(label "MCU_VREF"
-		(at 133.35 115.57 0)
-		(effects
-			(font
-				(size 1.27 1.27)
-			)
-			(justify left bottom)
 		)
 	)

Commit message: much work and .ioc file added
Connections:
- net +3V3A is gone; now on net +3V3: C8.1, L1.1
Changed lines of the file:
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@@
 			)
 		)
-		(property "Value" "+3V3A"
+		(property "Value" "+3V3"
 			(at 113.03 90.1699 0)
 			(effects
