File: canbus.kicad_sch (KiCad schematic)
At the start: 4 parts, among them U8 TJA1051TK-3

Commit message: wen branch and pr
Parts:
- added C79, C80: 100n, symbol Device:C
- added R51: 10k, symbol Device:R
- added U14: TJA1051TK-3, Package_SON:HVSON-8-1EP_3x3mm_P0.65mm_EP1.6x2.4mm, symbol 0_transceivers:TJA1051TK-3
Connections:
- net +3V3: now also C80.1, U14.5 (VIO)
- net +5V: now also C79.1, U14.3 (VCC)
- net GND: now also C79.2, C80.2, R51.2, U14.2 (GND), U14.9 (GND)
- net CAN_H renamed CAN1_H
- net CAN_L renamed CAN1_L
- net CAN_RX renamed CAN1_RX
- net CAN_TX renamed CAN1_TX
- net RS232_S renamed CAN1_S
- new net CAN2_H: U14.7 (CANH)
- new net CAN2_L: U14.6 (CANL)
- new net CAN2_RX: U14.4 (RXD)
- new net CAN2_S: R51.1, U14.8 (S)
- new net CAN2_TX: U14.1 (TXD)
Other:
- note added: "FDCAN TRANSCEIVER 1"
- note added: "FDCAN TRANSCEIVER 2"
- moved on the sheet: C43, C44, R16, U8

Commit message: much work and .ioc file added
Connections:
- net CAN1_H renamed FDCAN1_H
- net CAN1_L renamed FDCAN1_L
- net CAN1_RX renamed FDCAN1_RX
- net CAN1_TX renamed FDCAN1_TX
- net CAN2_H renamed FDCAN2_H
- net CAN2_L renamed FDCAN2_L
- net CAN2_RX renamed FDCAN2_RX
- net CAN2_TX renamed FDCAN2_TX
Other:
- note added: "FDCAN TRANSCEIVER 1 @ 5 Mbit/s"
- note added: "FDCAN TRANSCEIVER 2 @ 5 Mbit/s"
- note removed: "FDCAN TRANSCEIVER 1"
- note removed: "FDCAN TRANSCEIVER 2"

Commit message: start fix fp
Parts:
- C43, C44, C79, C80: footprint (none) -> 0_capacitor_smd:C_0402_1005Metric
- R16, R51: footprint (none) -> 0_resistor_smd:R_0402_1005Metric
- U14, U8: footprint Package_SON:HVSON-8-1EP_3x3mm_P0.65mm_EP1.6x2.4mm -> 0_transceivers:HVSON-8-1EP_3x3mm_P0.65mm_EP1.6x2.4mm
Changed lines of the file:
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@@
 			)
 		)
-		(property "Footprint" ""
+		(property "Footprint" "0_capacitor_smd:C_0402_1005Metric"
 			(at 207.9752 85.09 0)
 			(effects
@@
 			)
 		)
-		(property "Footprint" ""
+		(property "Footprint" "0_capacitor_smd:C_0402_1005Metric"
 			(at 115.2652 85.09 0)
 			(effects
@@
 			)
 		)
-		(property "Footprint" ""
+		(property "Footprint" "0_resistor_smd:R_0402_1005Metric"
 			(at 80.772 110.49 90)
 			(effects
@@
 			)
 		)
-		(property "Footprint" ""
+		(property "Footprint" "0_resistor_smd:R_0402_1005Metric"
 			(at 173.482 110.49 90)
 			(effects
@@
 			)
 		)
-		(property "Footprint" ""
+		(property "Footprint" "0_capacitor_smd:C_0402_1005Metric"
 			(at 180.0352 85.09 0)
 			(effects
@@
 			)
 		)
-		(property "Footprint" ""
+		(property "Footprint" "0_capacitor_smd:C_0402_1005Metric"
 			(at 87.3252 85.09 0)
 			(effects
@@
 			)
 		)
-		(property "Footprint" "Package_SON:HVSON-8-1EP_3x3mm_P0.65mm_EP1.6x2.4mm"
+		(property "Footprint" "0_transceivers:HVSON-8-1EP_3x3mm_P0.65mm_EP1.6x2.4mm"
 			(at 100.33 69.85 0)
 			(effects
@@
 			)
 		)
-		(property "Footprint" "Package_SON:HVSON-8-1EP_3x3mm_P0.65mm_EP1.6x2.4mm"
+		(property "Footprint" "0_transceivers:HVSON-8-1EP_3x3mm_P0.65mm_EP1.6x2.4mm"
 			(at 193.04 69.85 0)
 			(effects
