File: mcu_io.kicad_sch (KiCad schematic)
At the start: 1 part, among them U1 STM32H743ZITx

Commit message: sensors done, mcu worked on
Parts:
- added C26, C27, C28: 100n, 0_capacitor_smd:C_0402_1005Metric, symbol Device:C
- added C29, C30: 6p, 0_capacitor_smd:C_0402_1005Metric, symbol Device:C
- added C31, C32: 15p, 0_capacitor_smd:C_0402_1005Metric, symbol Device:C
- added JP1, JP2: J, 0_misc:SolderJumper-2_P1.3mm_Bridged_RoundedPad1.0x1.5mm, symbol 0_misc:SolderJumper_2_Bridged
- added R2: 1k, 0_resistor_smd:R_0402_1005Metric, symbol Device:R
- added SW1, SW2, SW3: SW_Push, symbol 0_misc:SW_Push
- added Y1: 25 MHz, symbol Device:Crystal_GND24
- added Y2: 32.768 kHz, symbol Device:Crystal
Connections:
- new net: JP1.1 (A), SW2.2
- new net: JP2.1 (A), SW3.2
- new net BOOT: C28.1, R2.2, SW3.1
- new net GND: C26.2, C27.2, C28.2, C29.1, C30.1, C31.1, C32.1, JP1.2 (B), JP2.2 (B), R2.1, SW1.2, Y1.2, Y1.4
- new net HSE_IN: C29.2, Y1.1
- new net HSE_OUT: C30.2, Y1.3
- new net LSE_IN: C31.2, Y2.1
- new net LSE_OUT: C32.2, Y2.2
- new net RST: C27.1, SW2.1
- new net USER_BUTTON: C26.1, SW1.1
Other:
- note added: "BOOT"
- note added: "HSE 25 MHz"
- note added: "LSE 32.768 kHz"
- note added: "RESET BUTTON"
- note added: "USER BUTTON"
- title: Hoppen FC -> MCU IO
- moved on the sheet: U1B, U1C

Commit message: rs232,can,ind,storage,usb v01
Parts:
- renumbered C26 to C20, C27 to C21, C28 to C22, C29 to C23, C30 to C24, C31 to C25, C32 to C26, R2 to R1
Changed lines of the file:
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@@
 	)
 	(rectangle
-		(start 182.88 251.46)
+		(start 182.88 254)
 		(end 226.06 279.4)
 		(stroke
@@
 	)
 	(rectangle
-		(start 129.54 251.46)
+		(start 129.54 254)
 		(end 177.8 279.4)
 		(stroke
@@
 	)
 	(rectangle
-		(start 231.14 251.46)
+		(start 231.14 254)
 		(end 276.86 279.4)
 		(stroke
@@
 	)
 	(rectangle
-		(start 81.28 251.46)
+		(start 81.28 254)
 		(end 124.46 279.4)
 		(stroke
@@
 	)
 	(rectangle
-		(start 33.02 251.46)
+		(start 33.02 254)
 		(end 76.2 279.4)
 		(stroke
@@
 	(text "HSE 25 MHz"
 		(exclude_from_sim no)
-		(at 194.31 248.92 0)
+		(at 194.31 251.46 0)
 		(effects
 			(font
@@
 	(text "BOOT\n"
 		(exclude_from_sim no)
-		(at 134.62 248.92 0)
+		(at 134.62 251.46 0)
 		(effects
 			(font
@@
 	(text "RESET BUTTON\n"
 		(exclude_from_sim no)
-		(at 95.25 248.92 0)
+		(at 95.25 251.46 0)
 		(effects
 			(font
@@
 	(text "LSE 32.768 kHz\n"
 		(exclude_from_sim no)
-		(at 246.38 248.92 0)
+		(at 246.38 251.46 0)
 		(effects
 			(font
@@
 	(text "USER BUTTON\n"
 		(exclude_from_sim no)
-		(at 45.72 248.92 0)
+		(at 45.72 251.46 0)
 		(effects
 			(font
@@
 	(wire
 		(pts
-			(xy 204.47 260.35) (xy 204.47 254)
+			(xy 204.47 260.35) (xy 204.47 256.54)
 		)
 		(stroke
@@
 	(wire
 		(pts
-			(xy 204.47 254) (xy 207.01 254)
+			(xy 204.47 256.54) (xy 207.01 256.54)
 		)
 		(stroke
@@
 	(wire
 		(pts
-			(xy 242.57 265.43) (xy 250.19 265.43)
+			(xy 207.01 256.54) (xy 207.01 257.81)
 		)
 		(stroke
@@
 	(wire
 		(pts
-			(xy 204.47 270.51) (xy 204.47 274.32)
+			(xy 242.57 265.43) (xy 250.19 265.43)
 		)
 		(stroke
@@
 	(wire
 		(pts
-			(xy 147.32 262.89) (xy 147.32 264.16)
+			(xy 204.47 270.51) (xy 204.47 274.32)
 		)
 		(stroke
@@
 	(wire
 		(pts
-			(xy 264.16 274.32) (xy 264.16 273.05)
+			(xy 147.32 262.89) (xy 147.32 264.16)
 		)
 		(stroke
@@
 	(wire
 		(pts
-			(xy 234.95 265.43) (xy 242.57 265.43)
+			(xy 264.16 274.32) (xy 264.16 273.05)
 		)
 		(stroke
@@
 	(wire
 		(pts
-			(xy 115.57 262.89) (xy 118.11 262.89)
+			(xy 234.95 265.43) (xy 242.57 265.43)
 		)
 		(stroke
@@
 	(wire
 		(pts
-			(xy 207.01 254) (xy 207.01 255.27)
+			(xy 115.57 262.89) (xy 118.11 262.89)
 		)
 		(stroke
@@
 		(dnp no)
 		(fields_autoplaced yes)
-		(property "Reference" "#PWR033"
+		(property "Reference" "#PWR018"
 			(at 242.57 280.67 0)
 			(effects
@@
 			(project "hoppen_fc"
 				(path "/abe950a1-9eef-4508-9fd4-31d3e723e029/c85454e5-a89e-41eb-a5ed-71b4fc4cf13a/b2889d66-ad44-4386-8a59-32f6d6b6b256"
-					(reference "#PWR033")
+					(reference "#PWR018")
 					(unit 1)
 				)
@@
 		(on_board yes)
 		(dnp no)
-		(property "Reference" "R2"
+		(property "Reference" "R1"
 			(at 140.97 267.9699 0)
 			(effects
@@
 			(project "hoppen_fc"
 				(path "/abe950a1-9eef-4508-9fd4-31d3e723e029/c85454e5-a89e-41eb-a5ed-71b4fc4cf13a/b2889d66-ad44-4386-8a59-32f6d6b6b256"
-					(reference "R2")
+					(reference "R1")
 					(unit 1)
 				)
@@
 		(dnp no)
 		(fields_autoplaced yes)
-		(property "Reference" "#PWR027"
+		(property "Reference" "#PWR012"
 			(at 138.43 280.67 0)
 			(effects
@@
 			(project "hoppen_fc"
 				(path "/abe950a1-9eef-4508-9fd4-31d3e723e029/c85454e5-a89e-41eb-a5ed-71b4fc4cf13a/b2889d66-ad44-4386-8a59-32f6d6b6b256"
-					(reference "#PWR027")
+					(reference "#PWR012")
 					(unit 1)
 				)
@@
 		(dnp no)
 		(fields_autoplaced yes)
-		(property "Reference" "C30"
+		(property "Reference" "C24"
 			(at 218.44 267.9699 0)
 			(effects
@@
 			(project "hoppen_fc"
 				(path "/abe950a1-9eef-4508-9fd4-31d3e723e029/c85454e5-a89e-41eb-a5ed-71b4fc4cf13a/b2889d66-ad44-4386-8a59-32f6d6b6b256"
-					(reference "C30")
+					(reference "C24")
 					(unit 1)
 				)
@@
 		(dnp no)
 		(fields_autoplaced yes)
-		(property "Reference" "#PWR034"
+		(property "Reference" "#PWR019"
 			(at 264.16 280.67 0)
 			(effects
@@
 			(project "hoppen_fc"
 				(path "/abe950a1-9eef-4508-9fd4-31d3e723e029/c85454e5-a89e-41eb-a5ed-71b4fc4cf13a/b2889d66-ad44-4386-8a59-32f6d6b6b256"
-					(reference "#PWR034")
+					(reference "#PWR019")
 					(unit 1)
 				)
@@
 		(dnp no)
 		(fields_autoplaced yes)
-		(property "Reference" "C32"
+		(property "Reference" "C26"
 			(at 267.97 267.9699 0)
 			(effects
@@
 			(project "hoppen_fc"
 				(path "/abe950a1-9eef-4508-9fd4-31d3e723e029/c85454e5-a89e-41eb-a5ed-71b4fc4cf13a/b2889d66-ad44-4386-8a59-32f6d6b6b256"
-					(reference "C32")
+					(reference "C26")
 					(unit 1)
 				)
@@
 		(dnp no)
 		(fields_autoplaced yes)
-		(property "Reference" "C29"
+		(property "Reference" "C23"
 			(at 196.85 267.9699 0)
 			(effects
@@
 			(project ""
 				(path "/abe950a1-9eef-4508-9fd4-31d3e723e029/c85454e5-a89e-41eb-a5ed-71b4fc4cf13a/b2889d66-ad44-4386-8a59-32f6d6b6b256"
-					(reference "C29")
+					(reference "C23")
 					(unit 1)
 				)
@@
 		(dnp no)
 		(fields_autoplaced yes)
-		(property "Reference" "C26"
+		(property "Reference" "C20"
 			(at 57.15 266.6999 0)
 			(effects
@@
 			(project "hoppen_fc"
 				(path "/abe950a1-9eef-4508-9fd4-31d3e723e029/c85454e5-a89e-41eb-a5ed-71b4fc4cf13a/b2889d66-ad44-4386-8a59-32f6d6b6b256"
-					(reference "C26")
+					(reference "C20")
 					(unit 1)
 				)
@@
 		(dnp no)
 		(fields_autoplaced yes)
-		(property "Reference" "C31"
+		(property "Reference" "C25"
 			(at 246.38 267.9699 0)
 			(effects
@@
 			(project "hoppen_fc"
 				(path "/abe950a1-9eef-4508-9fd4-31d3e723e029/c85454e5-a89e-41eb-a5ed-71b4fc4cf13a/b2889d66-ad44-4386-8a59-32f6d6b6b256"
-					(reference "C31")
+					(reference "C25")
 					(unit 1)
 				)
@@
 		(dnp no)
 		(fields_autoplaced yes)
-		(property "Reference" "#PWR028"
+		(property "Reference" "#PWR013"
 			(at 172.72 280.67 0)
 			(effects
@@
 			(project "hoppen_fc"
 				(path "/abe950a1-9eef-4508-9fd4-31d3e723e029/c85454e5-a89e-41eb-a5ed-71b4fc4cf13a/b2889d66-ad44-4386-8a59-32f6d6b6b256"
-					(reference "#PWR028")
+					(reference "#PWR013")
 					(unit 1)
 				)
@@
 		(dnp no)
 		(fields_autoplaced yes)
-		(property "Reference" "#PWR025"
+		(property "Reference" "#PWR011"
 			(at 118.11 280.67 0)
 			(effects
@@
 			(project "hoppen_fc"
 				(path "/abe950a1-9eef-4508-9fd4-31d3e723e029/c85454e5-a89e-41eb-a5ed-71b4fc4cf13a/b2889d66-ad44-4386-8a59-32f6d6b6b256"
-					(reference "#PWR025")
+					(reference "#PWR011")
 					(unit 1)
 				)
@@
 		(dnp no)
 		(fields_autoplaced yes)
-		(property "Reference" "C27"
+		(property "Reference" "C21"
 			(at 96.52 266.6999 0)
 			(effects
@@
 			(project "hoppen_fc"
 				(path "/abe950a1-9eef-4508-9fd4-31d3e723e029/c85454e5-a89e-41eb-a5ed-71b4fc4cf13a/b2889d66-ad44-4386-8a59-32f6d6b6b256"
-					(reference "C27")
+					(reference "C21")
 					(unit 1)
 				)
@@
 		(dnp no)
 		(fields_autoplaced yes)
-		(property "Reference" "#PWR029"
+		(property "Reference" "#PWR015"
 			(at 204.47 280.67 0)
 			(effects
@@
 			(project "hoppen_fc"
 				(path "/abe950a1-9eef-4508-9fd4-31d3e723e029/c85454e5-a89e-41eb-a5ed-71b4fc4cf13a/b2889d66-ad44-4386-8a59-32f6d6b6b256"
-					(reference "#PWR029")
+					(reference "#PWR015")
 					(unit 1)
 				)
@@
 		(dnp no)
 		(fields_autoplaced yes)
-		(property "Reference" "#PWR024"
+		(property "Reference" "#PWR010"
 			(at 68.58 280.67 0)
 			(effects
@@
 			(project "hoppen_fc"
 				(path "/abe950a1-9eef-4508-9fd4-31d3e723e029/c85454e5-a89e-41eb-a5ed-71b4fc4cf13a/b2889d66-ad44-4386-8a59-32f6d6b6b256"
-					(reference "#PWR024")
+					(reference "#PWR010")
 					(unit 1)
 				)
@@
 		(dnp no)
 		(fields_autoplaced yes)
-		(property "Reference" "C28"
+		(property "Reference" "C22"
 			(at 151.13 266.6999 0)
 			(effects
@@
 			(project "hoppen_fc"
 				(path "/abe950a1-9eef-4508-9fd4-31d3e723e029/c85454e5-a89e-41eb-a5ed-71b4fc4cf13a/b2889d66-ad44-4386-8a59-32f6d6b6b256"
-					(reference "C28")
+					(reference "C22")
 					(unit 1)
 				)
@@
 		(dnp no)
 		(fields_autoplaced yes)
-		(property "Reference" "#PWR032"
+		(property "Reference" "#PWR017"
 			(at 214.63 280.67 0)
 			(effects
@@
 			(project "hoppen_fc"
 				(path "/abe950a1-9eef-4508-9fd4-31d3e723e029/c85454e5-a89e-41eb-a5ed-71b4fc4cf13a/b2889d66-ad44-4386-8a59-32f6d6b6b256"
-					(reference "#PWR032")
+					(reference "#PWR017")
 					(unit 1)
 				)
@@
 	(symbol
 		(lib_id "power:GND")
-		(at 207.01 255.27 0)
+		(at 207.01 257.81 0)
 		(unit 1)
 		(exclude_from_sim no)
@@
 		(dnp no)
 		(fields_autoplaced yes)
-		(property "Reference" "#PWR030"
-			(at 207.01 261.62 0)
+		(property "Reference" "#PWR016"
+			(at 207.01 264.16 0)
 			(effects
 				(font
@@
 		)
 		(property "Value" "GND"
-			(at 207.01 260.35 0)
+			(at 207.01 262.89 0)
 			(effects
 				(font
@@
 		)
 		(property "Footprint" ""
-			(at 207.01 255.27 0)
+			(at 207.01 257.81 0)
 			(effects
 				(font
@@
 		)
 		(property "Datasheet" ""
-			(at 207.01 255.27 0)
+			(at 207.01 257.81 0)
 			(effects
 				(font
@@
 		)
 		(property "Description" "Power symbol creates a global label with name \"GND\" , ground"
-			(at 207.01 255.27 0)
+			(at 207.01 257.81 0)
 			(effects
 				(font
@@
 			(project "hoppen_fc"
 				(path "/abe950a1-9eef-4508-9fd4-31d3e723e029/c85454e5-a89e-41eb-a5ed-71b4fc4cf13a/b2889d66-ad44-4386-8a59-32f6d6b6b256"
-					(reference "#PWR030")
+					(reference "#PWR016")
 					(unit 1)
 				)
@@
 		(dnp no)
 		(fields_autoplaced yes)
-		(property "Reference" "#PWR031"
+		(property "Reference" "#PWR014"
 			(at 193.04 280.67 0)
 			(effects
@@
 			(project "hoppen_fc"
 				(path "/abe950a1-9eef-4508-9fd4-31d3e723e029/c85454e5-a89e-41eb-a5ed-71b4fc4cf13a/b2889d66-ad44-4386-8a59-32f6d6b6b256"
-					(reference "#PWR031")
+					(reference "#PWR014")
 					(unit 1)
 				)

Commit message: wen branch and pr
Connections:
- net RST_POST_SW: now reaches JP1.1 (A), SW2.2
- net BOOT_POST_SW: now reaches JP2.1 (A), SW3.2
Other:
- moved on the sheet: JP1, JP2, SW2, SW3
Changed lines of the file:
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@@
 	(wire
 		(pts
-			(xy 170.18 262.89) (xy 172.72 262.89)
+			(xy 171.45 262.89) (xy 172.72 262.89)
 		)
 		(stroke
@@
 	(wire
 		(pts
-			(xy 147.32 262.89) (xy 149.86 262.89)
+			(xy 147.32 262.89) (xy 148.59 262.89)
 		)
 		(stroke
@@
 	(wire
 		(pts
-			(xy 92.71 262.89) (xy 95.25 262.89)
+			(xy 92.71 262.89) (xy 93.98 262.89)
 		)
 		(stroke
@@
 	(wire
 		(pts
-			(xy 115.57 262.89) (xy 118.11 262.89)
+			(xy 116.84 262.89) (xy 118.11 262.89)
 		)
 		(stroke
@@
 	(wire
 		(pts
+			(xy 158.75 262.89) (xy 163.83 262.89)
+		)
+		(stroke
+			(width 0)
+			(type default)
+		)
+	)
+	(wire
+		(pts
 			(xy 118.11 262.89) (xy 118.11 273.05)
 		)
@@
 	(wire
 		(pts
-			(xy 105.41 262.89) (xy 107.95 262.89)
+			(xy 104.14 262.89) (xy 109.22 262.89)
 		)
 		(stroke
@@
 		(pts
 			(xy 85.09 262.89) (xy 92.71 262.89)
-		)
-		(stroke
-			(width 0)
-			(type default)
-		)
-	)
-	(wire
-		(pts
-			(xy 160.02 262.89) (xy 162.56 262.89)
 		)
 		(stroke
@@
 		)
 	)
+	(label "BOOT_POST_SW"
+		(at 158.75 262.89 0)
+		(effects
+			(font
+				(size 0.508 0.508)
+			)
+			(justify left bottom)
+		)
+	)
 	(label "RST"
 		(at 85.09 262.89 0)
@@
 			(font
 				(size 1.27 1.27)
+			)
+			(justify left bottom)
+		)
+	)
+	(label "RST_POST_SW"
+		(at 104.14 262.89 0)
+		(effects
+			(font
+				(size 0.508 0.508)
 			)
 			(justify left bottom)
@@
 	(symbol
 		(lib_id "0_misc:SW_Push")
-		(at 100.33 262.89 0)
+		(at 99.06 262.89 0)
 		(unit 1)
 		(exclude_from_sim no)
@@
 		(dnp no)
 		(property "Reference" "SW2"
-			(at 100.33 257.81 0)
+			(at 99.06 257.81 0)
 			(effects
 				(font
@@
 		)
 		(property "Value" "SW_Push"
-			(at 100.33 257.81 0)
+			(at 99.06 257.81 0)
 			(effects
 				(font
@@
 		)
 		(property "Footprint" ""
-			(at 100.33 257.81 0)
+			(at 99.06 257.81 0)
 			(effects
 				(font
@@
 		)
 		(property "Datasheet" "~"
-			(at 100.33 257.81 0)
+			(at 99.06 257.81 0)
 			(effects
 				(font
@@
 		)
 		(property "Description" "Push button switch, generic, two pins"
-			(at 100.33 262.89 0)
+			(at 99.06 262.89 0)
 			(effects
 				(font
@@
 	(symbol
 		(lib_id "0_misc:SolderJumper_2_Bridged")
-		(at 166.37 262.89 0)
+		(at 167.64 262.89 0)
 		(unit 1)
 		(exclude_from_sim no)
@@
 		(fields_autoplaced yes)
 		(property "Reference" "JP2"
-			(at 166.37 259.08 0)
+			(at 167.64 259.08 0)
 			(effects
 				(font
@@
 		)
 		(property "Value" "J"
-			(at 166.37 265.43 0)
+			(at 167.64 265.43 0)
 			(effects
 				(font
@@
 		)
 		(property "Footprint" "0_misc:SolderJumper-2_P1.3mm_Bridged_RoundedPad1.0x1.5mm"
-			(at 166.37 262.89 0)
+			(at 167.64 262.89 0)
 			(effects
 				(font
@@
 		)
 		(property "Datasheet" "~"
-			(at 166.37 262.89 0)
+			(at 167.64 262.89 0)
 			(effects
 				(font
@@
 		)
 		(property "Description" "Solder Jumper, 2-pole, closed/bridged"
-			(at 166.37 262.89 0)
+			(at 167.64 262.89 0)
 			(effects
 				(font
@@
 	(symbol
 		(lib_id "0_misc:SW_Push")
-		(at 154.94 262.89 0)
+		(at 153.67 262.89 0)
 		(unit 1)
 		(exclude_from_sim no)
@@
 		(dnp no)
 		(property "Reference" "SW3"
-			(at 154.94 257.81 0)
+			(at 153.67 257.81 0)
 			(effects
 				(font
@@
 		)
 		(property "Value" "SW_Push"
-			(at 154.94 257.81 0)
+			(at 153.67 257.81 0)
 			(effects
 				(font
@@
 		)
 		(property "Footprint" ""
-			(at 154.94 257.81 0)
+			(at 153.67 257.81 0)
 			(effects
 				(font
@@
 		)
 		(property "Datasheet" "~"
-			(at 154.94 257.81 0)
+			(at 153.67 257.81 0)
 			(effects
 				(font
@@
 		)
 		(property "Description" "Push button switch, generic, two pins"
-			(at 154.94 262.89 0)
+			(at 153.67 262.89 0)
 			(effects
 				(font
@@
 	(symbol
 		(lib_id "0_misc:SolderJumper_2_Bridged")
-		(at 111.76 262.89 0)
+		(at 113.03 262.89 0)
 		(unit 1)
 		(exclude_from_sim no)
@@
 		(fields_autoplaced yes)
 		(property "Reference" "JP1"
-			(at 111.76 259.08 0)
+			(at 113.03 259.08 0)
 			(effects
 				(font
@@
 		)
 		(property "Value" "J"
-			(at 111.76 265.43 0)
+			(at 113.03 265.43 0)
 			(effects
 				(font
@@
 		)
 		(property "Footprint" "0_misc:SolderJumper-2_P1.3mm_Bridged_RoundedPad1.0x1.5mm"
-			(at 111.76 262.89 0)
+			(at 113.03 262.89 0)
 			(effects
 				(font
@@
 		)
 		(property "Datasheet" "~"
-			(at 111.76 262.89 0)
+			(at 113.03 262.89 0)
 			(effects
 				(font
@@
 		)
 		(property "Description" "Solder Jumper, 2-pole, closed/bridged"
-			(at 111.76 262.89 0)
-			(effects
-				(font
+			(at 113.03 262.89 0)
+			(effects
+				(font

Commit message: much work and .ioc file added
Parts:
- C23, C24: value 6p -> 10p
- C25, C26: value 15p -> 20p
Connections:
- net BOOT: now also U1.138 (BOOT0)
- net GND: no longer JP2.2 (B)
- net HSE_IN: now also U1.23 (PH0)
- net HSE_OUT: now also U1.24 (PH1)
- net LSE_IN: now also U1.8 (PC14)
- net LSE_OUT: now also U1.9 (PC15)
- net USB_N: now reaches U1.103 (PA11)
- net USB_P: now reaches U1.104 (PA12)
- net SWCLK: now reaches U1.109 (PA14)
- net NRST: now reaches U1.25 (NRST)
- net SD_CMD: now reaches U1.34 (PA0)
- new net +3V3: JP2.2 (B)
Other:
- note added: "https://community.st.com/t5/stm32-mcus/how-to-select-a-compatible-crystal-and-load-capacitors-for-stm32/ta-p/780236"
- moved on the sheet: U1B, U1C
