File: misc.kicad_sch (KiCad schematic)
At the start: 0 parts

Commit message: yeah
Parts:
- added FID1, FID2, FID3, FID4, FID5, FID6: Fiducial, symbol Mechanical:Fiducial
- added H1, H2, H3, H4: M3, MountingHole:MountingHole_3.2mm_M3_DIN965_Pad, symbol Mechanical:MountingHole_Pad_MP
Connections:
- new net GND: H1.MP, H2.MP, H3.MP, H4.MP
Other:
- note added: "FIDUCIALS"
- note added: "Logos and Graphics"
- note added: "Mounting Holes"
- title: (none) -> Misc.

Commit message: wen branch and pr
Other:
- note added: "FIDUCIALS (FRONT & BACK)"
- note added: "M3 MOUNTING HOLES"
- note removed: "FIDUCIALS"
- note removed: "Mounting Holes"
Changed lines of the file:
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@@
 	(rectangle
 		(start 25.4 63.5)
-		(end 87.63 88.9)
+		(end 87.63 90.17)
 		(stroke
 			(width 0.254)
@@
 		)
 	)
-	(text "FIDUCIALS"
+	(text "FIDUCIALS (FRONT & BACK)"
 		(exclude_from_sim no)
-		(at 34.29 60.96 0)
+		(at 52.07 60.96 0)
 		(effects
 			(font
@@
 		)
 	)
-	(text "Mounting Holes"
+	(text "M3 MOUNTING HOLES"
 		(exclude_from_sim no)
-		(at 128.27 60.96 0)
+		(at 134.62 60.96 0)
 		(effects
 			(font

Commit message: start fix fp
Parts:
- FID1, FID2, FID3, FID4, FID5, FID6: footprint (none) -> Fiducial:Fiducial_1mm_Mask3mm
- H1, H2, H3, H4: footprint MountingHole:MountingHole_3.2mm_M3_DIN965_Pad -> MountingHole:MountingHole_3.2mm_M3_Pad_Via
