File: hoppen_fc/interface.kicad_sch (KiCad schematic)
At the start: 58 parts, among them J10 GH1.25-4P, J11 PH2.0-3P, J12 GH1.25-4P, J13 PH2.0-3P, J14 GH1.25-5P, J15 GH1.25-8P, J16 PH2.0-3P, J17 GH1.25-2P, J18 GH1.25-8P, J4 GH1.25-4P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

Commit message: comments
Other:
- note added: "ACCOMODATE FOR DSHOT TELEMETRY ASWELL"
- note added: "CHANGE TO UPRIGHT CONNECTORS?"
- note added: "SPLIT UP IN MORE DOCUMENTS AND ADD TVS DIODES"
Changed lines of the file:
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@@
+		)
+	)
+	(text "SPLIT UP IN MORE DOCUMENTS AND ADD TVS DIODES\n"
+		(exclude_from_sim no)
+		(at 102.108 19.812 0)
+		(effects
+			(font
+				(face "KiCad Font")
+				(size 2.54 2.54)
+				(thickness 0.508)
+				(bold yes)
+				(color 255 0 0 1)
+			)
 		)
 	)
@@
 		)
 	)
+	(text "ACCOMODATE FOR DSHOT TELEMETRY ASWELL"
+		(exclude_from_sim no)
+		(at 148.844 32.258 0)
+		(effects
+			(font
+				(face "KiCad Font")
+				(size 2.54 2.54)
+				(thickness 0.508)
+				(bold yes)
+				(color 255 0 0 1)
+			)
+		)
+	)
 	(text "LIDAR INTERFACE #2"
 		(exclude_from_sim no)
@@
 			)
 		)
+	)
+	(text "CHANGE TO UPRIGHT CONNECTORS?"
+		(exclude_from_sim no)
+		(at 312.166 24.638 0)
+		(effects
+			(font
+				(face "KiCad Font")
+				(size 2.54 2.54)
+				(thickness 0.508)
+				(bold yes)
+				(color 255 0 0 1)
+			)
+		)

Commit message: comments
Other:
- note added: "BIGGER CONNECTORS?"
Changed lines of the file:
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@@
+		)
+	)
+	(text "BIGGER CONNECTORS?"
+		(exclude_from_sim no)
+		(at 197.104 39.116 0)
+		(effects
+			(font
+				(face "KiCad Font")
+				(size 2.54 2.54)
+				(thickness 0.508)
+				(bold yes)
+				(color 255 0 0 1)
+			)
 		)
 	)
