File: hoppen_fc/canbus.kicad_sch (KiCad schematic)
At the start: 8 parts, among them U14 TJA1051TK-3, U8 TJA1051TK-3

Commit message: finished adding lcsc numbers
Parts:
- C73: renamed from C43; LCSC (none) -> C307331
- C74: renamed from C44; LCSC (none) -> C307331
- C75: renamed from C79; LCSC (none) -> C307331
- C76: renamed from C80; LCSC (none) -> C307331
- R30: renamed from R16; LCSC (none) -> C25744
- R31: renamed from R51; LCSC (none) -> C25744
- renumbered U8 to U13
Changed lines of the file:
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@@
 		(dnp no)
 		(fields_autoplaced yes)
-		(property "Reference" "C80"
+		(property "Reference" "C76"
 			(at 210.82 80.0099 0)
 			(effects
@@
 			)
 		)
+		(property "LCSC" "C307331"
+			(at 207.01 81.28 0)
+			(effects
+				(font
+					(size 1.27 1.27)
+				)
+				(hide yes)
+			)
+		)
 		(pin "2"
 		)
@@
 			(project "hoppen_fc"
 				(path "/abe950a1-9eef-4508-9fd4-31d3e723e029/c85454e5-a89e-41eb-a5ed-71b4fc4cf13a/4b2dd471-a6f8-4e49-8717-912e41e4e851"
-					(reference "C80")
+					(reference "C76")
 					(unit 1)
 				)
@@
 		(dnp no)
 		(fields_autoplaced yes)
-		(property "Reference" "#PWR057"
+		(property "Reference" "#PWR0108"
 			(at 114.3 77.47 0)
 			(effects
@@
 			(project "hoppen_fc"
 				(path "/abe950a1-9eef-4508-9fd4-31d3e723e029/c85454e5-a89e-41eb-a5ed-71b4fc4cf13a/4b2dd471-a6f8-4e49-8717-912e41e4e851"
-					(reference "#PWR057")
+					(reference "#PWR0108")
 					(unit 1)
 				)
@@
 		(dnp no)
 		(fields_autoplaced yes)
-		(property "Reference" "#PWR055"
+		(property "Reference" "#PWR0111"
 			(at 86.36 93.98 0)
 			(effects
@@
 			(project "hoppen_fc"
 				(path "/abe950a1-9eef-4508-9fd4-31d3e723e029/c85454e5-a89e-41eb-a5ed-71b4fc4cf13a/4b2dd471-a6f8-4e49-8717-912e41e4e851"
-					(reference "#PWR055")
+					(reference "#PWR0111")
 					(unit 1)
 				)
@@
 		(dnp no)
 		(fields_autoplaced yes)
-		(property "Reference" "C44"
+		(property "Reference" "C74"
 			(at 118.11 80.0099 0)
 			(effects
@@
 			)
 		)
+		(property "LCSC" "C307331"
+			(at 114.3 81.28 0)
+			(effects
+				(font
+					(size 1.27 1.27)
+				)
+				(hide yes)
+			)
+		)
 		(pin "2"
 		)
@@
 			(project "hoppen_fc"
 				(path "/abe950a1-9eef-4508-9fd4-31d3e723e029/c85454e5-a89e-41eb-a5ed-71b4fc4cf13a/4b2dd471-a6f8-4e49-8717-912e41e4e851"
-					(reference "C44")
+					(reference "C74")
 					(unit 1)
 				)
@@
 		(dnp no)
 		(fields_autoplaced yes)
-		(property "Reference" "#PWR0134"
+		(property "Reference" "#PWR0113"
 			(at 179.07 93.98 0)
 			(effects
@@
 			(project "hoppen_fc"
 				(path "/abe950a1-9eef-4508-9fd4-31d3e723e029/c85454e5-a89e-41eb-a5ed-71b4fc4cf13a/4b2dd471-a6f8-4e49-8717-912e41e4e851"
-					(reference "#PWR0134")
+					(reference "#PWR0113")
 					(unit 1)
 				)
@@
 		(dnp no)
 		(fields_autoplaced yes)
-		(property "Reference" "#PWR0138"
+		(property "Reference" "#PWR0116"
 			(at 195.58 123.19 0)
 			(effects
@@
 			(project "hoppen_fc"
 				(path "/abe950a1-9eef-4508-9fd4-31d3e723e029/c85454e5-a89e-41eb-a5ed-71b4fc4cf13a/4b2dd471-a6f8-4e49-8717-912e41e4e851"
-					(reference "#PWR0138")
+					(reference "#PWR0116")
 					(unit 1)
 				)
@@
 		(dnp no)
 		(fields_autoplaced yes)
-		(property "Reference" "#PWR056"
+		(property "Reference" "#PWR0112"
 			(at 114.3 93.98 0)
 			(effects
@@
 			(project "hoppen_fc"
 				(path "/abe950a1-9eef-4508-9fd4-31d3e723e029/c85454e5-a89e-41eb-a5ed-71b4fc4cf13a/4b2dd471-a6f8-4e49-8717-912e41e4e851"
-					(reference "#PWR056")
+					(reference "#PWR0112")
 					(unit 1)
 				)
@@
 		(dnp no)
 		(fields_autoplaced yes)
-		(property "Reference" "#PWR0139"
+		(property "Reference" "#PWR0110"
 			(at 207.01 77.47 0)
 			(effects
@@
 			(project "hoppen_fc"
 				(path "/abe950a1-9eef-4508-9fd4-31d3e723e029/c85454e5-a89e-41eb-a5ed-71b4fc4cf13a/4b2dd471-a6f8-4e49-8717-912e41e4e851"
-					(reference "#PWR0139")
+					(reference "#PWR0110")
 					(unit 1)
 				)
@@
 		(dnp no)
 		(fields_autoplaced yes)
-		(property "Reference" "R16"
+		(property "Reference" "R30"
 			(at 85.09 109.2199 0)
 			(effects
@@
 			)
 		)
+		(property "LCSC" "C25744"
+			(at 82.55 110.49 0)
+			(effects
+				(font
+					(size 1.27 1.27)
+				)
+				(hide yes)
+			)
+		)
 		(pin "1"
 		)
@@
 			(project "hoppen_fc"
 				(path "/abe950a1-9eef-4508-9fd4-31d3e723e029/c85454e5-a89e-41eb-a5ed-71b4fc4cf13a/4b2dd471-a6f8-4e49-8717-912e41e4e851"
-					(reference "R16")
+					(reference "R30")
 					(unit 1)
 				)
@@
 		(dnp no)
 		(fields_autoplaced yes)
-		(property "Reference" "#PWR0140"
+		(property "Reference" "#PWR0114"
 			(at 207.01 93.98 0)
 			(effects
@@
 			(project "hoppen_fc"
 				(path "/abe950a1-9eef-4508-9fd4-31d3e723e029/c85454e5-a89e-41eb-a5ed-71b4fc4cf13a/4b2dd471-a6f8-4e49-8717-912e41e4e851"
-					(reference "#PWR0140")
+					(reference "#PWR0114")
 					(unit 1)
 				)
@@
 		(dnp no)
 		(fields_autoplaced yes)
-		(property "Reference" "R51"
+		(property "Reference" "R31"
 			(at 177.8 109.2199 0)
 			(effects
@@
 			)
 		)
+		(property "LCSC" "C25744"
+			(at 175.26 110.49 0)
+			(effects
+				(font
+					(size 1.27 1.27)
+				)
+				(hide yes)
+			)
+		)
 		(pin "1"
 		)
@@
 			(project "hoppen_fc"
 				(path "/abe950a1-9eef-4508-9fd4-31d3e723e029/c85454e5-a89e-41eb-a5ed-71b4fc4cf13a/4b2dd471-a6f8-4e49-8717-912e41e4e851"
-					(reference "R51")
+					(reference "R31")
 					(unit 1)
 				)
@@
 		(dnp no)
 		(fields_autoplaced yes)
-		(property "Reference" "#PWR058"
+		(property "Reference" "#PWR0107"
 			(at 86.36 77.47 0)
 			(effects
@@
 			(project "hoppen_fc"
 				(path "/abe950a1-9eef-4508-9fd4-31d3e723e029/c85454e5-a89e-41eb-a5ed-71b4fc4cf13a/4b2dd471-a6f8-4e49-8717-912e41e4e851"
-					(reference "#PWR058")
+					(reference "#PWR0107")
 					(unit 1)
 				)
@@
 		(dnp no)
 		(fields_autoplaced yes)
-		(property "Reference" "#PWR059"
+		(property "Reference" "#PWR0115"
 			(at 102.87 123.19 0)
 			(effects
@@
 			(project "hoppen_fc"
 				(path "/abe950a1-9eef-4508-9fd4-31d3e723e029/c85454e5-a89e-41eb-a5ed-71b4fc4cf13a/4b2dd471-a6f8-4e49-8717-912e41e4e851"
-					(reference "#PWR059")
+					(reference "#PWR0115")
 					(unit 1)
 				)
@@
 		(dnp no)
 		(fields_autoplaced yes)
-		(property "Reference" "#PWR0133"
+		(property "Reference" "#PWR0109"
 			(at 179.07 77.47 0)
 			(effects
@@
 			(project "hoppen_fc"
 				(path "/abe950a1-9eef-4508-9fd4-31d3e723e029/c85454e5-a89e-41eb-a5ed-71b4fc4cf13a/4b2dd471-a6f8-4e49-8717-912e41e4e851"
-					(reference "#PWR0133")
+					(reference "#PWR0109")
 					(unit 1)
 				)
@@
 		(dnp no)
 		(fields_autoplaced yes)
-		(property "Reference" "C79"
+		(property "Reference" "C75"
 			(at 182.88 80.0099 0)
 			(effects
@@
 			)
 		)
+		(property "LCSC" "C307331"
+			(at 179.07 81.28 0)
+			(effects
+				(font
+					(size 1.27 1.27)
+				)
+				(hide yes)
+			)
+		)
 		(pin "2"
 		)
@@
 			(project "hoppen_fc"
 				(path "/abe950a1-9eef-4508-9fd4-31d3e723e029/c85454e5-a89e-41eb-a5ed-71b4fc4cf13a/4b2dd471-a6f8-4e49-8717-912e41e4e851"
-					(reference "C79")
+					(reference "C75")
 					(unit 1)
 				)
@@
 		(dnp no)
 		(fields_autoplaced yes)
-		(property "Reference" "C43"
+		(property "Reference" "C73"
 			(at 90.17 80.0099 0)
 			(effects
@@
 			)
 		)
+		(property "LCSC" "C307331"
+			(at 86.36 81.28 0)
+			(effects
+				(font
+					(size 1.27 1.27)
+				)
+				(hide yes)
+			)
+		)
 		(pin "2"
 		)
@@
 			(project "hoppen_fc"
 				(path "/abe950a1-9eef-4508-9fd4-31d3e723e029/c85454e5-a89e-41eb-a5ed-71b4fc4cf13a/4b2dd471-a6f8-4e49-8717-912e41e4e851"
-					(reference "C43")
+					(reference "C73")
 					(unit 1)
 				)
@@
 		(on_board yes)
 		(dnp no)
-		(property "Reference" "U8"
+		(property "Reference" "U13"
 			(at 106.68 88.9 0)
 			(effects
@@
 			(project ""
 				(path "/abe950a1-9eef-4508-9fd4-31d3e723e029/c85454e5-a89e-41eb-a5ed-71b4fc4cf13a/4b2dd471-a6f8-4e49-8717-912e41e4e851"
-					(reference "U8")
-					(unit 1)
-				)
+					(reference "U13")
+					(unit 1)
+				)

Commit message: routing and adding rf module
Parts:
- renumbered R30 to R29, R31 to R30
Changed lines of the file:
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@@
 		(dnp no)
 		(fields_autoplaced yes)
-		(property "Reference" "R30"
+		(property "Reference" "R29"
 			(at 85.09 109.2199 0)
 			(effects
@@
 			(project "hoppen_fc"
 				(path "/abe950a1-9eef-4508-9fd4-31d3e723e029/c85454e5-a89e-41eb-a5ed-71b4fc4cf13a/4b2dd471-a6f8-4e49-8717-912e41e4e851"
-					(reference "R30")
+					(reference "R29")
 					(unit 1)
 				)
@@
 		(dnp no)
 		(fields_autoplaced yes)
-		(property "Reference" "R31"
+		(property "Reference" "R30"
 			(at 177.8 109.2199 0)
 			(effects
@@
 			(project "hoppen_fc"
 				(path "/abe950a1-9eef-4508-9fd4-31d3e723e029/c85454e5-a89e-41eb-a5ed-71b4fc4cf13a/4b2dd471-a6f8-4e49-8717-912e41e4e851"
-					(reference "R31")
+					(reference "R30")
 					(unit 1)
 				)

Commit message: bump
Parts:
- added TP37, TP38, TP39, TP40: TestPoint, TestPoint:TestPoint_Pad_1.0x1.0mm, symbol Connector:TestPoint
- renumbered C73 to C60, C74 to C61, C75 to C62, C76 to C63, R29 to R32, R30 to R33, U13 to U15, U14 to U16
Connections:
- net FDCAN1_RX: now also TP39.1
- net FDCAN1_TX: now also TP37.1
- net FDCAN2_RX: now also TP40.1
- net FDCAN2_TX: now also TP38.1

Commit message: bump
Parts:
- renumbered TP37 to TP52, TP38 to TP53, TP39 to TP54, TP40 to TP55
Changed lines of the file:
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@@
 		(dnp no)
 		(fields_autoplaced yes)
-		(property "Reference" "TP38"
+		(property "Reference" "TP53"
 			(at 215.9 126.9999 90)
 			(effects
@@
 			(project "hoppen_fc"
 				(path "/abe950a1-9eef-4508-9fd4-31d3e723e029/c85454e5-a89e-41eb-a5ed-71b4fc4cf13a/4b2dd471-a6f8-4e49-8717-912e41e4e851"
-					(reference "TP38")
+					(reference "TP53")
 					(unit 1)
 				)
@@
 		(dnp no)
 		(fields_autoplaced yes)
-		(property "Reference" "TP40"
+		(property "Reference" "TP55"
 			(at 215.9 129.5399 90)
 			(effects
@@
 			(project "hoppen_fc"
 				(path "/abe950a1-9eef-4508-9fd4-31d3e723e029/c85454e5-a89e-41eb-a5ed-71b4fc4cf13a/4b2dd471-a6f8-4e49-8717-912e41e4e851"
-					(reference "TP40")
+					(reference "TP55")
 					(unit 1)
 				)
@@
 		(dnp no)
 		(fields_autoplaced yes)
-		(property "Reference" "TP37"
+		(property "Reference" "TP52"
 			(at 123.19 126.9999 90)
 			(effects
@@
 			(project "hoppen_fc"
 				(path "/abe950a1-9eef-4508-9fd4-31d3e723e029/c85454e5-a89e-41eb-a5ed-71b4fc4cf13a/4b2dd471-a6f8-4e49-8717-912e41e4e851"
-					(reference "TP37")
+					(reference "TP52")
 					(unit 1)
 				)
@@
 		(dnp no)
 		(fields_autoplaced yes)
-		(property "Reference" "TP39"
+		(property "Reference" "TP54"
 			(at 123.19 129.5399 90)
 			(effects
@@
 			(project "hoppen_fc"
 				(path "/abe950a1-9eef-4508-9fd4-31d3e723e029/c85454e5-a89e-41eb-a5ed-71b4fc4cf13a/4b2dd471-a6f8-4e49-8717-912e41e4e851"
-					(reference "TP39")
-					(unit 1)
-				)
+					(reference "TP54")
+					(unit 1)
+				)
