File: hoppen_fc/power_generation.kicad_sch (KiCad schematic)
At the start: 0 parts

Commit message: power input/generation reworked
Parts:
- added C101: 39p, 0_capacitor_smd:C_0402_1005Metric, symbol Device:C
- added C102: 2n7, 0_capacitor_smd:C_0402_1005Metric, symbol Device:C
- added C103, C104, C108: 1u, 0_capacitor_smd:C_0603_1608Metric, symbol Device:C
- added C105, C106, C107, C111, C113, C114, C98: 100n, 0_capacitor_smd:C_0402_1005Metric, symbol Device:C
- added C109, C110, C112: 10u, 0_capacitor_smd:C_0603_1608Metric, symbol Device:C
- added C115, C116: 10u, 0_capacitor_smd:C_1210_3225Metric, symbol Device:C
- added C117, C118, C119: 22u, 0_capacitor_smd:C_1210_3225Metric, symbol Device:C
- added D13, D8, D9: GREEN 0402, 0_diodes:LED_0402_1005Metric, symbol Device:LED
- added F2: 500 mA @ 6V, 0_power:F0603, symbol Device:Fuse
- added L3: 4.7 uH 9A, 0_inductors:IND-SMD_L11.6-W10.1, symbol Device:L
- added R21: 115k, 0_resistor_smd:R_0402_1005Metric, symbol Device:R
- added R22: 22k1, 0_resistor_smd:R_0402_1005Metric, symbol Device:R
- added R46: 15k8, 0_resistor_smd:R_0402_1005Metric, symbol Device:R
- added R47: 200k, 0_resistor_smd:R_0402_1005Metric, symbol Device:R
- added R49, R54, R55, R68: 10k, 0_resistor_smd:R_0402_1005Metric, symbol Device:R
- added R50: 100k, 0_resistor_smd:R_0402_1005Metric, symbol Device:R
- added R57: 3k57, 0_resistor_smd:R_0402_1005Metric, symbol Device:R
- added R60: 1k15, 0_resistor_smd:R_0402_1005Metric, symbol Device:R
- added R67: 90k, 0_resistor_smd:R_0402_1005Metric, symbol Device:R
- added R69, R72: 39k, 0_resistor_smd:R_0402_1005Metric, symbol Device:R
- added R70: 1k5, 0_resistor_smd:R_0402_1005Metric, symbol Device:R
- added R71: 1k, 0_resistor_smd:R_0402_1005Metric, symbol Device:R
- added R73: 10K, 0_resistor_smd:R_0402_1005Metric, symbol Device:R
- added U17: AP64500, 0_power:SO-8-EP, symbol 0_power:AP64500
- added U18: TPS2116DRL, 0_power:SOT-583-8_L2.1-W1.6-P0.50-LS1.6-BL, symbol 0_power:TPS2116DRL
- added U19: TPS74801DRC, 0_power:VSON-10, symbol 0_power:TPS74801DRC
Connections:
- new net: C110.2, R55.1, U19.1 (IN), U19.2 (IN), U19.4 (BIAS), U19.5 (EN)
- new net +3V3: C111.2, C112.2, R57.2, R71.1, U19.10 (OUT), U19.9 (OUT)
- new net +3V3_PRE_LED: D9.2 (A), R71.2
- new net +5V: C107.2, C108.2, C109.2, R54.1, R70.1, R72.2, U18.2 (VOUT), U18.7 (VOUT)
- new net +5V_EXT: C103.2, C105.2, C117.1, C118.1, C119.1, L3.2, R21.1, R49.1, U18.3 (VIN1), U18.5 (MODE)
- new net +5V_PRE_LED: D8.2 (A), R70.2
- new net +5V_VMON: C114.2, R72.1, R73.2
- new net +BAT_PROT: C115.1, C116.1, R67.2, R69.1, U17.2 (VIN), U17.3 (EN)
- new net +BAT_VMON: C113.2, R67.1, R68.2
- new net +VBUS: F2.1
- new net BAT_PROT_PRE_LED: D13.2 (A), R69.2
- new net BUCK_BST: C98.2, U17.1 (BST)
- new net BUCK_CLK: R47.1, U17.4 (RT/CLK)
- new net BUCK_COMP: C101.1, R46.1, U17.6 (COMP)
- new net BUCK_COMP_2: C102.1, R46.2
- new net BUCK_FB: R21.2, R22.1, U17.5 (FB)
- new net BUCK_SW: C98.1, L3.1, U17.8 (SW)
- new net GND: C101.2, C102.2, C103.1, C104.1, C105.1, C106.1, C107.1, C108.1, C109.1, C110.1, C111.1, C112.1, C113.1, C114.1, C115.2, C116.2, C117.2, C118.2, C119.2, D13.1 (K), D8.1 (K), D9.1 (K), R22.2, R47.2, R50.2, R60.1, R68.1, R73.1, U17.7 (GND), U17.9 (EPAD), U18.1 (GND), U19.11 (GND), U19.6 (GND)
- new net LDO_FB: R57.1, R60.2, U19.8 (FB)
- new net LDO_PG: R55.2, U19.3 (PG)
- new net MUX_PR1: R49.2, R50.1, U18.4 (PR1)
- new net MUX_ST: R54.2, U18.8 (ST)
- new net MUX_VBUS: C104.2, C106.2, F2.2, U18.6 (VIN2)
- no-connect marks 0 -> 1
Other:
- note added: "3V3 @ 1.5A LDO"
- note added: "5V BUCK"
- note added: "5V MUX"
- note added: "PWR LEDs"
- note added: "VOLTAGE MONITORING"
- company: (none) -> Hoppen
- title: (none) -> Power Generation

Commit message: finished routing, starting doublechecking and componenting
Parts:
- removed C115, C116: 10u, 0_capacitor_smd:C_1210_3225Metric, symbol Device:C
- added C67, C70: 10u, 0_capacitor_smd:C_0805_2012Metric, symbol Device:C
Connections:
- net +BAT_PROT: now also C67.1, C70.1
- net GND: now also C67.2, C70.2
Changed lines of the file:
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@@
 	)
 	(junction
+		(at 34.29 50.8)
+		(diameter 0)
+		(color 0 0 0 0)
+	)
+	(junction
 		(at 193.04 78.74)
 		(diameter 0)
@@
 	)
 	(junction
-		(at 34.29 50.8)
-		(diameter 0)
-		(color 0 0 0 0)
-	)
-	(junction
 		(at 193.04 90.17)
 		(diameter 0)
@@
 	)
 	(junction
+		(at 45.72 50.8)
+		(diameter 0)
+		(color 0 0 0 0)
+	)
+	(junction
 		(at 111.76 50.8)
 		(diameter 0)
@@
 	)
 	(junction
-		(at 45.72 50.8)
-		(diameter 0)
-		(color 0 0 0 0)
-	)
-	(junction
 		(at 54.61 50.8)
 		(diameter 0)
@@
 	(wire
 		(pts
-			(xy 29.21 50.8) (xy 34.29 50.8)
-		)
-		(stroke
-			(width 0)
-			(type default)
-		)
-	)
-	(wire
-		(pts
 			(xy 176.53 138.43) (xy 176.53 153.67)
 		)
@@
 	(wire
 		(pts
-			(xy 34.29 50.8) (xy 45.72 50.8)
-		)
-		(stroke
-			(width 0)
-			(type default)
-		)
-	)
-	(wire
-		(pts
 			(xy 35.56 129.54) (xy 35.56 128.27)
 		)
@@
 	(wire
 		(pts
-			(xy 45.72 50.8) (xy 54.61 50.8)
+			(xy 29.21 50.8) (xy 34.29 50.8)
 		)
 		(stroke
@@
 	(wire
 		(pts
+			(xy 45.72 50.8) (xy 54.61 50.8)
+		)
+		(stroke
+			(width 0)
+			(type default)
+		)
+	)
+	(wire
+		(pts
 			(xy 195.58 50.8) (xy 205.74 50.8)
 		)
@@
 	(wire
 		(pts
+			(xy 34.29 50.8) (xy 45.72 50.8)
+		)
+		(stroke
+			(width 0)
+			(type default)
+		)
+	)
+	(wire
+		(pts
 			(xy 237.49 50.8) (xy 237.49 53.34)
 		)
@@
 	)
 	(symbol
+		(lib_id "Device:C")
+		(at 45.72 54.61 0)
+		(unit 1)
+		(exclude_from_sim no)
+		(in_bom yes)
+		(on_board yes)
+		(dnp no)
+		(property "Reference" "C67"
+			(at 45.72 52.07 0)
+			(effects
+				(font
+					(size 1.27 1.27)
+				)
+				(justify left)
+			)
+		)
+		(property "Value" "10u"
+			(at 45.72 57.15 0)
+			(effects
+				(font
+					(size 1.27 1.27)
+				)
+				(justify left)
+			)
+		)
+		(property "Footprint" "0_capacitor_smd:C_0805_2012Metric"
+			(at 46.6852 58.42 0)
+			(effects
+				(font
+					(size 1.27 1.27)
+				)
+				(hide yes)
+			)
+		)
+		(property "Datasheet" "~"
+			(at 45.72 54.61 0)
+			(effects
+				(font
+					(size 1.27 1.27)
+				)
+				(hide yes)
+			)
+		)
+		(property "Description" "Unpolarized capacitor"
+			(at 45.72 54.61 0)
+			(effects
+				(font
+					(size 1.27 1.27)
+				)
+				(hide yes)
+			)
+		)
+		(property "LCSC" "C440198"
+			(at 45.72 54.61 0)
+			(effects
+				(font
+					(size 1.27 1.27)
+				)
+				(hide yes)
+			)
+		)
+		(pin "2"
+		)
+		(pin "1"
+		)
+		(instances
+			(project "hoppen_fc"
+				(path "/abe950a1-9eef-4508-9fd4-31d3e723e029/c85454e5-a89e-41eb-a5ed-71b4fc4cf13a/304fa278-ecd3-4686-8fe4-afe398f93fb0"
+					(reference "C67")
+					(unit 1)
+				)
+			)
+		)
+	)
+	(symbol
 		(lib_id "power:GND")
 		(at 86.36 119.38 0)
@@
 	)
 	(symbol
-		(lib_id "Device:C")
-		(at 34.29 54.61 0)
-		(unit 1)
-		(exclude_from_sim no)
-		(in_bom yes)
-		(on_board yes)
-		(dnp no)
-		(fields_autoplaced yes)
-		(property "Reference" "C116"
-			(at 38.1 53.3399 0)
-			(effects
-				(font
-					(size 1.27 1.27)
-				)
-				(justify left)
-			)
-		)
-		(property "Value" "10u"
-			(at 38.1 55.8799 0)
-			(effects
-				(font
-					(size 1.27 1.27)
-				)
-				(justify left)
-			)
-		)
-		(property "Footprint" "0_capacitor_smd:C_1210_3225Metric"
-			(at 35.2552 58.42 0)
-			(effects
-				(font
-					(size 1.27 1.27)
-				)
-				(hide yes)
-			)
-		)
-		(property "Datasheet" "~"
-			(at 34.29 54.61 0)
-			(effects
-				(font
-					(size 1.27 1.27)
-				)
-				(hide yes)
-			)
-		)
-		(property "Description" "Unpolarized capacitor"
-			(at 34.29 54.61 0)
-			(effects
-				(font
-					(size 1.27 1.27)
-				)
-				(hide yes)
-			)
-		)
-		(property "LCSC" "C13585"
-			(at 34.29 54.61 0)
-			(effects
-				(font
-					(size 1.27 1.27)
-				)
-				(hide yes)
-			)
-		)
-		(pin "2"
-		)
-		(pin "1"
-		)
-		(instances
-			(project "hoppen_fc"
-				(path "/abe950a1-9eef-4508-9fd4-31d3e723e029/c85454e5-a89e-41eb-a5ed-71b4fc4cf13a/304fa278-ecd3-4686-8fe4-afe398f93fb0"
-					(reference "C116")
-					(unit 1)
-				)
-			)
-		)
-	)
-	(symbol
 		(lib_id "Device:R")
 		(at 52.07 118.11 90)
@@
 	)
 	(symbol
+		(lib_id "Device:C")
+		(at 34.29 54.61 0)
+		(unit 1)
+		(exclude_from_sim no)
+		(in_bom yes)
+		(on_board yes)
+		(dnp no)
+		(property "Reference" "C70"
+			(at 34.29 52.07 0)
+			(effects
+				(font
+					(size 1.27 1.27)
+				)
+				(justify left)
+			)
+		)
+		(property "Value" "10u"
+			(at 34.29 57.15 0)
+			(effects
+				(font
+					(size 1.27 1.27)
+				)
+				(justify left)
+			)
+		)
+		(property "Footprint" "0_capacitor_smd:C_0805_2012Metric"
+			(at 35.2552 58.42 0)
+			(effects
+				(font
+					(size 1.27 1.27)
+				)
+				(hide yes)
+			)
+		)
+		(property "Datasheet" "~"
+			(at 34.29 54.61 0)
+			(effects
+				(font
+					(size 1.27 1.27)
+				)
+				(hide yes)
+			)
+		)
+		(property "Description" "Unpolarized capacitor"
+			(at 34.29 54.61 0)
+			(effects
+				(font
+					(size 1.27 1.27)
+				)
+				(hide yes)
+			)
+		)
+		(property "LCSC" "C440198"
+			(at 34.29 54.61 0)
+			(effects
+				(font
+					(size 1.27 1.27)
+				)
+				(hide yes)
+			)
+		)
+		(pin "2"
+		)
+		(pin "1"
+		)
+		(instances
+			(project "hoppen_fc"
+				(path "/abe950a1-9eef-4508-9fd4-31d3e723e029/c85454e5-a89e-41eb-a5ed-71b4fc4cf13a/304fa278-ecd3-4686-8fe4-afe398f93fb0"
+					(reference "C70")
+					(unit 1)
+				)
+			)
+		)
+	)
+	(symbol
 		(lib_id "Device:R")
 		(at 237.49 59.69 0)
@@
 					(unit 1)
 				)
-			)
-		)
-	)
-	(symbol
-		(lib_id "Device:C")
-		(at 45.72 54.61 0)
-		(unit 1)
-		(exclude_from_sim no)
-		(in_bom yes)
-		(on_board yes)
-		(dnp no)
-		(fields_autoplaced yes)
-		(property "Reference" "C115"
-			(at 49.53 53.3399 0)
-			(effects
-				(font
-					(size 1.27 1.27)
-				)
-				(justify left)
-			)
-		)
-		(property "Value" "10u"
-			(at 49.53 55.8799 0)
-			(effects
-				(font
-					(size 1.27 1.27)
-				)
-				(justify left)
-			)
-		)
-		(property "Footprint" "0_capacitor_smd:C_1210_3225Metric"
-			(at 46.6852 58.42 0)
-			(effects
-				(font
-					(size 1.27 1.27)
-				)
-				(hide yes)
-			)
-		)
-		(property "Datasheet" "~"
-			(at 45.72 54.61 0)
-			(effects
-				(font
-					(size 1.27 1.27)
-				)
-				(hide yes)
-			)
-		)
-		(property "Description" "Unpolarized capacitor"
-			(at 45.72 54.61 0)
-			(effects
-				(font
-					(size 1.27 1.27)
-				)
-				(hide yes)
-			)
-		)
-		(property "LCSC" "C13585"
-			(at 45.72 54.61 0)
-			(effects
-				(font
-					(size 1.27 1.27)
-				)
-				(hide yes)
-			)
-		)
-		(pin "2"
-		)
-		(pin "1"
-		)
-		(instances
-			(project "hoppen_fc"
-				(path "/abe950a1-9eef-4508-9fd4-31d3e723e029/c85454e5-a89e-41eb-a5ed-71b4fc4cf13a/304fa278-ecd3-4686-8fe4-afe398f93fb0"
-					(reference "C115")
-					(unit 1)
-				)

Commit message: finished adding lcsc numbers
Parts:
- removed C101: 39p, 0_capacitor_smd:C_0402_1005Metric, symbol Device:C
- removed C112: 10u, 0_capacitor_smd:C_0603_1608Metric, symbol Device:C
- removed R55: 10k, 0_resistor_smd:R_0402_1005Metric, symbol Device:R
- added C36: 47p, 0_capacitor_smd:C_0402_1005Metric, symbol Device:C
- added C50: 10u, 0_capacitor_smd:C_0805_2012Metric, symbol Device:C
- C35: renamed from C98; LCSC (none) -> C307331
- C40: renamed from C103; LCSC (none) -> C15849
- C41: renamed from C105; LCSC (none) -> C307331
- C42: renamed from C107; LCSC (none) -> C307331
- C43: renamed from C108; LCSC (none) -> C15849
- C44: renamed from C109; footprint 0_capacitor_smd:C_0603_1608Metric -> 0_capacitor_smd:C_0805_2012Metric; LCSC (none) -> C440198
- C45: renamed from C104; LCSC (none) -> C15849
- C46: renamed from C106; LCSC (none) -> C307331
- C47: renamed from C102; LCSC (none) -> C106251
- C48: renamed from C110; footprint 0_capacitor_smd:C_0603_1608Metric -> 0_capacitor_smd:C_0805_2012Metric; LCSC (none) -> C440198
- C49: renamed from C111; LCSC (none) -> C307331
- C51: renamed from C113; LCSC (none) -> C307331
- C52: renamed from C114; LCSC (none) -> C307331
- D2: renamed from D13; value GREEN 0402 -> GREEN 0805; footprint 0_diodes:LED_0402_1005Metric -> 0_diodes:LED_0805_2012Metric; LCSC (none) -> C2297
- D3: renamed from D8; value GREEN 0402 -> GREEN 0805; footprint 0_diodes:LED_0402_1005Metric -> 0_diodes:LED_0805_2012Metric; LCSC (none) -> C2297
- D4: renamed from D9; value GREEN 0402 -> GREEN 0805; footprint 0_diodes:LED_0402_1005Metric -> 0_diodes:LED_0805_2012Metric; LCSC (none) -> C2297
- R10: renamed from R69; value 39k -> 33k; LCSC (none) -> C25779
- R11: renamed from R70; value 1k5 -> 1k; LCSC (none) -> C11702
- R12: renamed from R57; LCSC (none) -> C270609
- R13: renamed from R71; LCSC (none) -> C11702
- R14: renamed from R60; LCSC (none) -> C5159680
- R15: renamed from R67; value 90k -> 100k; LCSC (none) -> C25741
- R16: renamed from R72; value 39k -> 33k; LCSC (none) -> C25779
- R17: renamed from R68; LCSC (none) -> C25744
- R18: renamed from R73; value 10K -> 10k; LCSC (none) -> C25744
- R3: renamed from R21; LCSC (none) -> C3013150
- R4: renamed from R49; LCSC (none) -> C25744
- R5: renamed from R54; LCSC (none) -> C25744
- R6: renamed from R47; LCSC (none) -> C25764
- R7: renamed from R46; LCSC (none) -> C26956
- R8: renamed from R22; LCSC (none) -> C43473
- R9: renamed from R50; LCSC (none) -> C25741
- U6: renamed from U19; LCSC (none) -> C105263
- renumbered C70 to C33, C67 to C34, C117 to C37, C118 to C38, C119 to C39, F2 to F1, L3 to L2, U17 to U4, U18 to U5
Connections:
- net +3V3: now also C50.1
- net +5V: now also C48.2, U6.1 (IN), U6.2 (IN), U6.4 (BIAS), U6.5 (EN)
- net +5V_EXT: now also C36.1
- net BUCK_FB: now also C36.2
- net GND: now also C50.2
- net LDO_PG: no longer names the net of U6.3 (PG)
- no-connect marks 1 -> 2
Other:
- moved on the sheet: C37, C38, C39, L2, R3, R8

Commit message: ready for routing?
Changed lines of the file:
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@@
 	)
 	(junction
+		(at 130.81 50.8)
+		(diameter 0)
+		(color 0 0 0 0)
+	)
+	(junction
 		(at 124.46 67.31)
 		(diameter 0)
@@
 	)
 	(junction
-		(at 129.54 50.8)
-		(diameter 0)
-		(color 0 0 0 0)
-	)
-	(junction
 		(at 265.43 50.8)
 		(diameter 0)
@@
 	(wire
 		(pts
+			(xy 130.81 50.8) (xy 137.16 50.8)
+		)
+		(stroke
+			(width 0)
+			(type default)
+		)
+	)
+	(wire
+		(pts
 			(xy 62.23 184.15) (xy 73.66 184.15)
 		)
@@
 	(wire
 		(pts
-			(xy 129.54 49.53) (xy 129.54 50.8)
+			(xy 130.81 49.53) (xy 130.81 50.8)
 		)
 		(stroke
@@
 	(wire
 		(pts
-			(xy 124.46 50.8) (xy 129.54 50.8)
+			(xy 124.46 50.8) (xy 130.81 50.8)
 		)
 		(stroke
@@
 	(wire
 		(pts
-			(xy 129.54 49.53) (xy 128.27 49.53)
-		)
-		(stroke
-			(width 0)
-			(type default)
-		)
-	)
-	(wire
-		(pts
 			(xy 220.98 134.62) (xy 220.98 132.08)
 		)
@@
 	(wire
 		(pts
-			(xy 129.54 50.8) (xy 137.16 50.8)
-		)
-		(stroke
-			(width 0)
-			(type default)
-		)
-	)
-	(wire
-		(pts
 			(xy 205.74 50.8) (xy 210.82 50.8)
 		)
@@
 	(symbol
 		(lib_id "power:+3.3V")
-		(at 128.27 49.53 0)
+		(at 130.81 49.53 0)
 		(unit 1)
 		(exclude_from_sim no)
@@
 		(fields_autoplaced yes)
 		(property "Reference" "#PWR035"
-			(at 128.27 53.34 0)
+			(at 130.81 53.34 0)
 			(effects
 				(font
@@
 		)
 		(property "Value" "+5V_EXT"
-			(at 128.27 44.45 0)
+			(at 130.81 44.45 0)
 			(effects
 				(font
@@
 		)
 		(property "Footprint" ""
-			(at 128.27 49.53 0)
+			(at 130.81 49.53 0)
 			(effects
 				(font
@@
 		)
 		(property "Datasheet" ""
-			(at 128.27 49.53 0)
+			(at 130.81 49.53 0)
 			(effects
 				(font
@@
 		)
 		(property "Description" "Power symbol creates a global label with name \"+3.3V\""
-			(at 128.27 49.53 0)
+			(at 130.81 49.53 0)
 			(effects
 				(font

Commit message: routing and adding rf module
Parts:
- removed R10: 33k, 0_resistor_smd:R_0402_1005Metric, symbol Device:R
- removed R5: 10k, 0_resistor_smd:R_0402_1005Metric, symbol Device:R
- added R8: 10k, 0_resistor_smd:R_0402_1005Metric, symbol Device:R
- added TP4, TP5, TP6: TestPoint, TestPoint:TestPoint_Pad_1.0x1.0mm, symbol Connector:TestPoint
- C43: value 1u -> 10u; footprint 0_capacitor_smd:C_0603_1608Metric -> 0_capacitor_smd:C_0805_2012Metric; LCSC C15849 -> C440198
- L2: value 4.7 uH 9A -> 4.7 uH 6A; footprint 0_inductors:IND-SMD_L11.6-W10.1 -> 0_inductors:IND-SMD_L7.2-W6.6_GPSR07X0; LCSC C6364675 -> C5189754
- R9: value 100k -> 5k1; LCSC C25741 -> C25905
- renumbered R11 to R10, R12 to R11, R13 to R12, R14 to R13, R15 to R14, R16 to R15, R17 to R16, R18 to R17, R6 to R5, R7 to R6, R8 to R7
Connections:
- net +3V3: now also TP6.1
- net +5V: now also TP5.1
- net +5V_EXT: now also TP4.1
- net +BAT_PROT: now also R9.1
- net BAT_PROT_PRE_LED: now also R9.2
- net GND: now also R8.2; no longer R9.2
- net MUX_PR1: now also R8.1; no longer R9.1
- net MUX_ST: no longer names the net of U5.8 (ST)
- no-connect marks 2 -> 3
Other:
- moved on the sheet: C42, C44

Commit message: bump
Parts:
- renumbered TP4 to TP3, TP5 to TP4, TP6 to TP5
Changed lines of the file:
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@@
 		(dnp no)
 		(fields_autoplaced yes)
-		(property "Reference" "TP4"
+		(property "Reference" "TP3"
 			(at 143.51 42.4179 0)
 			(effects
@@
 			(project "hoppen_fc"
 				(path "/abe950a1-9eef-4508-9fd4-31d3e723e029/c85454e5-a89e-41eb-a5ed-71b4fc4cf13a/304fa278-ecd3-4686-8fe4-afe398f93fb0"
-					(reference "TP4")
+					(reference "TP3")
 					(unit 1)
 				)
@@
 		(dnp no)
 		(fields_autoplaced yes)
-		(property "Reference" "TP6"
+		(property "Reference" "TP5"
 			(at 266.7 127.5079 0)
 			(effects
@@
 			(project "hoppen_fc"
 				(path "/abe950a1-9eef-4508-9fd4-31d3e723e029/c85454e5-a89e-41eb-a5ed-71b4fc4cf13a/304fa278-ecd3-4686-8fe4-afe398f93fb0"
-					(reference "TP6")
+					(reference "TP5")
 					(unit 1)
 				)
@@
 		(dnp no)
 		(fields_autoplaced yes)
-		(property "Reference" "TP5"
+		(property "Reference" "TP4"
 			(at 275.59 46.2279 0)
 			(effects
@@
 			(project "hoppen_fc"
 				(path "/abe950a1-9eef-4508-9fd4-31d3e723e029/c85454e5-a89e-41eb-a5ed-71b4fc4cf13a/304fa278-ecd3-4686-8fe4-afe398f93fb0"
-					(reference "TP5")
-					(unit 1)
-				)
+					(reference "TP4")
+					(unit 1)
+				)

Commit message: bump
Parts:
- removed C33, C44, C48, C50: 10u, 0_capacitor_smd:C_0805_2012Metric, symbol Device:C
- removed C36: 47p, 0_capacitor_smd:C_0402_1005Metric, symbol Device:C
- removed C40, C45: 1u, 0_capacitor_smd:C_0603_1608Metric, symbol Device:C
- removed C46, C49: 100n, 0_capacitor_smd:C_0402_1005Metric, symbol Device:C
- removed R7: 22k1, 0_resistor_smd:R_0402_1005Metric, symbol Device:R
- removed TP3: TestPoint, TestPoint:TestPoint_Pad_1.0x1.0mm, symbol Connector:TestPoint
- removed U5: TPS2116DRL, 0_power:SOT-583-8_L2.1-W1.6-P0.50-LS1.6-BL, symbol 0_power:TPS2116DRL
- added C37: 22u, 0_capacitor_smd:C_0805_2012Metric, symbol Device:C
- added R10: 100k, 0_resistor_smd:R_0402_1005Metric, symbol Device:R
- added R11, R5: 33k, 0_resistor_smd:R_0402_1005Metric, symbol Device:R
- added R9: 20k, 0_resistor_smd:R_0402_1005Metric, symbol Device:R
- added TP5: TestPoint, TestPoint:TestPoint_Pad_1.0x1.0mm, symbol Connector:TestPoint
- added U6: TPS2121, Package_DFN_QFN:Texas_VQFN-HR-12_2x2.5mm_P0.5mm, symbol 0_power:TPS2121
- C36: renamed from C37; footprint 0_capacitor_smd:C_1210_3225Metric -> 0_capacitor_smd:C_0805_2012Metric; LCSC C12891 -> C45783
- C38: footprint 0_capacitor_smd:C_1210_3225Metric -> 0_capacitor_smd:C_0805_2012Metric; LCSC C12891 -> C45783
- C39: value 22u -> 100n; footprint 0_capacitor_smd:C_1210_3225Metric -> 0_capacitor_smd:C_0402_1005Metric; LCSC C12891 -> C307331
- C41, C42: value 100n -> 22u; footprint 0_capacitor_smd:C_0402_1005Metric -> 0_capacitor_smd:C_0805_2012Metric; LCSC C307331 -> C45783
- C43: value 10u -> 22u; LCSC C440198 -> C45783
- F1: footprint 0_power:F0603 -> Fuse:Fuse_0603_1608Metric
- R13: renamed from R10; LCSC C11702 -> C106235
- R15: renamed from R12; LCSC C11702 -> C106235
- R3: value 115k -> 100k; LCSC C3013150 -> C25741
- R4: value 10k -> 53k6; LCSC C25744 -> C53398
- renumbered C47 to C40, C51 to C44, C52 to C45, R9 to R12, R11 to R14, R13 to R16, R14 to R17, R15 to R18, R16 to R19, R17 to R20, R5 to R6, R6 to R7, TP5 to TP6, U4 to U5, U6 to U7
Connections:
- net +3V3: now also C42.1, C43.1
- net +5V: now also C41.1, U6.1 (OUT), U6.8 (OUT); no longer C42.2, C43.2, TP4.1
- net +5V_EXT: now also R3.2, R4.2, C37.1, U6.7 (IN1); no longer C39.1, C41.2, R3.1, R4.1
- net BUCK_FB: now also R4.1, R8.2, TP5.1; no longer R3.2
- net BUCK_SW: now also TP4.1
- net GND: now also C41.2, C42.2, C43.2, R8.1, C37.2, R11.1, R5.1, R9.1, U6.12 (GND), U6.4 (OV2), U6.5 (OV1), U6.9 (ST); no longer C41.1, C42.1, C43.1, R8.2
- net MUX_PR1: now also R3.1, R5.2, U6.6 (PR1); no longer R4.2, R8.1
- net MUX_VBUS renamed MUX_IN2
- net MUX_IN2: now also R10.2, U6.2 (IN2)
- new net MUX_ILM: R9.2, U6.10 (ILM)
- new net MUX_PR2: R10.1, R11.2, U6.3 (CP2)
- new net MUX_SS: C39.1, U6.11 (SS)
- no-connect marks 3 -> 2
Other:
- moved on the sheet: C34

Commit message: bump
Parts:
- removed TP4: TestPoint, TestPoint:TestPoint_Pad_1.0x1.0mm, symbol Connector:TestPoint
- renumbered TP5 to TP21, TP6 to TP22
Changed lines of the file:
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@@
 	)
 	(junction
-		(at 92.71 50.8)
-		(diameter 0)
-		(color 0 0 0 0)
-	)
-	(junction
 		(at 236.22 140.97)
 		(diameter 0)
@@
 	(wire
 		(pts
-			(xy 91.44 50.8) (xy 92.71 50.8)
-		)
-		(stroke
-			(width 0)
-			(type default)
-		)
-	)
-	(wire
-		(pts
 			(xy 226.06 57.15) (xy 227.33 57.15)
 		)
@@
 	(wire
 		(pts
-			(xy 92.71 50.8) (xy 93.98 50.8)
+			(xy 91.44 50.8) (xy 93.98 50.8)
 		)
 		(stroke
@@
 	(wire
 		(pts
-			(xy 92.71 45.72) (xy 92.71 50.8)
-		)
-		(stroke
-			(width 0)
-			(type default)
-		)
-	)
-	(wire
-		(pts
 			(xy 237.49 78.74) (xy 237.49 92.71)
 		)
@@
 	)
 	(symbol
-		(lib_id "Connector:TestPoint")
-		(at 92.71 45.72 0)
-		(unit 1)
-		(exclude_from_sim no)
-		(in_bom yes)
-		(on_board yes)
-		(dnp no)
-		(fields_autoplaced yes)
-		(property "Reference" "TP4"
-			(at 95.25 42.4179 0)
-			(effects
-				(font
-					(size 1.27 1.27)
-				)
-				(justify left)
-			)
-		)
-		(property "Value" "TestPoint"
-			(at 95.25 43.6879 0)
-			(effects
-				(font
-					(size 1.27 1.27)
-				)
-				(justify left)
-				(hide yes)
-			)
-		)
-		(property "Footprint" "TestPoint:TestPoint_Pad_1.0x1.0mm"
-			(at 97.79 45.72 0)
-			(effects
-				(font
-					(size 1.27 1.27)
-				)
-				(hide yes)
-			)
-		)
-		(property "Datasheet" "~"
-			(at 97.79 45.72 0)
-			(effects
-				(font
-					(size 1.27 1.27)
-				)
-				(hide yes)
-			)
-		)
-		(property "Description" "test point"
-			(at 92.71 45.72 0)
-			(effects
-				(font
-					(size 1.27 1.27)
-				)
-				(hide yes)
-			)
-		)
-		(pin "1"
-		)
-		(instances
-			(project "hoppen_fc"
-				(path "/abe950a1-9eef-4508-9fd4-31d3e723e029/c85454e5-a89e-41eb-a5ed-71b4fc4cf13a/304fa278-ecd3-4686-8fe4-afe398f93fb0"
-					(reference "TP4")
-					(unit 1)
-				)
-			)
-		)
-	)
-	(symbol
 		(lib_id "power:+3.3V")
 		(at 24.13 163.83 0)
@@
 		(dnp no)
 		(fields_autoplaced yes)
-		(property "Reference" "TP6"
+		(property "Reference" "TP22"
 			(at 266.7 127.5079 0)
 			(effects
@@
 			(project "hoppen_fc"
 				(path "/abe950a1-9eef-4508-9fd4-31d3e723e029/c85454e5-a89e-41eb-a5ed-71b4fc4cf13a/304fa278-ecd3-4686-8fe4-afe398f93fb0"
-					(reference "TP6")
+					(reference "TP22")
 					(unit 1)
 				)
@@
 		(dnp no)
 		(fields_autoplaced yes)
-		(property "Reference" "TP5"
+		(property "Reference" "TP21"
 			(at 95.25 64.0079 0)
 			(effects
@@
 			(project "hoppen_fc"
 				(path "/abe950a1-9eef-4508-9fd4-31d3e723e029/c85454e5-a89e-41eb-a5ed-71b4fc4cf13a/304fa278-ecd3-4686-8fe4-afe398f93fb0"
-					(reference "TP5")
+					(reference "TP21")
 					(unit 1)
 				)
