File: hoppen_fc/power_generation.kicad_sch (KiCad schematic)
At the start: 40 parts, among them U5 AP64500, U6 TPS2121, U7 TPS74801DRC

Commit message: production v1
Parts:
- removed R10, R3: 100k, 0_resistor_smd:R_0402_1005Metric, symbol Device:R
- removed R11, R5: 33k, 0_resistor_smd:R_0402_1005Metric, symbol Device:R
Connections:
- net MUX_PR1 is gone; now on net GND: U6.6 (PR1)
- net MUX_PR2 is gone; now on net GND: U6.3 (CP2)
- net +5V_EXT: now also U6.2 (IN2); no longer U6.7 (IN1)
- net MUX_IN2: now also U6.7 (IN1); no longer U6.2 (IN2)
