File: hoppen_fc/hoppen_fc.kicad_pcb (KiCad board)
At the start: 6 copper layers, 0 parts

Commit message: routing and adding rf module
Parts:
- added B1: FUET-5030, 0_indicators:BUZ-SMD_FST-5030, F.Cu at (136.0, 95.0)
- added C1: 2u2, 0_capacitor_smd:C_0603_1608Metric, F.Cu at (138.6, 56.3)
- added C10: 100n, 0_capacitor_smd:C_0402_1005Metric, F.Cu at (144.9, 58.0)
- added C100: 100n, 0_capacitor_smd:C_0402_1005Metric, F.Cu at (108.3, 55.3)
- added C101: 1u, 0_capacitor_smd:C_0603_1608Metric, F.Cu at (151.6, 25.2)
- added C102: 100n, 0_capacitor_smd:C_0402_1005Metric, F.Cu at (142.9, 20.9)
- added C103: 100n, 0_capacitor_smd:C_0402_1005Metric, F.Cu at (142.9, 22.8)
- added C104: 100n, 0_capacitor_smd:C_0402_1005Metric, F.Cu at (142.9, 24.8)
- added C105: 100n, 0_capacitor_smd:C_0402_1005Metric, F.Cu at (142.9, 26.8)
- added C11: 100n, 0_capacitor_smd:C_0402_1005Metric, F.Cu at (144.9, 60.0)
- added C12: 100n, 0_capacitor_smd:C_0402_1005Metric, F.Cu at (144.9, 61.9)
- added C13: 100n, 0_capacitor_smd:C_0402_1005Metric, F.Cu at (144.9, 63.9)
- added C14: 100n, 0_capacitor_smd:C_0402_1005Metric, F.Cu at (147.7, 56.0)
- added C15: 1u, 0_capacitor_smd:C_0603_1608Metric, F.Cu at (138.6, 63.8)
- added C16: 100n, 0_capacitor_smd:C_0402_1005Metric, F.Cu at (147.7, 58.0)
- added C17: 1u, 0_capacitor_smd:C_0603_1608Metric, F.Cu at (138.6, 66.3)
- added C18: 1u, 0_capacitor_smd:C_0603_1608Metric, F.Cu at (138.6, 68.8)
- added C19: 100n, 0_capacitor_smd:C_0402_1005Metric, F.Cu at (147.7, 60.0)
- added C2: 2u2, 0_capacitor_smd:C_0603_1608Metric, F.Cu at (138.6, 58.8)
- added C20: 100n, 0_capacitor_smd:C_0402_1005Metric, F.Cu at (140.8, 38.0)
- added C21: 100n, 0_capacitor_smd:C_0402_1005Metric, F.Cu at (140.8, 40.0)
- added C22: 100n, 0_capacitor_smd:C_0402_1005Metric, F.Cu at (140.8, 42.0)
- added C23: 10p, 0_capacitor_smd:C_0402_1005Metric, F.Cu at (140.8, 43.9)
- added C24: 10p, 0_capacitor_smd:C_0402_1005Metric, F.Cu at (140.8, 45.9)
- added C25: 10p, 0_capacitor_smd:C_0402_1005Metric, F.Cu at (140.8, 47.9)
- added C26: 10p, 0_capacitor_smd:C_0402_1005Metric, F.Cu at (140.8, 49.8)
- added C27: 100n, 0_capacitor_smd:C_0402_1005Metric, F.Cu at (48.0, 74.5)
- added C28: 1u, 0_capacitor_smd:C_0603_1608Metric, F.Cu at (53.0, 66.0)
- added C29: 10u, 0_capacitor_smd:C_0805_2012Metric, F.Cu at (35.9, 81.0)
- added C3: 4u7, 0_capacitor_smd:C_0603_1608Metric, F.Cu at (138.6, 61.3)
- added C30: 10u, 0_capacitor_smd:C_0805_2012Metric, F.Cu at (35.9, 84.0)
- added C31: 10u, 0_capacitor_smd:C_0805_2012Metric, F.Cu at (35.9, 87.0)
- added C32: 100n, 0_capacitor_smd:C_0402_1005Metric, F.Cu at (133.1, 67.0)
- added C33: 10u, 0_capacitor_smd:C_0805_2012Metric, F.Cu at (36.0, 77.0)
- added C34: 10u, 0_capacitor_smd:C_0805_2012Metric, F.Cu at (94.6, 25.8)
- added C35: 100n, 0_capacitor_smd:C_0402_1005Metric, F.Cu at (98.2, 34.2)
- added C36: 47p, 0_capacitor_smd:C_0402_1005Metric, F.Cu at (98.2, 36.2)
- added C37: 22u, 0_capacitor_smd:C_1210_3225Metric, F.Cu at (116.0, 94.0)
- added C38: 22u, 0_capacitor_smd:C_1210_3225Metric, F.Cu at (116.0, 98.2)
- added C39: 22u, 0_capacitor_smd:C_1210_3225Metric, F.Cu at (116.0, 102.5)
- added C4: 100n, 0_capacitor_smd:C_0402_1005Metric, F.Cu at (142.0, 56.0)
- added C40: 1u, 0_capacitor_smd:C_0603_1608Metric, F.Cu at (112.3, 35.3)
- added C41: 100n, 0_capacitor_smd:C_0402_1005Metric, F.Cu at (98.2, 38.1)
- added C42: 100n, 0_capacitor_smd:C_0402_1005Metric, F.Cu at (101.1, 34.2)
- added C43: 10u, 0_capacitor_smd:C_0805_2012Metric, F.Cu at (94.6, 28.8)
- added C44: 10u, 0_capacitor_smd:C_0805_2012Metric, F.Cu at (94.6, 31.8)
- added C45: 1u, 0_capacitor_smd:C_0603_1608Metric, F.Cu at (112.3, 37.8)
- added C46: 100n, 0_capacitor_smd:C_0402_1005Metric, F.Cu at (101.1, 36.2)
- added C47: 2n7, 0_capacitor_smd:C_0402_1005Metric, F.Cu at (101.1, 38.1)
- added C48: 10u, 0_capacitor_smd:C_0805_2012Metric, F.Cu at (94.6, 34.8)
- added C49: 100n, 0_capacitor_smd:C_0402_1005Metric, F.Cu at (104.0, 34.2)
- added C5: 100n, 0_capacitor_smd:C_0402_1005Metric, F.Cu at (142.0, 58.0)
- added C50: 10u, 0_capacitor_smd:C_0805_2012Metric, F.Cu at (94.6, 37.8)
- added C51: 100n, 0_capacitor_smd:C_0402_1005Metric, F.Cu at (104.0, 36.2)
- added C52: 100n, 0_capacitor_smd:C_0402_1005Metric, F.Cu at (104.0, 38.1)
- added C53: 4u7, 0_capacitor_smd:C_0603_1608Metric, F.Cu at (129.1, 45.1)
- added C54: 100n, 0_capacitor_smd:C_0402_1005Metric, F.Cu at (125.7, 38.0)
- added C55: 100n, 0_capacitor_smd:C_0402_1005Metric, F.Cu at (125.7, 40.0)
- added C56: 4u7, 0_capacitor_smd:C_0603_1608Metric, F.Cu at (129.1, 47.6)
- added C57: 100n, 0_capacitor_smd:C_0402_1005Metric, F.Cu at (125.7, 42.0)
- added C58: 4u7, 0_capacitor_smd:C_0603_1608Metric, F.Cu at (129.1, 50.1)
- added C59: 100n, 0_capacitor_smd:C_0402_1005Metric, F.Cu at (125.7, 43.9)
- added C6: 100n, 0_capacitor_smd:C_0402_1005Metric, F.Cu at (142.0, 60.0)
- added C60: 100n, 0_capacitor_smd:C_0402_1005Metric, F.Cu at (125.7, 45.9)
- added C61: 100n, 0_capacitor_smd:C_0402_1005Metric, F.Cu at (125.7, 47.9)
- added C62: 100n, 0_capacitor_smd:C_0402_1005Metric, F.Cu at (96.7, 73.3)
- added C63: 1u, 0_capacitor_smd:C_0603_1608Metric, F.Cu at (130.5, 29.3)
- added C64: 100n, 0_capacitor_smd:C_0402_1005Metric, F.Cu at (133.9, 29.1)
- added C65: 100n, 0_capacitor_smd:C_0402_1005Metric, F.Cu at (133.9, 31.0)
- added C66: 1u, 0_capacitor_smd:C_0603_1608Metric, F.Cu at (130.5, 31.8)
- added C67: 1u, 0_capacitor_smd:C_0603_1608Metric, F.Cu at (156.0, 64.8)
- added C68: 100n, 0_capacitor_smd:C_0402_1005Metric, F.Cu at (152.6, 56.0)
- added C69: 100n, 0_capacitor_smd:C_0402_1005Metric, F.Cu at (152.6, 58.0)
- added C7: 100n, 0_capacitor_smd:C_0402_1005Metric, F.Cu at (142.0, 61.9)
- added C70: 100n, 0_capacitor_smd:C_0402_1005Metric, F.Cu at (152.6, 60.0)
- added C71: 100n, 0_capacitor_smd:C_0402_1005Metric, F.Cu at (152.6, 61.9)
- added C72: 100n, 0_capacitor_smd:C_0402_1005Metric, F.Cu at (152.6, 63.9)
- added C73: 100n, 0_capacitor_smd:C_0402_1005Metric, F.Cu at (152.6, 69.0)
- added C74: 100n, 0_capacitor_smd:C_0402_1005Metric, F.Cu at (152.6, 71.0)
- added C75: 100n, 0_capacitor_smd:C_0402_1005Metric, F.Cu at (152.6, 72.9)
- added C76: 100n, 0_capacitor_smd:C_0402_1005Metric, F.Cu at (152.6, 74.9)
- added C77: 100n, 0_capacitor_smd:C_0402_1005Metric, F.Cu at (102.5, 51.4)
- added C78: 100n, 0_capacitor_smd:C_0402_1005Metric, F.Cu at (102.5, 53.3)
- added C79: 10u, 0_capacitor_smd:C_0805_2012Metric, F.Cu at (94.6, 42.8)
- added C8: 100n, 0_capacitor_smd:C_0402_1005Metric, F.Cu at (142.0, 63.9)
- added C80: 10u, 0_capacitor_smd:C_0805_2012Metric, F.Cu at (94.6, 45.9)
- added C81: 100n, 0_capacitor_smd:C_0402_1005Metric, F.Cu at (102.5, 55.3)
- added C82: 100n, 0_capacitor_smd:C_0402_1005Metric, F.Cu at (102.5, 57.3)
- added C83: 100n, 0_capacitor_smd:C_0402_1005Metric, F.Cu at (102.5, 59.2)
- added C84: 100n, 0_capacitor_smd:C_0402_1005Metric, F.Cu at (102.5, 61.2)
- added C85: 10u, 0_capacitor_smd:C_0805_2012Metric, F.Cu at (94.6, 48.9)
- added C86: 10u, 0_capacitor_smd:C_0805_2012Metric, F.Cu at (99.0, 42.8)
- added C87: 100n, 0_capacitor_smd:C_0402_1005Metric, F.Cu at (105.4, 51.4)
- added C88: 100n, 0_capacitor_smd:C_0402_1005Metric, F.Cu at (105.4, 53.3)
- added C89: 100n, 0_capacitor_smd:C_0402_1005Metric, F.Cu at (105.4, 55.3)
- added C9: 100n, 0_capacitor_smd:C_0402_1005Metric, F.Cu at (144.9, 56.0)
- added C90: 100n, 0_capacitor_smd:C_0402_1005Metric, F.Cu at (105.4, 57.3)
- added C91: 10u, 0_capacitor_smd:C_0805_2012Metric, F.Cu at (99.0, 45.9)
- added C92: 10u, 0_capacitor_smd:C_0805_2012Metric, F.Cu at (99.0, 48.9)
- added C93: 100n, 0_capacitor_smd:C_0402_1005Metric, F.Cu at (105.4, 59.2)
- added C94: 100n, 0_capacitor_smd:C_0402_1005Metric, F.Cu at (105.4, 61.2)
- added C95: 100n, 0_capacitor_smd:C_0402_1005Metric, F.Cu at (108.3, 51.4)
- added C96: 10u, 0_capacitor_smd:C_0805_2012Metric, F.Cu at (103.5, 42.8)
- added C97: 10u, 0_capacitor_smd:C_0805_2012Metric, F.Cu at (103.5, 45.9)
- added C98: 100n, 0_capacitor_smd:C_0402_1005Metric, F.Cu at (108.3, 53.3)
- added C99: 10u, 0_capacitor_smd:C_0805_2012Metric, F.Cu at (103.5, 48.9)
- added D1: SMBJ28CA, PCM_JLCPCB:D_SMB, F.Cu at (43.0, 64.2)
- added D10: SK6812, 0_indicators:LED-SMD_4P-L2.0-W2.0-BR, F.Cu at (123.0, 100.1)
- added D11: SK6812, 0_indicators:LED-SMD_4P-L2.0-W2.0-BR, F.Cu at (123.0, 103.8)
- added D12: SK6812, 0_indicators:LED-SMD_4P-L2.0-W2.0-BR, F.Cu at (123.0, 107.4)
- added D13: SK6812, 0_indicators:LED-SMD_4P-L2.0-W2.0-BR, F.Cu at (123.0, 111.0)
- added D2: GREEN 0805, 0_diodes:LED_0805_2012Metric, F.Cu at (103.9, 108.1)
- added D3: GREEN 0805, 0_diodes:LED_0805_2012Metric, F.Cu at (107.0, 108.1)
- added D4: GREEN 0805, 0_diodes:LED_0805_2012Metric, F.Cu at (110.0, 108.1)
- added D5: SMF5V0A, 0_diodes:D_SMF, F.Cu at (128.0, 57.0)
- added D6: SMF18A, PCM_JLCPCB:D_SOD-123FL, F.Cu at (108.5, 46.8)
- added D7: 1N4148W, Diode_SMD:D_SOD-123, F.Cu at (147.3, 17.9)
- added D8: GREEN 0805, 0_diodes:LED_0805_2012Metric, F.Cu at (113.0, 108.0)
- added D9: BLUE 0805, 0_diodes:LED_0805_2012Metric, F.Cu at (116.0, 108.0)
- added F1: 500 mA @ 6V, 0_power:F0603, F.Cu at (108.2, 19.7)
- added FID1: Fiducial, Fiducial:Fiducial_1mm_Mask2mm, F.Cu at (105.0, 66.0)
- added FID2: Fiducial, Fiducial:Fiducial_1mm_Mask2mm, F.Cu at (104.8, 69.6)
- added FID3: Fiducial, Fiducial:Fiducial_1mm_Mask2mm, F.Cu at (108.4, 66.1)
- added FID4: Fiducial, Fiducial:Fiducial_1mm_Mask2mm, F.Cu at (108.4, 69.6)
- added FID5: Fiducial, Fiducial:Fiducial_1mm_Mask2mm, F.Cu at (111.9, 66.1)
- added FID6: Fiducial, Fiducial:Fiducial_1mm_Mask2mm, F.Cu at (111.9, 69.6)
- added H1: M3, 0_misc:MountingHole_3.2mm_M3_Pad_Via, F.Cu at (85.0, 85.0)
- added H2: M3, 0_misc:MountingHole_3.2mm_M3_Pad_Via, F.Cu at (175.0, 85.0)
- added H3: M3, 0_misc:MountingHole_3.2mm_M3_Pad_Via, F.Cu at (85.0, 125.0)
- added H4: M3, 0_misc:MountingHole_3.2mm_M3_Pad_Via, F.Cu at (175.0, 125.0)
- added J1: XT30_MALE, 0_connectors:XT30PW-M, F.Cu at (88.0, 96.0)
- added J10: GH1.25-4P, 0_connectors:SM04B-GHS-TB-LF-SN, F.Cu at (174.0, 116.0)
- added J11: PH2.0-3P, 0_connectors:S3B-PH-SM4-TB-LF-SN, F.Cu at (114.0, 86.0)
- added J12: GH1.25-4P, 0_connectors:SM04B-GHS-TB-LF-SN, F.Cu at (135.0, 124.0)
- added J13: PH2.0-3P, 0_connectors:S3B-PH-SM4-TB-LF-SN, F.Cu at (126.0, 86.0)
- added J14: GH1.25-5P, 0_connectors:SM05B-GHS-TB-LF-SN, F.Cu at (174.0, 105.0)
- added J15: GH1.25-8P, 0_connectors:SM08B-GHS-TB-LF-SN, F.Cu at (163.0, 124.0)
- added J16: PH2.0-3P, 0_connectors:S3B-PH-SM4-TB-LF-SN, F.Cu at (138.0, 86.0)
- added J17: GH1.25-2P, 0_connectors:SM02B-GHS-TB-LF-SN, F.Cu at (96.1, 123.9)
- added J18: GH1.25-8P, 0_connectors:SM08B-GHS-TB-LF-SN, F.Cu at (148.0, 124.0)
- added J2: USB_C_Receptacle_USB2.0_16P, 0_connectors:USB-C_SMD-TYPE-C-31-M-12_1, F.Cu at (85.5, 116.0)
- added J3: MicroSD Card Holder, 0_storage:microSD_HC_Hirose_DM3D-SF, B.Cu at (125.6, 17.4)
- added J4: GH1.25-4P, 0_connectors:SM04B-GHS-TB-LF-SN, F.Cu at (113.3, 124.0)
- added J5: GH1.25-2P, 0_connectors:SM02B-GHS-TB-LF-SN, F.Cu at (104.0, 124.0)
- added J6: GH1.25-4P, 0_connectors:SM04B-GHS-TB-LF-SN, F.Cu at (174.0, 94.0)
- added J7: PH2.0-3P, 0_connectors:S3B-PH-SM4-TB-LF-SN, F.Cu at (102.0, 86.0)
- added J8: GH1.25-2P, 0_connectors:SM02B-GHS-TB-LF-SN, F.Cu at (83.6, 107.0)
- added J9: GH1.25-4P, 0_connectors:SM04B-GHS-TB-LF-SN, F.Cu at (124.0, 124.0)
- added JP1: J, 0_misc:SolderJumper-2_P1.3mm_Bridged_RoundedPad1.0x1.5mm, F.Cu at (151.0, 38.8)
- added JP2: J, 0_misc:SolderJumper-2_P1.3mm_Bridged_RoundedPad1.0x1.5mm, F.Cu at (151.0, 42.4)
- added JP3: J, 0_misc:SolderJumper-2_P1.3mm_Bridged_RoundedPad1.0x1.5mm, F.Cu at (111.9, 52.1)
- added JP4: J, 0_misc:SolderJumper-2_P1.3mm_Bridged_RoundedPad1.0x1.5mm, F.Cu at (111.9, 55.7)
- added JP5: SolderJumper_3_Open, Jumper:SolderJumper-3_P1.3mm_Open_Pad1.0x1.5mm, F.Cu at (108.5, 43.1)
- added L1: 600R@100MHz, Inductor_SMD:L_0603_1608Metric, F.Cu at (138.6, 71.3)
- added L2: 4.7 uH 6A, 0_inductors:IND-SMD_L7.2-W6.6_GPSR07X0, F.Cu at (110.0, 96.0)
- added Q1: NMOS, 0_transistors:DFN-8, B.Cu at (57.0, 73.0)
- added Q2: MMBT3904, Package_TO_SOT_SMD:SOT-23, F.Cu at (152.1, 20.0)
- added R1: 1k, 0_resistor_smd:R_0402_1005Metric, F.Cu at (143.7, 50.7)
- added R10: 1k, 0_resistor_smd:R_0402_1005Metric, F.Cu at (101.2, 24.3)
- added R11: 3k57, 0_resistor_smd:R_0402_1005Metric, F.Cu at (101.2, 26.2)
- added R12: 1k, 0_resistor_smd:R_0402_1005Metric, F.Cu at (101.2, 28.2)
- added R13: 1k15, 0_resistor_smd:R_0402_1005Metric, F.Cu at (101.2, 30.2)
- added R14: 100k, 0_resistor_smd:R_0402_1005Metric, F.Cu at (101.2, 32.2)
- added R15: 33k, 0_resistor_smd:R_0402_1005Metric, F.Cu at (104.1, 22.3)
- added R16: 10k, 0_resistor_smd:R_0402_1005Metric, F.Cu at (104.1, 24.3)
- added R17: 10k, 0_resistor_smd:R_0402_1005Metric, F.Cu at (104.1, 26.2)
- added R18: 33k, 0_resistor_smd:R_0402_1005Metric, F.Cu at (93.8, 65.3)
- added R19: 10k, 0_resistor_smd:R_0402_1005Metric, F.Cu at (93.8, 67.3)
- added R2: 10m, Resistor_SMD:R_1206_3216Metric, F.Cu at (48.5, 84.0)
- added R20: 22R, 0_resistor_smd:R_0402_1005Metric, F.Cu at (93.8, 69.3)
- added R21: 22R, 0_resistor_smd:R_0402_1005Metric, F.Cu at (93.8, 71.3)
- added R22: 5k1, 0_resistor_smd:R_0402_1005Metric, F.Cu at (93.8, 73.3)
- added R23: 5k1, 0_resistor_smd:R_0402_1005Metric, F.Cu at (93.8, 75.2)
- added R24: 47k, 0_resistor_smd:R_0402_1005Metric, F.Cu at (134.4, 10.9)
- added R25: 22R, 0_resistor_smd:R_0402_1005Metric, F.Cu at (134.4, 12.9)
- added R26: 22R, 0_resistor_smd:R_0402_1005Metric, F.Cu at (134.4, 14.9)
- added R27: 47k, 0_resistor_smd:R_0402_1005Metric, F.Cu at (134.4, 16.9)
- added R28: 47k, 0_resistor_smd:R_0402_1005Metric, F.Cu at (134.4, 18.9)
- added R29: 10k, 0_resistor_smd:R_0402_1005Metric, F.Cu at (155.5, 69.0)
- added R3: 115k, 0_resistor_smd:R_0402_1005Metric, F.Cu at (98.3, 22.3)
- added R30: 10k, 0_resistor_smd:R_0402_1005Metric, F.Cu at (155.5, 71.0)
- added R31: 22R, 0_resistor_smd:R_0402_1005Metric, F.Cu at (93.8, 51.4)
- added R32: 22R, 0_resistor_smd:R_0402_1005Metric, F.Cu at (93.8, 53.4)
- added R33: 47k, 0_resistor_smd:R_0402_1005Metric, F.Cu at (93.8, 55.3)
- added R34: 120R, 0_resistor_smd:R_0402_1005Metric, F.Cu at (93.8, 57.3)
- added R35: 47k, 0_resistor_smd:R_0402_1005Metric, F.Cu at (93.8, 59.3)
- added R36: 100k, 0_resistor_smd:R_0402_1005Metric, F.Cu at (93.8, 61.3)
- added R37: 22R, 0_resistor_smd:R_0402_1005Metric, F.Cu at (96.7, 51.4)
- added R38: 10k, 0_resistor_smd:R_0402_1005Metric, F.Cu at (96.7, 53.4)
- added R39: 22R, 0_resistor_smd:R_0402_1005Metric, F.Cu at (96.7, 55.3)
- added R4: 10k, 0_resistor_smd:R_0402_1005Metric, F.Cu at (98.3, 24.3)
- added R40: 120R, 0_resistor_smd:R_0402_1005Metric, F.Cu at (96.7, 57.3)
- added R41: 47k, 0_resistor_smd:R_0402_1005Metric, F.Cu at (96.7, 59.3)
- added R42: 22R, 0_resistor_smd:R_0402_1005Metric, F.Cu at (96.7, 61.3)
- added R43: 22R, 0_resistor_smd:R_0402_1005Metric, F.Cu at (99.6, 51.4)
- added R44: 47k, 0_resistor_smd:R_0402_1005Metric, F.Cu at (99.6, 53.4)
- added R45: 47k, 0_resistor_smd:R_0402_1005Metric, F.Cu at (99.6, 55.3)
- added R46: 1k, 0_resistor_smd:R_0402_1005Metric, F.Cu at (142.9, 10.9)
- added R47: 220R, 0_resistor_smd:R_0402_1005Metric, F.Cu at (142.9, 12.9)
- added R48: 1k, 0_resistor_smd:R_0402_1005Metric, F.Cu at (142.9, 14.9)
- added R49: 10k, 0_resistor_smd:R_0402_1005Metric, F.Cu at (142.9, 16.9)
- added R5: 200k, 0_resistor_smd:R_0402_1005Metric, F.Cu at (98.3, 26.2)
- added R50: 22R, 0_resistor_smd:R_0402_1005Metric, F.Cu at (142.9, 18.9)
- added R6: 15k8, 0_resistor_smd:R_0402_1005Metric, F.Cu at (98.3, 28.2)
- added R7: 22k1, 0_resistor_smd:R_0402_1005Metric, F.Cu at (98.3, 30.2)
- added R8: 10k, 0_resistor_smd:R_0402_1005Metric, F.Cu at (98.3, 32.2)
- added R9: 5k1, 0_resistor_smd:R_0402_1005Metric, F.Cu at (101.2, 22.3)
- added S1: ~, 0_misc:right_hand_rule, F.Cu at (159.0, 92.0)
- added SW1: SW_Push, 0_misc:SW-SMD_L3.9-W3.0-P4.45, F.Cu at (130.0, 101.5)
- added SW2: SW_Push, 0_misc:SW-SMD_L3.9-W3.0-P4.45, F.Cu at (169.0, 105.0)
- added SW3: SW_Push, 0_misc:SW-SMD_L3.9-W3.0-P4.45, F.Cu at (130.0, 110.0)
- added TP10: TestPoint, TestPoint:TestPoint_Pad_1.0x1.0mm, F.Cu at (119.6, 47.7)
- added TP11: TestPoint, TestPoint:TestPoint_Pad_1.0x1.0mm, F.Cu at (119.6, 50.8)
- added TP12: TestPoint, TestPoint:TestPoint_Pad_1.0x1.0mm, F.Cu at (122.7, 38.5)
- added TP13: TestPoint, TestPoint:TestPoint_Pad_1.0x1.0mm, F.Cu at (122.7, 41.6)
- added TP14: TestPoint, TestPoint:TestPoint_Pad_1.0x1.0mm, F.Cu at (122.7, 44.6)
- added TP15: TestPoint, TestPoint:TestPoint_Pad_1.0x1.0mm, F.Cu at (122.7, 47.7)
- added TP16: TestPoint, TestPoint:TestPoint_Pad_1.0x1.0mm, F.Cu at (122.7, 50.8)
- added TP2: TestPoint, TestPoint:TestPoint_Pad_1.0x1.0mm, F.Cu at (51.0, 78.0)
- added TP3: TestPoint, TestPoint:TestPoint_Pad_1.0x1.0mm, F.Cu at (51.0, 81.0)
- added TP4: TestPoint, TestPoint:TestPoint_Pad_1.0x1.0mm, F.Cu at (114.6, 11.4)
- added TP5: TestPoint, TestPoint:TestPoint_Pad_1.0x1.0mm, F.Cu at (114.6, 14.5)
- added TP6: TestPoint, TestPoint:TestPoint_Pad_1.0x1.0mm, F.Cu at (114.6, 17.6)
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Other:
- board outline added: 100 x 50 mm

Commit message: sync
Parts:
- added C98: 100n, 0_capacitor_smd:C_0402_1005Metric, F.Cu at (196.5, 68.8)
- added J19: U.FL, Connector_Coaxial:U.FL_Hirose_U.FL-R-SMT-1_Vertical, F.Cu at (218.5, 61.0)
- added U18: RFM95W-868S2, 0_rf:HOPERF_RFM9XW_SMD, F.Cu at (199.5, 59.0)

Commit message: bump
Parts:
- removed C100, C102, C103, C104, C105, C88, C89, C90, C93, C94, C95, C98 (x2): 100n, 0_capacitor_smd:C_0402_1005Metric
- removed C101: 1u, 0_capacitor_smd:C_0603_1608Metric
- removed C91, C92, C96, C97, C99: 10u, 0_capacitor_smd:C_0805_2012Metric
- removed the D9 at (116.0, 108.0)
- removed J19: U.FL, Connector_Coaxial:U.FL_Hirose_U.FL-R-SMT-1_Vertical
- removed TP10, TP11, TP12, TP13, TP14, TP15, TP16, TP3, TP7, TP8, TP9: TestPoint, TestPoint:TestPoint_Pad_1.0x1.0mm
- removed the TP5 at (114.6, 14.5)
- removed the U11 at (123.3, 31.6)
- removed the U15 at (113.6, 47.4)
- removed the U16 at (112.3, 59.9)
- removed the U5 at (113.2, 31.9)
- added D13: SMF18A, Diode_SMD:D_SOD-123, B.Cu at (94.5, 107.0)
- added R51: 47k, 0_resistor_smd:R_0402_1005Metric, B.Cu at (131.2, 89.0)
- added R52: 47k, 0_resistor_smd:R_0402_1005Metric, B.Cu at (131.2, 87.0)
- added R53: 120R, 0_resistor_smd:R_0402_1005Metric, B.Cu at (172.8, 94.7)
- added R54: 120R, 0_resistor_smd:R_0402_1005Metric, B.Cu at (172.8, 118.8)
- added R55: 100k, 0_resistor_smd:R_0402_1005Metric, B.Cu at (96.7, 105.8)
- added R56: 10k, 0_resistor_smd:R_0402_1005Metric, B.Cu at (96.7, 106.8)
- added R57: 22R, 0_resistor_smd:R_0402_1005Metric, B.Cu at (139.2, 100.7)
- added R58: 22R, 0_resistor_smd:R_0402_1005Metric, F.Cu at (131.2, 123.4)
- added TP1: TestPoint, TestPoint:TestPoint_Pad_1.0x1.0mm, F.Cu at (142.9, 120.8)
- added TP36: TestPoint, TestPoint:TestPoint_Pad_1.0x1.0mm, B.Cu at (155.0, 92.6)
- added TP37: TestPoint, TestPoint:TestPoint_Pad_1.0x1.0mm, B.Cu at (155.0, 90.5)
- added TP38: TestPoint, TestPoint:TestPoint_Pad_1.0x1.0mm, F.Cu at (164.4, 93.0)
- added TP39: TestPoint, TestPoint:TestPoint_Pad_1.0x1.0mm, F.Cu at (164.4, 115.0)
- added TP40: TestPoint, TestPoint:TestPoint_Pad_1.0x1.0mm, F.Cu at (164.4, 95.0)
- added TP41: TestPoint, TestPoint:TestPoint_Pad_1.0x1.0mm, F.Cu at (164.4, 117.0)
- added TP5: TestPoint, TestPoint:TestPoint_Pad_1.0x1.0mm, F.Cu at (113.5, 98.5)
- added TP5: TestPoint, TestPoint:TestPoint_Pad_1.0x1.0mm, F.Cu at (103.0, 90.5)
- added U12: W25Q128JVS, 0_storage:SOIC-8_5.3x5.3mm_P1.27mm, B.Cu at (141.4, 126.0)
- added U13: FM24C64B, Package_SO:SOIC-8_3.9x4.9mm_P1.27mm, B.Cu at (130.9, 126.0)
- added U19: PD4E1U, 0_transistors:SOT-363_SC-70-6, B.Cu at (111.7, 119.8)
- added U20: PD4E1U, 0_transistors:SOT-363_SC-70-6, B.Cu at (125.6, 87.0)
- added U21: 74AHCT1G125, 0_transceivers:SOT-23-5, B.Cu at (125.4, 116.1)
- added U22: PD4E1U, 0_transistors:SOT-363_SC-70-6, F.Cu at (168.2, 105.0)
- added U24: RFM95W-868S2, 0_rf:HOPERF_RFM9XW_SMD, B.Cu at (171.5, 105.0)
- added U4: LM74700, 0_power:SOT-23-6, B.Cu at (97.4, 102.2)
- added U7: TPS74801DRC, 0_power:VSON-10, B.Cu at (110.2, 106.0)
- C1, C10, C11, C12, C13, C14, C16, C2, C30, C31, C4, C46, C5, C54, C55, C57, C59, C6, C7, C79, C8, C80, C9, FID4, FID5, FID6, JP1, JP2, JP3, JP4, Q2, R1, R18, R19, R2, R21, R23, R28, R30, R39, R42, U17: moved to B.Cu
- C15, C17, C45: value 1u -> 100n; footprint 0_capacitor_smd:C_0603_1608Metric -> 0_capacitor_smd:C_0402_1005Metric; moved to B.Cu
- C18: footprint 0_capacitor_smd:C_0603_1608Metric -> 0_capacitor_smd:C_0402_1005Metric
- C20, C21: value 100n -> 1u
- C23, C24, C25: value 10p -> 100n; moved to B.Cu
- C27: value 100n -> 10p
- C28: value 1u -> 10p; footprint 0_capacitor_smd:C_0603_1608Metric -> 0_capacitor_smd:C_0402_1005Metric
- C29: value 10u -> 10p; footprint 0_capacitor_smd:C_0805_2012Metric -> 0_capacitor_smd:C_0402_1005Metric
- C3: value 4u7 -> 10u; footprint 0_capacitor_smd:C_0603_1608Metric -> 0_capacitor_smd:C_0805_2012Metric; moved to B.Cu
- C32, C51, C64, C73, C74, C75, C76, C77, C78, C81, C82: value 100n -> 10u; footprint 0_capacitor_smd:C_0402_1005Metric -> 0_capacitor_smd:C_0805_2012Metric; moved to B.Cu
- C33, C44, C48, C50, C85: value 10u -> 100n; footprint 0_capacitor_smd:C_0805_2012Metric -> 0_capacitor_smd:C_0402_1005Metric; moved to B.Cu
- C36: value 47p -> 22u; footprint 0_capacitor_smd:C_0402_1005Metric -> 0_capacitor_smd:C_0805_2012Metric
- C37, C38: footprint 0_capacitor_smd:C_1210_3225Metric -> 0_capacitor_smd:C_0805_2012Metric
- C39: value 22u -> 470n; footprint 0_capacitor_smd:C_1210_3225Metric -> 0_capacitor_smd:C_0402_1005Metric; moved to B.Cu
- C40: value 1u -> 2n7; footprint 0_capacitor_smd:C_0603_1608Metric -> 0_capacitor_smd:C_0402_1005Metric
- C41, C42, C69, C70, C71, C87: value 100n -> 22u; footprint 0_capacitor_smd:C_0402_1005Metric -> 0_capacitor_smd:C_0805_2012Metric; moved to B.Cu
- C43: value 10u -> 22u; moved to B.Cu
- C47: value 2n7 -> 100n; moved to B.Cu
- C49: value 100n -> 1u; moved to B.Cu
- C52: value 100n -> 10u; footprint 0_capacitor_smd:C_0402_1005Metric -> 0_capacitor_smd:C_0805_2012Metric
- C53, C56, C58: value 4u7 -> 100n; footprint 0_capacitor_smd:C_0603_1608Metric -> 0_capacitor_smd:C_0402_1005Metric; moved to B.Cu
- C63, C66, C67: value 1u -> 100n; footprint 0_capacitor_smd:C_0603_1608Metric -> 0_capacitor_smd:C_0402_1005Metric
- C72, C83, C84: value 100n -> 22u; footprint 0_capacitor_smd:C_0402_1005Metric -> 0_capacitor_smd:C_0805_2012Metric
- C86: value 10u -> 22u
- D1: footprint PCM_JLCPCB:D_SMB -> Diode_SMD:D_SMB; moved to B.Cu
- D6: value SMF18A -> 1N4148W; footprint PCM_JLCPCB:D_SOD-123FL -> Diode_SMD:D_SOD-123
- D7: value 1N4148W -> GREEN 0805; footprint Diode_SMD:D_SOD-123 -> 0_diodes:LED_0805_2012Metric
- D8: value GREEN 0805 -> BLUE 0805
- F1: footprint 0_power:F0603 -> Fuse:Fuse_0603_1608Metric
- J1: value XT30_MALE -> XT30 M
- J10: value GH1.25-4P -> B6B-PH; footprint 0_connectors:SM04B-GHS-TB-LF-SN -> Connector_JST:JST_PH_B6B-PH-K_1x06_P2.00mm_Vertical
- J11: value PH2.0-3P -> B6B-PH; footprint 0_connectors:S3B-PH-SM4-TB-LF-SN -> Connector_JST:JST_PH_B6B-PH-K_1x06_P2.00mm_Vertical
- J12, J4, J9: value GH1.25-4P -> BM04B-GHS1.25; footprint 0_connectors:SM04B-GHS-TB-LF-SN -> 0_connectors:BM04B-GHS1.25
- J13: value PH2.0-3P -> BM04B-GHS1.25; footprint 0_connectors:S3B-PH-SM4-TB-LF-SN -> 0_connectors:BM04B-GHS1.25
- J14: value GH1.25-5P -> BM02B-GHS1.25; footprint 0_connectors:SM05B-GHS-TB-LF-SN -> 0_connectors:BM02B-GHS1.25
- J15: value GH1.25-8P -> BM05B-GHS1.25; footprint 0_connectors:SM08B-GHS-TB-LF-SN -> 0_connectors:BM05B-GHS1.25
- J16: value PH2.0-3P -> BM02B-GHS1.25; footprint 0_connectors:S3B-PH-SM4-TB-LF-SN -> 0_connectors:BM02B-GHS1.25
- J17, J5, J8: value GH1.25-2P -> BM04B-GHS1.25; footprint 0_connectors:SM02B-GHS-TB-LF-SN -> 0_connectors:BM04B-GHS1.25
- J18: value GH1.25-8P -> U.FL; footprint 0_connectors:SM08B-GHS-TB-LF-SN -> Connector_Coaxial:U.FL_Hirose_U.FL-R-SMT-1_Vertical; moved to B.Cu
- J6: value GH1.25-4P -> BM06B-GHS1.25; footprint 0_connectors:SM04B-GHS-TB-LF-SN -> 0_connectors:BM06B-GHS-1.25
- J7: value PH2.0-3P -> BM08B-GHS1.25; footprint 0_connectors:S3B-PH-SM4-TB-LF-SN -> 0_connectors:BM08B-GHS1.25
- R10: value 1k -> 100k; moved to B.Cu
- R11: value 3k57 -> 33k; moved to B.Cu
- R12: value 1k -> 5k1; moved to B.Cu
- R13: value 1k15 -> 1k; moved to B.Cu
- R14: value 100k -> 3k57; moved to B.Cu
- R15: value 33k -> 1k; moved to B.Cu
- R16: value 10k -> 1k15; moved to B.Cu
- R17: value 10k -> 100k; moved to B.Cu
- R20, R31, R37: value 22R -> 10k; moved to B.Cu
- R22: value 5k1 -> 22R; moved to B.Cu
- R24: value 47k -> 5k1; moved to B.Cu
- R25: value 22R -> 47k
- R27, R45: value 47k -> 22R; moved to B.Cu
- R29, R49: value 10k -> 47k; moved to B.Cu
- R3: value 115k -> 100k; moved to B.Cu
- R32: value 22R -> 10k
- R33: value 47k -> 10k
- R34: value 120R -> 1k
- R35: value 47k -> 220R; moved to B.Cu
- R36: value 100k -> 1k
- R38: value 10k -> 22R; moved to B.Cu
- R4: value 10k -> 53k6
- R40: value 120R -> 22R; moved to B.Cu
- R41, R44: value 47k -> 22R
- R46: value 1k -> 22R
- R47: value 220R -> 47k; moved to B.Cu
- R48: value 1k -> 47k; moved to B.Cu
- R5: value 200k -> 33k; moved to B.Cu
- R50: value 22R -> 47k; moved to B.Cu
- R6: value 15k8 -> 200k; moved to B.Cu
- R7: value 22k1 -> 15k8
- R9: value 5k1 -> 20k; moved to B.Cu
- U18: value RFM95W-868S2 -> PD4E1U; footprint 0_rf:HOPERF_RFM9XW_SMD -> 0_transistors:SOT-363_SC-70-6
- U2: value INA180 -> PD4E1U; footprint 0_transceivers:SOT-23-5 -> 0_transistors:SOT-363_SC-70-6; moved to B.Cu
- U3: value LM74700 -> INA180; footprint 0_power:SOT-23-6 -> 0_transceivers:SOT-23-5
- U6: value TPS74801DRC -> TPS2121; footprint 0_power:VSON-10 -> Package_DFN_QFN:Texas_VQFN-HR-12_2x2.5mm_P0.5mm; moved to B.Cu
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- renumbered D11 to D10, D12 to D11, D13 to D12, D10 to D9, U9 to U10, U10 to U11, U12 to U14, U13 to U15, U14 to U16, U4 to U5, U7 to U8, U8 to U9
Connections:
- C15 pad 1: /Architecture/MCU Power/MCU_VDDA -> +3V3
- C16 pad 1: /Architecture/MCU Power/MCU_VDDA -> +3V3
- C20 pad 1: /Architecture/MCU IO/USER_BUTTON -> +3V3
- C21 pad 1: /Architecture/MCU IO/RST -> /Architecture/MCU Power/MCU_VDDA
- C22 pad 1: /Architecture/MCU IO/BOOT -> /Architecture/MCU Power/MCU_VDDA
- C23 pad 1: GND -> /Architecture/MCU IO/USER_BTN
- C23 pad 2: /Architecture/MCU IO/HSE_IN -> GND
- C24 pad 1: GND -> /Architecture/Interfaces - Comms/NRST
- C24 pad 2: /Architecture/MCU IO/HSE_OUT -> GND
- C25 pad 1: GND -> /Architecture/MCU IO/BOOT
- C25 pad 2: /Architecture/MCU IO/LSE_IN -> GND
- C26 pad 2: /Architecture/MCU IO/LSE_OUT -> /Architecture/MCU IO/HSE_IN
- C27 pad 1: +BAT -> GND
- C27 pad 2: GND -> /Architecture/MCU IO/HSE_OUT
- C28 pad 1: +BAT -> GND
- C28 pad 2: /Architecture/Power Input/ID_VCAP -> /Architecture/MCU IO/LSE_IN
- C29 pad 1: +BAT_PROT_PRE_MEAS -> GND
- C29 pad 2: GND -> /Architecture/MCU IO/LSE_OUT
- C30 pad 1: +BAT_PROT_PRE_MEAS -> +BAT
- C30 pad 2: GND -> /Architecture/Power Input/ID_VCAP
- C32 pad 1: +3V3 -> +BAT_PROT_PRE_MEAS
- C33 pad 1: +BAT_PROT -> +3V3
- C36 pad 2: /Architecture/Power Generation/BUCK_FB -> GND
- C39 pad 1: +5V_EXT -> /Architecture/Power Generation/MUX_SS
- C40 pad 1: GND -> /Architecture/Power Generation/BUCK_COMP_2
- C40 pad 2: +5V_EXT -> GND
- C41 pad 1: GND -> +5V
- C41 pad 2: +5V_EXT -> GND
- C42 pad 1: GND -> +3V3
- C42 pad 2: +5V -> GND
- C43 pad 1: GND -> +3V3
- C43 pad 2: +5V -> GND
- C44 pad 2: +5V -> /Architecture/MCU IO/+BAT_VMON
- C45 pad 2: /Architecture/Power Generation/MUX_VBUS -> /Architecture/MCU IO/+5V_VMON
- C46 pad 1: GND -> +3V3
- C46 pad 2: /Architecture/Power Generation/MUX_VBUS -> GND
- C47 pad 1: /Architecture/Power Generation/BUCK_COMP_2 -> +3V3
- C48 pad 1: GND -> +3V3
- C48 pad 2: +5V -> GND
- C49 pad 1: GND -> +3V3
- C49 pad 2: +3V3 -> GND
- C51 pad 2: /Architecture/MCU IO/+BAT_VMON -> /Architecture/Sensors/MAG_CAP
- C52 pad 1: GND -> +3V3
- C52 pad 2: /Architecture/MCU IO/+5V_VMON -> GND
- C56 pad 1: +3V3 -> /Architecture/RS232/RS232_C1_P
- C56 pad 2: GND -> /Architecture/RS232/RS232_C1_N
- C57 pad 1: +3V3 -> /Architecture/RS232/RS232_V_N
- C58 pad 1: +3V3 -> /Architecture/RS232/RS232_V_P
- C59 pad 1: +3V3 -> /Architecture/RS232/RS232_C2_P
- C59 pad 2: GND -> /Architecture/RS232/RS232_C2_N
- C60 pad 1: +3V3 -> +5V
- C61 pad 1: Net-(U9-CAP) -> +3V3
- C62 pad 1: /Architecture/MCU IO/+VBUS_VMON -> +5V
- C63 pad 1: GND -> +3V3
- C63 pad 2: +3V3 -> GND
- C64 pad 1: GND -> +3V3
- C64 pad 2: +3V3 -> GND
- C65 pad 1: +3V3 -> +5V
- C66 pad 1: +3V3 -> +5V
- C67 pad 1: +3V3 -> +5V
- C68 pad 1: +3V3 -> +5V
- C69 pad 1: /Architecture/RS232/RS232_C1_P -> +5V
- C69 pad 2: /Architecture/RS232/RS232_C1_N -> GND
- C70 pad 1: /Architecture/RS232/RS232_V_N -> +5V
- C71 pad 1: /Architecture/RS232/RS232_V_P -> +5V
- C72 pad 1: /Architecture/RS232/RS232_C2_P -> +5V
- C72 pad 2: /Architecture/RS232/RS232_C2_N -> GND
- C74 pad 1: +3V3 -> +5V
- C75 pad 1: +5V -> +BAT_PROT
- C76 pad 1: +3V3 -> +BAT_PROT
- C77 pad 1: +5V -> +BAT_PROT
- C81 pad 1: +5V_EXT -> +BAT_PROT
- C82 pad 1: /Architecture/Interfaces/CAM_PWR -> +BAT_PROT
- C84 pad 1: +BAT_PROT -> +5V
- C85 pad 1: +BAT_PROT -> /Architecture/MCU IO/EXT_BAT_VMON
- C86 pad 1: +BAT_PROT -> /Architecture/Interfaces - Comms/EXT_UART_PWR
- C87 pad 1: +5V_EXT -> +3V3
- D6 pad 1: /Architecture/Interfaces/EXT_BAT -> +3V3
- D6 pad 2: GND -> /Architecture/Indicators/BUZZER_N
- D7 pad 1: +3V3 -> /Architecture/Indicators/LED_1
- D7 pad 2: /Architecture/Indicators/BUZZER_N -> /Architecture/MCU IO/DBG_LED_1
- D8 pad 1: /Architecture/Indicators/LED_1 -> /Architecture/Indicators/LED_2
- D8 pad 2: /Architecture/MCU IO/DBG_LED_1 -> /Architecture/MCU IO/DBG_LED_2
- F1 pad 2: /Architecture/Power Generation/MUX_VBUS -> /Architecture/Power Generation/MUX_IN2
- J10 pad 1: +5V_EXT -> +BAT_PROT
- J10 pad 2: /Architecture/FDCAN/FDCAN2_H -> +BAT_PROT
- J10 pad 3: /Architecture/FDCAN/FDCAN2_L -> /Architecture/Interfaces - Actuators/PWM3
- J10 pad 4: GND -> /Architecture/Interfaces - Actuators/PWM4
- J11 pad 2: /Architecture/MCU IO/PWM2 -> +BAT_PROT
- J11 pad 3: GND -> /Architecture/Interfaces - Actuators/PWM5
- J12 pad 1: /Architecture/Interfaces/EXT_UART_PWR -> +5V
- J12 pad 2: /Architecture/Interfaces/EXT_UART_TX_T -> /Architecture/FDCAN/FDCAN1_H
- J12 pad 3: /Architecture/Interfaces/EXT_UART_RX_T -> /Architecture/FDCAN/FDCAN1_L
- J13 pad 1: +BAT_PROT -> +5V
- J13 pad 2: /Architecture/MCU IO/PWM3 -> /Architecture/FDCAN/FDCAN2_H
- J13 pad 3: GND -> /Architecture/FDCAN/FDCAN2_L
- J14 pad 1: +3V3 -> /Architecture/Interfaces - Comms/EXT_BAT
- J14 pad 2: /Architecture/Interfaces/SWDIO -> GND
- J15 pad 1: +5V -> +3V3
- J15 pad 2: /Architecture/Interfaces/VN_RS232_TX -> /Architecture/Interfaces - Comms/SWDIO
- J15 pad 3: /Architecture/Interfaces/VN_RS232_RX -> /Architecture/Interfaces - Comms/SWCLK
- J15 pad 4: /Architecture/MCU IO/VN_PPS -> /Architecture/Interfaces - Comms/NRST
- J15 pad 5: /Architecture/MCU IO/VN_SYNC -> GND
- J16 pad 1: +BAT_PROT -> /Architecture/Interfaces - Comms/EXT_LED_D_5V
- J16 pad 2: /Architecture/MCU IO/PWM4 -> GND
- J17 pad 1: /Architecture/Interfaces/EXT_LED_D_5V -> /Architecture/Interfaces - Comms/EXT_UART_PWR
- J17 pad 2: GND -> /Architecture/Interfaces - Comms/EXT_UART_TX_T
- J18 pad 1: +5V -> /Architecture/Radio/RFM_ANT
- J18 pad 2: /Architecture/Interfaces/RTK_UART_TX -> GND
- J4 pad 2: /Architecture/Interfaces/LIDAR1_T_UART_TX -> /Architecture/Interfaces - Sensors/LIDAR1_T_UART_TX
- J4 pad 3: /Architecture/Interfaces/LIDAR1_T_UART_RX -> /Architecture/Interfaces - Sensors/LIDAR1_T_UART_RX
- J5 pad 1: /Architecture/Interfaces/CAM_PWR -> +5V
- J5 pad 2: GND -> /Architecture/Interfaces - Sensors/LIDAR2_T_UART_TX
- J6 pad 1: +5V_EXT -> +5V
- J6 pad 2: /Architecture/FDCAN/FDCAN1_H -> /Architecture/Interfaces - Sensors/RTK_UART_TX_T
- J6 pad 3: /Architecture/FDCAN/FDCAN1_L -> /Architecture/Interfaces - Sensors/RTK_UART_RX_T
- J6 pad 4: GND -> /Architecture/MCU IO/RTK_PPS
- J7 pad 1: +BAT_PROT -> +5V
- J7 pad 2: /Architecture/MCU IO/PWM1 -> /Architecture/Interfaces - Sensors/VN_RS232_TX
- J7 pad 3: GND -> /Architecture/Interfaces - Sensors/VN_RS232_RX
- J8 pad 1: /Architecture/Interfaces/EXT_BAT -> +5V
- J8 pad 2: GND -> /Architecture/Interfaces - Actuators/ESC_TX_1
- J9 pad 2: /Architecture/Interfaces/LIDAR2_T_UART_TX -> /Architecture/Interfaces - Actuators/ESC_TX_2
- J9 pad 3: /Architecture/Interfaces/LIDAR2_T_UART_TX -> /Architecture/Interfaces - Actuators/PWM2
- JP3 pad 1: /Architecture/Interfaces/FDCAN_T_1_J -> /Architecture/Interfaces - Comms/FDCAN_T_1_J
- JP4 pad 1: /Architecture/Interfaces/FDCAN_T_2_J -> /Architecture/Interfaces - Comms/FDCAN_T_2_J
- JP5 pad 2: /Architecture/Interfaces/EXT_UART_PWR -> /Architecture/Interfaces - Comms/EXT_UART_PWR
- Q1 pad 2: Net-(Q1-G) -> /Architecture/Power Input/ID_GATE
- R10 pad 1: +5V -> /Architecture/Power Generation/MUX_PR2
- R10 pad 2: /Architecture/Power Generation/+5V_PRE_LED -> /Architecture/Power Generation/MUX_IN2
- R11 pad 1: /Architecture/Power Generation/LDO_FB -> GND
- R11 pad 2: +3V3 -> /Architecture/Power Generation/MUX_PR2
- R12 pad 1: +3V3 -> +BAT_PROT
- R12 pad 2: /Architecture/Power Generation/+3V3_PRE_LED -> /Architecture/Power Generation/BAT_PROT_PRE_LED
- R13 pad 1: GND -> +5V
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Routing:
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- added copper zone on B.Cu, net +3V3
- added copper zone on In3.Cu, net +3V3
- added copper zone on B.Cu, net +5V
- added copper zone on F.Cu, net +5V
- added copper zone on In3.Cu, net +5V
- added copper zone on B.Cu, net +5V_EXT
- added copper zone on F.Cu, net +5V_EXT
- added copper zone on B.Cu, net +BAT
- added copper zone on F.Cu, net +BAT
- added copper zone on In3.Cu, net +BAT
- added copper zone on B.Cu, net +BAT_PROT
- added copper zone on F.Cu, net +BAT_PROT
- added copper zone on In3.Cu, net +BAT_PROT
- added copper zone on B.Cu, net +BAT_PROT_PRE_MEAS
- added copper zone on F.Cu, net +BAT_PROT_PRE_MEAS
- added copper zone on In3.Cu, net +BAT_PROT_PRE_MEAS
- added copper zone on F.Cu, net /Architecture/Power Generation/BUCK_SW
- added copper zone on B.Cu, net GND
- added copper zone on F.Cu, net GND
- added copper zone on In1.Cu, net GND
- added copper zone on In3.Cu, net GND
- added copper zone on In4.Cu, net GND
Other:
- board size 100 x 50 mm -> 95 x 50 mm
- rule pad_to_mask_clearance: 0.1 -> 0.11
- board text added: "+BAT"
- board text added: "BUCKS ABOVE"
- board text added: "V1"

Commit message: bump
Parts:
- removed TP2, TP4: TestPoint, TestPoint:TestPoint_Pad_1.0x1.0mm
- added S2: ~, 0_misc:right_hand_rule_2, F.Cu at (157.9, 120.1)
- added TP20: TestPoint, TestPoint:TestPoint_Pad_1.0x1.0mm, F.Cu at (100.9, 90.9)
- added TP23: TestPoint, TestPoint:TestPoint_Pad_1.0x1.0mm, B.Cu at (165.4, 119.0)
- added TP24: TestPoint, TestPoint:TestPoint_Pad_1.0x1.0mm, B.Cu at (154.3, 122.3)
- added TP25: TestPoint, TestPoint:TestPoint_Pad_1.0x1.0mm, B.Cu at (165.0, 123.7)
- added TP26: TestPoint, TestPoint:TestPoint_Pad_1.0x1.0mm, B.Cu at (148.8, 122.0)
- added TP27: TestPoint, TestPoint:TestPoint_Pad_1.0x1.0mm, B.Cu at (161.9, 122.4)
- added TP28: TestPoint, TestPoint:TestPoint_Pad_1.0x1.0mm, B.Cu at (149.8, 120.0)
- added TP29: TestPoint, TestPoint:TestPoint_Pad_1.0x1.0mm, B.Cu at (152.4, 124.4)
- added TP30: TestPoint, TestPoint:TestPoint_Pad_1.0x1.0mm, B.Cu at (169.4, 127.4)
- added TP31: TestPoint, TestPoint:TestPoint_Pad_1.0x1.0mm, B.Cu at (157.4, 125.4)
- added TP32: TestPoint, TestPoint:TestPoint_Pad_1.0x1.0mm, B.Cu at (155.1, 119.6)
- added TP33: TestPoint, TestPoint:TestPoint_Pad_1.0x1.0mm, B.Cu at (149.9, 111.9)
- added TP34: TestPoint, TestPoint:TestPoint_Pad_1.0x1.0mm, B.Cu at (158.4, 120.4)
- added TP35: TestPoint, TestPoint:TestPoint_Pad_1.0x1.0mm, B.Cu at (160.9, 117.0)
- added TP36: TestPoint, TestPoint:TestPoint_Pad_1.0x1.0mm, B.Cu at (146.6, 118.4)
- added TP37: TestPoint, TestPoint:TestPoint_Pad_1.0x1.0mm, B.Cu at (143.2, 116.9)
- added TP38: TestPoint, TestPoint:TestPoint_Pad_1.0x1.0mm, B.Cu at (147.5, 85.4)
- added TP39: TestPoint, TestPoint:TestPoint_Pad_1.0x1.0mm, B.Cu at (141.1, 117.5)
- added TP40: TestPoint, TestPoint:TestPoint_Pad_1.0x1.0mm, B.Cu at (142.5, 119.6)
- added TP41: TestPoint, TestPoint:TestPoint_Pad_1.0x1.0mm, B.Cu at (141.2, 94.8)
- added TP42: TestPoint, TestPoint:TestPoint_Pad_1.0x1.0mm, B.Cu at (139.5, 122.1)
- added TP43: TestPoint, TestPoint:TestPoint_Pad_1.0x1.0mm, B.Cu at (150.0, 88.2)
- added TP44: TestPoint, TestPoint:TestPoint_Pad_1.0x1.0mm, F.Cu at (138.1, 87.1)
- added TP45: TestPoint, TestPoint:TestPoint_Pad_1.0x1.0mm, B.Cu at (138.3, 117.5)
- added TP46: TestPoint, TestPoint:TestPoint_Pad_1.0x1.0mm, B.Cu at (148.3, 89.9)
- added TP47: TestPoint, TestPoint:TestPoint_Pad_1.0x1.0mm, B.Cu at (131.8, 119.9)
- added TP48: TestPoint, TestPoint:TestPoint_Pad_1.0x1.0mm, B.Cu at (133.8, 119.9)
- added TP49: TestPoint, TestPoint:TestPoint_Pad_1.0x1.0mm, B.Cu at (147.4, 83.4)
- C39: value 470n -> 100n
- Q1: footprint 0_transistors:DFN-8 -> 0_transistors:Diodes_PowerDI3333-8
- R2: value 10m -> 5m; footprint Resistor_SMD:R_1206_3216Metric -> Resistor_SMD:R_2512_6332Metric
- R41: moved to B.Cu
- U3: value INA180 -> INA293A
- moved S1 9.25 mm to (170.7, 123.0)
- moved R2 2.15 mm to (102.9, 85.5)
- moved Q1 1.24 mm to (95.0, 95.0), turned to 90 degrees
- moved R15 0.81 mm to (104.4, 120.8)
- moved D2 0.80 mm to (101.6, 126.4)
- moved R12 0.80 mm to (104.5, 126.4)
- moved D4 0.80 mm to (101.6, 120.8)
- renumbered TP5 to TP21, TP6 to TP22, TP36 to TP50, TP37 to TP51, TP38 to TP52, TP39 to TP53, TP40 to TP54, TP41 to TP55, U24 to U23
Connections:
- U1 pad 132: /Architecture/MCU IO/CAM_EN -> unconnected-(U1C-PG15-Pad132)
Routing:
- net GND: track 196.0 -> 142.5 mm, vias 221 -> 249
- net /Architecture/MCU IO/IMU_ACC_CS: track 18.9 -> 29.7 mm, vias 0 -> 1
- net +BAT_PROT: track 60.4 -> 68.3 mm, vias 23 -> 19
- net +5V: track 211.6 -> 204.3 mm, vias 23 -> 28
- net /Architecture/MCU IO/SPI2_SCK: track 15.8 -> 23.0 mm
- net /Architecture/Power Generation/MUX_IN2: track 11.3 -> 14.4 mm, vias 2 -> 3
- net /Architecture/MCU IO/SD_CMD: track 17.9 -> 20.1 mm
- net /Architecture/MCU IO/MAG_INT: track 32.7 -> 34.2 mm
- net /Architecture/Interfaces - Sensors/LIDAR2_T_UART_TX: track 27.3 -> 28.4 mm
- net +3V3: track 120.5 -> 119.5 mm
- net /Architecture/Interfaces - Comms/SWCLK: track 33.9 -> 32.9 mm
- net +BAT_PROT_PRE_MEAS: track 10.9 -> 11.9 mm, vias 17 -> 14
- net /Architecture/MCU IO/SD_D0: track 33.5 -> 34.4 mm
- net /Architecture/MCU IO/SD_D1: track 33.3 -> 34.1 mm
- net /Architecture/Interfaces - Actuators/PWM2: track 58.1 -> 58.7 mm
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- added copper zone on In2.Cu, net GND
Other:
- outline, holes or cut-outs redrawn
- rule pad_to_mask_clearance: 0.11 -> 0.1
- board text added: "+"
- board text added: "+ H L -"
- board text added: "+ IO CK R -"
- board text added: "+ TX RX PPS EVT -"
- board text added: "-"
- board text added: "- +"
- board text added: "- - PWM4 PWM3 + +"
- board text added: "- - PWM6 PWM5 + +"
- board text added: "- PWM TX +"
- board text added: "- RX TX +"
- board text added: "- RX TX SYN PPS RRX RTX +"
- board text added: "- SIG"
- board text added: "1"
- board text added: "1_MISO"
- board text added: "1_MOSI"
- board text added: "1_SCK"
- board text added: "2"
- board text added: "3V3"
- board text added: "3V3 5V BAT"
- board text added: "4_MISO"
- board text added: "4_MOSI"
- board text added: "4_SCK"
- board text added: "5V"
- board text added: "868 MHz"
- board text added: "A_CS"
- board text added: "BARO"
- board text added: "BOOT"
- board text added: "BUCK"
- board text added: "BUTT"
- board text added: "B_CS"
- board text added: "CAN 1"
- board text added: "CAN 2"
- board text added: "CLK"
- board text added: "CMD"
- board text added: "CS"
- board text added: "D0"
- board text added: "D1"
- board text added: "D2"
- board text added: "D3"
- board text added: "ESC"
- board text added: "EXT. BAT"
- board text added: "FB"
- board text added: "GPS"
- board text added: "G_CS"
- board text added: "IMON"
- board text added: "IMU"
- board text added: "INT_A"
- board text added: "INT_G"
- board text added: "IO0"
- board text added: "IO1"
- board text added: "IO2"
- board text added: "IO3"
- board text added: "LIDAR"
- board text added: "MAG"
- board text added: "M_CS"
- board text added: "M_INT"
- board text added: "NRST"
- board text added: "RST"
- board text added: "RX"
- board text added: "R_RX"
- board text added: "R_TX"
- board text added: "SCL"
- board text added: "SDA"
- board text added: "TERM 1"
- board text added: "TERM 2"
- board text added: "TOAD V1"
- board text added: "TX"
- board text added: "VDDA"
- board text added: "VN"
- board text removed: "+BAT"
- board text removed: "BUCKS ABOVE"
- board text removed: "V1"

Commit message: bump
Parts:
- D13: value SMF18A -> SMF28CA; footprint Diode_SMD:D_SOD-123 -> PCM_JLCPCB:D_SOD-123FL
- moved D13 0.20 mm to (94.5, 106.8), turned to -90 degrees
Connections:
- D13 pad 1: /Architecture/Interfaces - Comms/EXT_BAT -> GND
- D13 pad 2: GND -> /Architecture/Interfaces - Comms/EXT_BAT
Routing:
- net /Architecture/Interfaces - Comms/EXT_BAT: track 9.43 -> 8.22 mm
