File: hoppen_fc/hoppen_fc.kicad_pcb (KiCad board)
At the start: 6 copper layers, 95 x 50 mm, 265 parts, among them J1 XT30 M, J10 B6B-PH, J11 B6B-PH, J12 BM04B-GHS1.25, J13 BM04B-GHS1.25, J14 BM02B-GHS1.25, J15 BM05B-GHS1.25, J16 BM02B-GHS1.25, J17 BM04B-GHS1.25, J18 U.FL, J2 USB_C_Receptacle_USB2.0_16P, J3 MicroSD Card Holder, J4 BM04B-GHS1.25, J5 BM04B-GHS1.25, J6 BM06B-GHS1.25, J7 BM08B-GHS1.25, J8 BM04B-GHS1.25, J9 BM04B-GHS1.25, Q1 NMOS, Q2 MMBT3904, SW1 SW_Push, SW2 SW_Push, SW3 SW_Push, U1 STM32H743ZITx, U10 MMC5983MA, U11 USBLC6-2SC6, U12 W25Q128JVS, U13 FM24C64B, U14 SP3223, U15 TJA1051TK-3, U16 TJA1051TK-3, U17 74AHCT1G125, U18 PD4E1U, U19 PD4E1U, U2 PD4E1U, U20 PD4E1U, U21 74AHCT1G125, U22 PD4E1U, U23 RFM95W-868S2, U3 INA293A, U4 LM74700, U5 AP64500, U6 TPS2121, U7 TPS74801DRC, U8 MS5607-02BA, U9 BMI088, Y1 25 MHz Crystal, Y2 32.768 kHz

Commit message: production v1
Parts:
- removed R10, R3: 100k, 0_resistor_smd:R_0402_1005Metric
- removed R11, R5: 33k, 0_resistor_smd:R_0402_1005Metric
- C39, R9, U6: moved to F.Cu
- R1: value 1k -> 10k
- moved C39 1.90 mm to (104.8, 105.0), turned to 90 degrees
- moved R9 1.90 mm to (104.8, 106.9), turned to 90 degrees
- moved C58 0.81 mm to (163.0, 86.4)
- moved U6 0.10 mm to (102.5, 105.9), turned to -90 degrees
Connections:
- U1 pad 58: unconnected-(U1C-PE7-Pad58) -> /Architecture/Interfaces - Actuators/ESC_TX_1
- U1 pad 59: /Architecture/Interfaces - Actuators/ESC_TX_1 -> unconnected-(U1C-PE8-Pad59)
- U6 pad 2: /Architecture/Power Generation/MUX_IN2 -> +5V_EXT
- U6 pad 3: /Architecture/Power Generation/MUX_PR2 -> GND
- U6 pad 6: /Architecture/Power Generation/MUX_PR1 -> GND
- U6 pad 7: +5V_EXT -> /Architecture/Power Generation/MUX_IN2
Routing:
- net /Architecture/Power Generation/MUX_IN2: track 14.4 -> 4.49 mm, vias 3 -> 0
- net +5V_EXT: track 10.6 -> 5.06 mm, vias 8 -> 11
- net GND: track 142.5 -> 139.5 mm, vias 249 -> 252
- net /Architecture/Power Generation/MUX_PR2: track 2.96 -> 0.00 mm
- net /Architecture/Power Generation/MUX_PR1: track 2.26 -> 0.00 mm
- net +5V: track 204.3 -> 202.9 mm
- net /Architecture/RS232/RS232_V_P: track 2.87 -> 3.71 mm
Other:
- board text added: "DESIGNED BY SVERRE"
- board text added: "MAX 6S"
- board text added: "MUX"
- board text removed: "EXT. BAT"
