File: hoppen_fc/interfaces_actuators.kicad_sch (KiCad schematic)
At the start: 20 parts, among them J10 PH2.0-3P, J11 PH2.0-3P, J8 GH1.25-4P, J9 GH1.25-4P

Commit message: bump
Parts:
- removed C86, C89, C92, C95: 100n, 0_capacitor_smd:C_0402_1005Metric, symbol Device:C
- removed C87, C88, C90, C91, C93, C94, C96, C97: 10u, 0_capacitor_smd:C_0805_2012Metric, symbol Device:C
- removed J10, J11: PH2.0-3P, 0_connectors:S3B-PH-SM4-TB-LF-SN, symbol 0_connectors:Conn_01x03_Mounting
- removed R46, R47: 47k, 0_resistor_smd:R_0402_1005Metric, symbol Device:R
- added C73, C74, C75, C76, C77, C78, C79, C80, C81, C82: 10u, 0_capacitor_smd:C_0805_2012Metric, symbol Device:C
- added J10, J11: B6B-PH, Connector_JST:JST_PH_B6B-PH-K_1x06_P2.00mm_Vertical, symbol 0_connectors:Conn_01x06
- added R49, R50, R51, R52: 47k, 0_resistor_smd:R_0402_1005Metric, symbol Device:R
- added U19, U20: PD4E1U, 0_transistors:SOT-363_SC-70-6, symbol 0_diodes:PD4E1U
- J8, J9: value GH1.25-4P -> BM04B-GHS1.25; footprint 0_connectors:SM04B-GHS-TB-LF-SN -> 0_connectors:BM04B-GHS1.25; LCSC C189895 -> C161692
- renumbered R44 to R47, R45 to R48
Connections:
- net +BAT_PROT: now also C75.1, C76.1, C77.1, C78.1, C79.1, C80.1, C81.1, C82.1, J10.1 (Pin_1), J10.2 (Pin_2), J11.1 (Pin_1), J11.2 (Pin_2); no longer J8.1 (Pin_1), J9.1 (Pin_1)
- net ESC_TX_1: now also U19.3 (D2+)
- net ESC_TX_2: now also U19.4 (D2-)
- net GND: now also C73.2, C74.2, C75.2, C76.2, C77.2, C78.2, C79.2, C80.2, C81.2, C82.2, J10.5 (Pin_5), J10.6 (Pin_6), J11.5 (Pin_5), J11.6 (Pin_6), R49.2, R50.2, R51.2, R52.2, U19.2 (GND), U20.2 (GND)
- net PWM1: now also U19.1 (D1+)
- net PWM2: now also U19.6 (D1-)
- net PWM3: now also J10.3 (Pin_3), R49.1, U20.4 (D2-)
- net PWM4: now also J10.4 (Pin_4), R50.1, U20.6 (D1-)
- new net +5V: C73.1, C74.1, J8.1 (Pin_1), J9.1 (Pin_1)
- new net PWM5: J11.3 (Pin_3), R51.1, U20.3 (D2+)
- new net PWM6: J11.4 (Pin_4), R52.1, U20.1 (D1+)
- no-connect marks 0 -> 2
Other:
- note added: "ESD PROTECTION"
- note added: "SERVO #1 & #2"
- note added: "SERVO #3 & #4"
- note removed: "SERVO #1"
- note removed: "SERVO #2"
