File: hoppen_fc/interfaces_sensors.kicad_sch (KiCad schematic)
At the start: 20 parts, among them J4 GH1.25-4P, J5 GH1.25-4P, J6 Conn_01x06_Shield_Mounting, J7 GH1.25-8P, U19 PD4E1U, U20 PD4E1U, U21 PD4E1U, U22 PD4E1U

Commit message: bump
Parts:
- removed C82, C83, C84, C85: 4u7, 0_capacitor_smd:C_0603_1608Metric, symbol Device:C
- removed U19, U20, U21: PD4E1U, 0_transistors:SOT-363_SC-70-6, symbol 0_diodes:PD4E1U
- added C69, C70, C71, C72: 22u, 0_capacitor_smd:C_0805_2012Metric, symbol Device:C
- J4, J5: value GH1.25-4P -> BM04B-GHS1.25; footprint 0_connectors:SM04B-GHS-TB-LF-SN -> 0_connectors:BM04B-GHS1.25; LCSC C189895 -> C161692
- J6: value Conn_01x06_Shield_Mounting -> BM06B-GHS1.25; footprint (none) -> 0_connectors:BM06B-GHS-1.25; LCSC (none) -> C225122
- J7: value GH1.25-8P -> BM08B-GHS1.25; footprint 0_connectors:SM08B-GHS-TB-LF-SN -> 0_connectors:BM08B-GHS1.25; LCSC C265111 -> C133062
- R39: renamed from R36; LCSC C25092 -> C2929994
- R40: renamed from R37; LCSC C25092 -> C2929994
- R41: renamed from R38; LCSC C25092 -> C2929994
- R42: renamed from R39; LCSC C25092 -> C2929994
- R43: renamed from R40; LCSC C25092 -> C2929994
- R44: renamed from R41; LCSC C25092 -> C2929994
- R45: renamed from R42; LCSC C25092 -> C2929994
- R46: renamed from R43; LCSC C25092 -> C2929994
- renumbered U22 to U18
Connections:
- net +5V: now also C69.1, C70.1, C71.1, C72.1
- net GND: now also C69.2, C70.2, C71.2, C72.2
- net VN_UART_RX_T: now also U18.3 (D2+); no longer U18.4 (D2-)
- net VN_UART_TX_T: now also U18.4 (D2-); no longer U18.3 (D2+)
- net RTK_UART_TX_T: now reaches J6.2 (Pin_2), R43.1
- net RTK_UART_RX_T: now reaches J6.3 (Pin_3), R44.1
- no-connect marks 8 -> 1
Other:
- note added: "LIDAR INTERFACE #2"
