File: hoppen_fc/mcu_power.kicad_sch (KiCad schematic)
At the start: 21 parts, among them U1 STM32H743ZITx

Commit message: finished routing, starting doublechecking and componenting
Parts:
- L1: footprint (none) -> Inductor_SMD:L_0603_1608Metric; LCSC (none) -> C1002
Changed lines of the file:
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@@
 			)
 		)
-		(property "Footprint" ""
+		(property "Footprint" "Inductor_SMD:L_0603_1608Metric"
 			(at 123.19 102.87 0)
 			(effects
@@
 			(effects
 				(font
+					(size 1.27 1.27)
+				)
+				(hide yes)
+			)
+		)
+		(property "LCSC" "C1002"
+			(at 123.19 102.87 90)
+			(effects
+				(font

Commit message: finished adding lcsc numbers
Parts:
- C1: renamed from C18; LCSC (none) -> C23630
- C10: renamed from C9; LCSC (none) -> C307331
- C11: renamed from C10; LCSC (none) -> C307331
- C12: renamed from C11; LCSC (none) -> C307331
- C13: renamed from C14; LCSC (none) -> C307331
- C14: renamed from C17; LCSC (none) -> C307331
- C15: renamed from C12; LCSC (none) -> C15849
- C16: renamed from C15; LCSC (none) -> C307331
- C17: renamed from C8; LCSC (none) -> C15849
- C18: renamed from C13; LCSC (none) -> C15849
- C19: renamed from C16; LCSC (none) -> C307331
- C2: renamed from C19; LCSC (none) -> C23630
- C3: renamed from C1; LCSC (none) -> C19666
- C4: renamed from C2; LCSC (none) -> C307331
- C5: renamed from C3; LCSC (none) -> C307331
- C6: renamed from C4; LCSC (none) -> C307331
- C7: renamed from C5; LCSC (none) -> C307331
- C8: renamed from C6; LCSC (none) -> C307331
- C9: renamed from C7; LCSC (none) -> C307331

Commit message: bump
Parts:
- removed C15: 1u, 0_capacitor_smd:C_0603_1608Metric, symbol Device:C
- added C21: 1u, 0_capacitor_smd:C_0402_1005Metric, symbol Device:C
- added C4, C5, C6: 100n, 0_capacitor_smd:C_0402_1005Metric, symbol Device:C
- added TP1: TestPoint, TestPoint:TestPoint_Pad_1.0x1.0mm, symbol Connector:TestPoint
- C18: footprint 0_capacitor_smd:C_0603_1608Metric -> 0_capacitor_smd:C_0402_1005Metric; LCSC C15849 -> C52923
- C20: renamed from C17; footprint 0_capacitor_smd:C_0603_1608Metric -> 0_capacitor_smd:C_0402_1005Metric; LCSC C15849 -> C52923
- C3: value 4u7 -> 10u; footprint 0_capacitor_smd:C_0603_1608Metric -> 0_capacitor_smd:C_0805_2012Metric; LCSC C19666 -> C440198
- renumbered C7 to C10, C8 to C11, C9 to C12, C10 to C13, C11 to C14, C12 to C15, C13 to C16, C14 to C17, C16 to C19, C19 to C22, C4 to C7, C5 to C8, C6 to C9
Connections:
- net +3V3: now also C4.1, C5.1, C6.1
- net GND: now also C21.2, C4.2, C5.2, C6.2
- net MCU_VDDA: now also C21.1, TP1.1
Other:
- moved on the sheet: C1, C10, C11, C12, C13, C14, C15, C16, C17, C19, C2, C20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

Commit message: bump
Changed lines of the file:
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@@
-	(wire
-		(pts
-			(xy 161.29 127) (xy 154.94 127)
-		)
-		(stroke
-			(width 0)
-			(type default)
-		)
-	)
 	(wire
 		(pts
@@
 	(symbol
 		(lib_id "power:GND")
-		(at 154.94 127 0)
+		(at 161.29 127 0)
 		(unit 1)
 		(exclude_from_sim no)
@@
 		(fields_autoplaced yes)
 		(property "Reference" "#PWR012"
-			(at 154.94 133.35 0)
+			(at 161.29 133.35 0)
 			(effects
 				(font
@@
 		)
 		(property "Value" "GND"
-			(at 154.94 132.08 0)
+			(at 161.29 132.08 0)
 			(effects
 				(font
@@
 		)
 		(property "Footprint" ""
-			(at 154.94 127 0)
+			(at 161.29 127 0)
 			(effects
 				(font
@@
 		)
 		(property "Datasheet" ""
-			(at 154.94 127 0)
+			(at 161.29 127 0)
 			(effects
 				(font
@@
 		)
 		(property "Description" "Power symbol creates a global label with name \"GND\" , ground"
-			(at 154.94 127 0)
-			(effects
-				(font
+			(at 161.29 127 0)
+			(effects
+				(font
