File: hoppen_fc/power_input.kicad_sch (KiCad schematic)
At the start: 12 parts, among them J1 XT30 M, Q1 NMOS, U3 INA180, U4 LM74700

Commit message: bump
Parts:
- removed TP2: TestPoint, TestPoint:TestPoint_Pad_1.0x1.0mm, symbol Connector:TestPoint
- removed U3: INA180, 0_transceivers:SOT-23-5, symbol 0_power:INA180
- added U3: INA293A, 0_transceivers:SOT-23-5, symbol 0_power:INA293
- Q1: footprint 0_transistors:DFN-8 -> 0_transistors:Diodes_PowerDI3333-8
- R2: value 10m -> 5m; footprint Resistor_SMD:R_1206_3216Metric -> Resistor_SMD:R_2512_6332Metric; LCSC C105362 -> C185817
- U4: LCSC C2941042 -> C2802568
- renumbered TP3 to TP20
Connections:
- net +3V3: now also U3.5 (VS)
- net +BAT_IMON: now also U3.1 (OUT)
- net +BAT_PROT: now also U3.4 (IN-)
- net +BAT_PROT_PRE_MEAS: now also U3.3 (IN+)
- net GND: now also U3.2 (GND)
Changed lines of the file:
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@@
 		)
 	)
-	(text_box "DESIGN:\nVds 60V\nVgs 20V\nRds@10V 2.8mohm\nId 80A"
+	(text_box "DESIGN:\nVds 60V\nVgs 20V\nRds@4.5V 8.5mohm\nId 80A"
 		(exclude_from_sim no)
 		(at 158.75 53.34 0)
@@
 	)
 	(junction
-		(at 205.74 67.31)
-		(diameter 0)
-		(color 0 0 0 0)
-	)
-	(junction
 		(at 177.8 67.31)
 		(diameter 0)
@@
 	(wire
 		(pts
-			(xy 205.74 67.31) (xy 212.09 67.31)
+			(xy 195.58 67.31) (xy 212.09 67.31)
 		)
 		(stroke
@@
 		(pts
 			(xy 207.01 90.17) (xy 214.63 90.17)
-		)
-		(stroke
-			(width 0)
-			(type default)
-		)
-	)
-	(wire
-		(pts
-			(xy 195.58 67.31) (xy 205.74 67.31)
 		)
 		(stroke
@@
 	)
 	(symbol
-		(lib_id "Connector:TestPoint")
-		(at 205.74 67.31 0)
-		(unit 1)
-		(exclude_from_sim no)
-		(in_bom yes)
-		(on_board yes)
-		(dnp no)
-		(fields_autoplaced yes)
-		(property "Reference" "TP2"
-			(at 208.28 62.7379 0)
-			(effects
-				(font
-					(size 1.27 1.27)
-				)
-				(justify left)
-			)
-		)
-		(property "Value" "TestPoint"
-			(at 208.28 65.2779 0)
-			(effects
-				(font
-					(size 1.27 1.27)
-				)
-				(justify left)
-				(hide yes)
-			)
-		)
-		(property "Footprint" "TestPoint:TestPoint_Pad_1.0x1.0mm"
-			(at 210.82 67.31 0)
-			(effects
-				(font
-					(size 1.27 1.27)
-				)
-				(hide yes)
-			)
-		)
-		(property "Datasheet" "~"
-			(at 210.82 67.31 0)
-			(effects
-				(font
-					(size 1.27 1.27)
-				)
-				(hide yes)
-			)
-		)
-		(property "Description" "test point"
-			(at 205.74 67.31 0)
-			(effects
-				(font
-					(size 1.27 1.27)
-				)
-				(hide yes)
-			)
-		)
-		(pin "1"
-		)
-		(instances
-			(project "hoppen_fc"
-				(path "/abe950a1-9eef-4508-9fd4-31d3e723e029/c85454e5-a89e-41eb-a5ed-71b4fc4cf13a/45aa82bb-5d0c-4be2-bfbe-f6adc776653e"
-					(reference "TP2")
-					(unit 1)
-				)
-			)
-		)
-	)
-	(symbol
 		(lib_id "power:+3.3V")
 		(at 250.19 64.77 0)
@@
 	)
 	(symbol
-		(lib_id "0_power:INA180")
+		(lib_id "Device:D_TVS")
+		(at 82.55 77.47 90)
+		(unit 1)
+		(exclude_from_sim no)
+		(in_bom yes)
+		(on_board yes)
+		(dnp no)
+		(fields_autoplaced yes)
+		(property "Reference" "D1"
+			(at 85.09 76.1999 90)
+			(effects
+				(font
+					(size 1.27 1.27)
+				)
+				(justify right)
+			)
+		)
+		(property "Value" "SMBJ28CA"
+			(at 85.09 78.7399 90)
+			(effects
+				(font
+					(size 1.27 1.27)
+				)
+				(justify right)
+			)
+		)
+		(property "Footprint" "Diode_SMD:D_SMB"
+			(at 82.55 77.47 0)
+			(effects
+				(font
+					(size 1.27 1.27)
+				)
+				(hide yes)
+			)
+		)
+		(property "Datasheet" "~"
+			(at 82.55 77.47 0)
+			(effects
+				(font
+					(size 1.27 1.27)
+				)
+				(hide yes)
+			)
+		)
+		(property "Description" "Bidirectional transient-voltage-suppression diode"
+			(at 82.55 77.47 0)
+			(effects
+				(font
+					(size 1.27 1.27)
+				)
+				(hide yes)
+			)
+		)
+		(property "LCSC" "C19077583"
+			(at 82.55 77.47 90)
+			(effects
+				(font
+					(size 1.27 1.27)
+				)
+				(hide yes)
+			)
+		)
+		(pin "2"
+		)
+		(pin "1"
+		)
+		(instances
+			(project ""
+				(path "/abe950a1-9eef-4508-9fd4-31d3e723e029/c85454e5-a89e-41eb-a5ed-71b4fc4cf13a/45aa82bb-5d0c-4be2-bfbe-f6adc776653e"
+					(reference "D1")
+					(unit 1)
+				)
+			)
+		)
+	)
+	(symbol
+		(lib_id "0_power:INA293")
 		(at 224.79 87.63 0)
 		(unit 1)
@@
 			)
 		)
-		(property "Value" "INA180"
+		(property "Value" "INA293A"
 			(at 224.79 77.47 0)
 			(effects
@@
 			)
 		)
-		(property "Datasheet" "https://www.ti.com/lit/ds/symlink/ina180.pdf?ts=1767065031120"
+		(property "Datasheet" "https://www.ti.com/lit/ds/symlink/ina293.pdf?ts=1774067049648"
 			(at 224.79 59.182 0)
 			(effects
@@
 			)
 		)
-		(property "Description" "26V, 350kHz current sense amplifier"
+		(property "Description" "INA293 –4 V to 110 V, 1.3-MHz, Ultra-Precise Current Sense Amplifier"
 			(at 224.79 62.738 0)
 			(effects
@@
 			)
 		)
-		(property "LCSC" "C122228"
+		(property "LCSC" "C1855790"
 			(at 224.79 57.15 0)
 			(effects
@@
 			)
 		)
+		(pin "1"
+		)
+		(pin "5"
+		)
+		(pin "2"
+		)
 		(pin "3"
 		)
 		(pin "4"
-		)
-		(pin "2"
-		)
-		(pin "5"
-		)
-		(pin "1"
 		)
 		(instances
@@
 				(path "/abe950a1-9eef-4508-9fd4-31d3e723e029/c85454e5-a89e-41eb-a5ed-71b4fc4cf13a/45aa82bb-5d0c-4be2-bfbe-f6adc776653e"
 					(reference "U3")
-					(unit 1)
-				)
-			)
-		)
-	)
-	(symbol
-		(lib_id "Device:D_TVS")
-		(at 82.55 77.47 90)
-		(unit 1)
-		(exclude_from_sim no)
-		(in_bom yes)
-		(on_board yes)
-		(dnp no)
-		(fields_autoplaced yes)
-		(property "Reference" "D1"
-			(at 85.09 76.1999 90)
-			(effects
-				(font
-					(size 1.27 1.27)
-				)
-				(justify right)
-			)
-		)
-		(property "Value" "SMBJ28CA"
-			(at 85.09 78.7399 90)
-			(effects
-				(font
-					(size 1.27 1.27)
-				)
-				(justify right)
-			)
-		)
-		(property "Footprint" "Diode_SMD:D_SMB"
-			(at 82.55 77.47 0)
-			(effects
-				(font
-					(size 1.27 1.27)
-				)
-				(hide yes)
-			)
-		)
-		(property "Datasheet" "~"
-			(at 82.55 77.47 0)
-			(effects
-				(font
-					(size 1.27 1.27)
-				)
-				(hide yes)
-			)
-		)
-		(property "Description" "Bidirectional transient-voltage-suppression diode"
-			(at 82.55 77.47 0)
-			(effects
-				(font
-					(size 1.27 1.27)
-				)
-				(hide yes)
-			)
-		)
-		(property "LCSC" "C19077583"
-			(at 82.55 77.47 90)
-			(effects
-				(font
-					(size 1.27 1.27)
-				)
-				(hide yes)
-			)
-		)
-		(pin "2"
-		)
-		(pin "1"
-		)
-		(instances
-			(project ""
-				(path "/abe950a1-9eef-4508-9fd4-31d3e723e029/c85454e5-a89e-41eb-a5ed-71b4fc4cf13a/45aa82bb-5d0c-4be2-bfbe-f6adc776653e"
-					(reference "D1")
 					(unit 1)
 				)
@@
 			)
 		)
-		(property "LCSC" "C2941042"
+		(property "LCSC" "C2802568"
 			(at 151.13 54.356 0)
 			(effects
@@
 			)
 		)
-		(property "Footprint" "0_transistors:DFN-8"
+		(property "Footprint" "0_transistors:Diodes_PowerDI3333-8"
 			(at 153.67 64.77 0)
 			(effects
@@
 			)
 		)
-		(property "Value" "10m"
+		(property "Value" "5m"
 			(at 224.79 63.5 90)
 			(effects
@@
 			)
 		)
-		(property "Footprint" "Resistor_SMD:R_1206_3216Metric"
+		(property "Footprint" "Resistor_SMD:R_2512_6332Metric"
 			(at 224.79 69.088 90)
 			(effects
@@
 			)
 		)
-		(property "LCSC" "C105362"
+		(property "LCSC" "C185817"
 			(at 224.79 67.31 90)
 			(effects
@@
 		(dnp no)
 		(fields_autoplaced yes)
-		(property "Reference" "TP3"
+		(property "Reference" "TP20"
 			(at 252.73 85.5979 0)
 			(effects
@@
 			(project "hoppen_fc"
 				(path "/abe950a1-9eef-4508-9fd4-31d3e723e029/c85454e5-a89e-41eb-a5ed-71b4fc4cf13a/45aa82bb-5d0c-4be2-bfbe-f6adc776653e"
-					(reference "TP3")
+					(reference "TP20")
 					(unit 1)
 				)

Commit message: bump
Parts:
- Q1: LCSC C467174 -> C2802568
- U4: LCSC C2802568 -> C2941042
Changed lines of the file:
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@@
 		)
 		(instances
-			(project ""
+			(project "hoppen_fc"
 				(path "/abe950a1-9eef-4508-9fd4-31d3e723e029/c85454e5-a89e-41eb-a5ed-71b4fc4cf13a/45aa82bb-5d0c-4be2-bfbe-f6adc776653e"
 					(reference "D1")
@@
 		)
 		(instances
-			(project ""
+			(project "hoppen_fc"
 				(path "/abe950a1-9eef-4508-9fd4-31d3e723e029/c85454e5-a89e-41eb-a5ed-71b4fc4cf13a/45aa82bb-5d0c-4be2-bfbe-f6adc776653e"
 					(reference "U3")
@@
 			)
 		)
-		(property "LCSC" "C2802568"
+		(property "LCSC" "C2941042"
 			(at 151.13 54.356 0)
 			(effects
@@
 		)
 		(instances
-			(project ""
+			(project "hoppen_fc"
 				(path "/abe950a1-9eef-4508-9fd4-31d3e723e029/c85454e5-a89e-41eb-a5ed-71b4fc4cf13a/45aa82bb-5d0c-4be2-bfbe-f6adc776653e"
 					(reference "U4")
@@
 		)
 		(instances
-			(project ""
+			(project "hoppen_fc"
 				(path "/abe950a1-9eef-4508-9fd4-31d3e723e029/c85454e5-a89e-41eb-a5ed-71b4fc4cf13a/45aa82bb-5d0c-4be2-bfbe-f6adc776653e"
 					(reference "J1")
@@
 		)
 		(instances
-			(project ""
+			(project "hoppen_fc"
 				(path "/abe950a1-9eef-4508-9fd4-31d3e723e029/c85454e5-a89e-41eb-a5ed-71b4fc4cf13a/45aa82bb-5d0c-4be2-bfbe-f6adc776653e"
 					(reference "#PWR031")
@@
 			)
 		)
-		(property "LCSC" "C467174"
+		(property "LCSC" "C2802568"
 			(at 151.13 69.85 90)
 			(effects
@@
 		)
 		(instances
-			(project ""
+			(project "hoppen_fc"
 				(path "/abe950a1-9eef-4508-9fd4-31d3e723e029/c85454e5-a89e-41eb-a5ed-71b4fc4cf13a/45aa82bb-5d0c-4be2-bfbe-f6adc776653e"
 					(reference "Q1")
@@
 		)
 		(instances
-			(project ""
+			(project "hoppen_fc"
 				(path "/abe950a1-9eef-4508-9fd4-31d3e723e029/c85454e5-a89e-41eb-a5ed-71b4fc4cf13a/45aa82bb-5d0c-4be2-bfbe-f6adc776653e"
 					(reference "R2")
