File: hoppen_fc/radio.kicad_sch (KiCad schematic)
At the start: 1 part, among them U18 RFM95W-868S2

Commit message: sync
Parts:
- added C98: 100n, 0_capacitor_smd:C_0402_1005Metric, symbol Device:C
- added J19: U.FL, Connector_Coaxial:U.FL_Hirose_U.FL-R-SMT-1_Vertical, symbol Connector:Conn_Coaxial
Connections:
- net GND: now reaches U18.1 (GND)
- net GND: now also U18.10 (GND), U18.8 (GND), C98.2, J19.2 (Ext)
- net +3V3: now reaches U18.13 (3.3V)
- net +3V3: now also C98.1
- net RADIO_DIO0: now reaches U18.14 (DIO0)
- net RADIO_DIO1: now reaches U18.15 (DIO1)
- net SPI3_MISO: now reaches U18.2 (MISO)
- net SPI3_MOSI: now reaches U18.3 (MOSI)
- net SPI3_SCK: now reaches U18.4 (SCK)
- net RADIO_CS: now reaches U18.5 (NSS)
- net RADIO_RST: now reaches U18.6 (RESET)
- net RADIO_DIO5: now reaches U18.7 (DIO5)
- net RFM_ANT: now reaches U18.9 (ANT)
- net RFM_ANT: now also J19.1 (In)
- no-connect marks 0 -> 3
Other:
- title: (none) -> LoRa
- moved on the sheet: U18

Commit message: comments
Other:
- note added: "REMOVE?"
Changed lines of the file:
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@@
+		)
+	)
+	(text "REMOVE?"
+		(exclude_from_sim no)
+		(at 94.488 43.942 0)
+		(effects
+			(font
+				(face "KiCad Font")
+				(size 2.54 2.54)
+				(thickness 0.508)
+				(bold yes)
+				(color 255 0 0 1)
+			)
 		)
 	)

Commit message: bump
Parts:
- renumbered C98 to C104
Changed lines of the file:
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@@
 		(dnp no)
 		(fields_autoplaced yes)
-		(property "Reference" "#PWR0211"
+		(property "Reference" "#PWR0206"
 			(at 191.77 105.41 0)
 			(effects
@@
 			(project "hoppen_fc"
 				(path "/abe950a1-9eef-4508-9fd4-31d3e723e029/c85454e5-a89e-41eb-a5ed-71b4fc4cf13a/497505dd-337e-4de8-b212-9653d17f2ba6"
-					(reference "#PWR0211")
+					(reference "#PWR0206")
 					(unit 1)
 				)
@@
 		(dnp no)
 		(fields_autoplaced yes)
-		(property "Reference" "#PWR0210"
+		(property "Reference" "#PWR0204"
 			(at 134.62 68.58 0)
 			(effects
@@
 			(project "hoppen_fc"
 				(path "/abe950a1-9eef-4508-9fd4-31d3e723e029/c85454e5-a89e-41eb-a5ed-71b4fc4cf13a/497505dd-337e-4de8-b212-9653d17f2ba6"
-					(reference "#PWR0210")
+					(reference "#PWR0204")
 					(unit 1)
 				)
@@
 		(dnp no)
 		(fields_autoplaced yes)
-		(property "Reference" "#PWR0208"
+		(property "Reference" "#PWR0205"
 			(at 140.97 83.82 0)
 			(effects
@@
 			(project "hoppen_fc"
 				(path "/abe950a1-9eef-4508-9fd4-31d3e723e029/c85454e5-a89e-41eb-a5ed-71b4fc4cf13a/497505dd-337e-4de8-b212-9653d17f2ba6"
-					(reference "#PWR0208")
+					(reference "#PWR0205")
 					(unit 1)
 				)
@@
 		(dnp no)
 		(fields_autoplaced yes)
-		(property "Reference" "#PWR0209"
+		(property "Reference" "#PWR0207"
 			(at 132.08 125.73 0)
 			(effects
@@
 			(project "hoppen_fc"
 				(path "/abe950a1-9eef-4508-9fd4-31d3e723e029/c85454e5-a89e-41eb-a5ed-71b4fc4cf13a/497505dd-337e-4de8-b212-9653d17f2ba6"
-					(reference "#PWR0209")
+					(reference "#PWR0207")
 					(unit 1)
 				)
@@
 		(dnp no)
 		(fields_autoplaced yes)
-		(property "Reference" "C98"
+		(property "Reference" "C104"
 			(at 144.78 69.8499 0)
 			(effects
@@
 			(project ""
 				(path "/abe950a1-9eef-4508-9fd4-31d3e723e029/c85454e5-a89e-41eb-a5ed-71b4fc4cf13a/497505dd-337e-4de8-b212-9653d17f2ba6"
-					(reference "C98")
-					(unit 1)
-				)
+					(reference "C104")
+					(unit 1)
+				)

Commit message: bump
Parts:
- removed C104: 100n, 0_capacitor_smd:C_0402_1005Metric, symbol Device:C
- added C87: 22u, 0_capacitor_smd:C_0805_2012Metric, symbol Device:C
- U23: renamed from U18; now left out of the parts list
- renumbered J19 to J18
Connections:
- net +3V3: now also C87.1
- net GND: now also C87.2
- net RADIO_DIO2: now reaches U23.16 (DIO2)
- net RADIO_DIO5: no longer names the net of U23.7 (DIO5)
- net SPI3_MISO renamed SPI2_MISO
- net SPI3_MOSI renamed SPI2_MOSI
- net SPI3_SCK renamed SPI2_SCK
Other:
- note removed: "REMOVE?"
Changed lines of the file:
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@@
-		)
-	)
-	(text "REMOVE?"
-		(exclude_from_sim no)
-		(at 94.488 43.942 0)
-		(effects
-			(font
-				(face "KiCad Font")
-				(size 2.54 2.54)
-				(thickness 0.508)
-				(bold yes)
-				(color 255 0 0 1)
-			)
 		)
 	)
@@
 	)
 	(no_connect
-		(at 147.32 104.14)
+		(at 147.32 96.52)
 	)
 	(no_connect
@@
 	(wire
 		(pts
+			(xy 147.32 104.14) (xy 161.29 104.14)
+		)
+		(stroke
+			(width 0)
+			(type default)
+		)
+	)
+	(wire
+		(pts
 			(xy 134.62 114.3) (xy 134.62 116.84)
-		)
-		(stroke
-			(width 0)
-			(type default)
-		)
-	)
-	(wire
-		(pts
-			(xy 147.32 96.52) (xy 161.29 96.52)
 		)
 		(stroke
@@
 		)
 	)
-	(label "RADIO_CS"
-		(at 120.65 99.06 180)
+	(label "SPI2_MISO"
+		(at 120.65 96.52 180)
 		(effects
 			(font
@@
 		)
 	)
-	(label "SPI3_MISO"
-		(at 120.65 96.52 180)
+	(label "SPI2_MOSI"
+		(at 120.65 93.98 180)
 		(effects
 			(font
@@
 		)
 	)
-	(label "SPI3_MOSI"
-		(at 120.65 93.98 180)
+	(label "SPI2_SCK"
+		(at 120.65 91.44 180)
 		(effects
 			(font
@@
 		)
 	)
-	(label "SPI3_SCK"
-		(at 120.65 91.44 180)
-		(effects
-			(font
-				(size 1.27 1.27)
-			)
-			(justify right bottom)
-		)
-	)
-	(hierarchical_label "{SPI3}"
+	(hierarchical_label "RADIO_DIO2"
+		(shape bidirectional)
+		(at 161.29 104.14 0)
+		(effects
+			(font
+				(size 1.27 1.27)
+			)
+			(justify left)
+		)
+	)
+	(hierarchical_label "{SPI2}"
 		(shape bidirectional)
 		(at 102.87 87.63 180)
@@
 			)
 			(justify right)
-		)
-	)
-	(hierarchical_label "RADIO_DIO5"
-		(shape bidirectional)
-		(at 161.29 96.52 0)
-		(effects
-			(font
-				(size 1.27 1.27)
-			)
-			(justify left)
 		)
 	)
@@
 		(unit 1)
 		(exclude_from_sim no)
-		(in_bom yes)
+		(in_bom no)
 		(on_board yes)
 		(dnp no)
 		(fields_autoplaced yes)
-		(property "Reference" "U18"
+		(property "Reference" "U23"
 			(at 136.7633 83.82 0)
 			(effects
@@
 			(project ""
 				(path "/abe950a1-9eef-4508-9fd4-31d3e723e029/c85454e5-a89e-41eb-a5ed-71b4fc4cf13a/497505dd-337e-4de8-b212-9653d17f2ba6"
-					(reference "U18")
+					(reference "U23")
 					(unit 1)
 				)
@@
 		(dnp no)
 		(fields_autoplaced yes)
-		(property "Reference" "#PWR0206"
+		(property "Reference" "#PWR0207"
 			(at 191.77 105.41 0)
 			(effects
@@
 			(project "hoppen_fc"
 				(path "/abe950a1-9eef-4508-9fd4-31d3e723e029/c85454e5-a89e-41eb-a5ed-71b4fc4cf13a/497505dd-337e-4de8-b212-9653d17f2ba6"
-					(reference "#PWR0206")
+					(reference "#PWR0207")
 					(unit 1)
 				)
@@
 		(dnp no)
 		(fields_autoplaced yes)
-		(property "Reference" "J19"
+		(property "Reference" "J18"
 			(at 195.58 90.4631 0)
 			(effects
@@
 			(project ""
 				(path "/abe950a1-9eef-4508-9fd4-31d3e723e029/c85454e5-a89e-41eb-a5ed-71b4fc4cf13a/497505dd-337e-4de8-b212-9653d17f2ba6"
-					(reference "J19")
+					(reference "J18")
 					(unit 1)
 				)
@@
 		(dnp no)
 		(fields_autoplaced yes)
-		(property "Reference" "#PWR0204"
+		(property "Reference" "#PWR0205"
 			(at 134.62 68.58 0)
 			(effects
@@
 			(project "hoppen_fc"
 				(path "/abe950a1-9eef-4508-9fd4-31d3e723e029/c85454e5-a89e-41eb-a5ed-71b4fc4cf13a/497505dd-337e-4de8-b212-9653d17f2ba6"
-					(reference "#PWR0204")
+					(reference "#PWR0205")
 					(unit 1)
 				)
@@
 		(dnp no)
 		(fields_autoplaced yes)
-		(property "Reference" "#PWR0205"
+		(property "Reference" "#PWR0206"
 			(at 140.97 83.82 0)
 			(effects
@@
 			(project "hoppen_fc"
 				(path "/abe950a1-9eef-4508-9fd4-31d3e723e029/c85454e5-a89e-41eb-a5ed-71b4fc4cf13a/497505dd-337e-4de8-b212-9653d17f2ba6"
-					(reference "#PWR0205")
+					(reference "#PWR0206")
 					(unit 1)
 				)
@@
 		(dnp no)
 		(fields_autoplaced yes)
-		(property "Reference" "#PWR0207"
+		(property "Reference" "#PWR0208"
 			(at 132.08 125.73 0)
 			(effects
@@
 			(project "hoppen_fc"
 				(path "/abe950a1-9eef-4508-9fd4-31d3e723e029/c85454e5-a89e-41eb-a5ed-71b4fc4cf13a/497505dd-337e-4de8-b212-9653d17f2ba6"
-					(reference "#PWR0207")
+					(reference "#PWR0208")
 					(unit 1)
 				)
@@
 		(dnp no)
 		(fields_autoplaced yes)
-		(property "Reference" "C104"
+		(property "Reference" "C87"
 			(at 144.78 69.8499 0)
 			(effects
@@
 			)
 		)
-		(property "Value" "100n"
+		(property "Value" "22u"
 			(at 144.78 72.3899 0)
 			(effects
@@
 			)
 		)
-		(property "Footprint" "0_capacitor_smd:C_0402_1005Metric"
+		(property "Footprint" "0_capacitor_smd:C_0805_2012Metric"
 			(at 141.9352 74.93 0)
 			(effects
@@
 			)
 		)
-		(property "LCSC" "C307331"
+		(property "LCSC" "C45783"
 			(at 140.97 71.12 0)
 			(effects
@@
 		)
 		(instances
-			(project ""
+			(project "hoppen_fc"
 				(path "/abe950a1-9eef-4508-9fd4-31d3e723e029/c85454e5-a89e-41eb-a5ed-71b4fc4cf13a/497505dd-337e-4de8-b212-9653d17f2ba6"
-					(reference "C104")
+					(reference "C87")
 					(unit 1)
 				)
