File: hoppen_fc/storage.kicad_sch (KiCad schematic)
At the start: 11 parts, among them J19 MicroSD Card Holder, U6 W25Q128JVS

Commit message: finished adding lcsc numbers
Parts:
- C63: renamed from C50; LCSC (none) -> C15849
- C64: renamed from C37; LCSC (none) -> C307331
- C65: renamed from C36; LCSC (none) -> C307331
- C66: renamed from C51; LCSC (none) -> C15849
- R25: renamed from R11; value 10k -> 47k; LCSC (none) -> C25792
- R26: renamed from R10; LCSC (none) -> C25092
- R27: renamed from R8; LCSC (none) -> C25092
- R28: renamed from R9; value 10k -> 47k; LCSC (none) -> C25792
- R29: renamed from R12; value 10k -> 47k; LCSC (none) -> C25792
- renumbered J19 to J3, U6 to U11

Commit message: ready for routing?
Connections:
- net SD_CLK_T: now reaches J3.5 (CLK), R26.2
Changed lines of the file:
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@@
+		)
+	)
+	(label "SD_CLK_T"
+		(at 195.58 105.41 0)
+		(effects
+			(font
+				(size 0.635 0.635)
+			)
+			(justify left bottom)
 		)
 	)

Commit message: routing and adding rf module
Parts:
- renumbered R25 to R24, R26 to R25, R27 to R26, R28 to R27, R29 to R28
Changed lines of the file:
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@@
 		(dnp no)
 		(fields_autoplaced yes)
-		(property "Reference" "R29"
+		(property "Reference" "R28"
 			(at 255.27 123.1899 0)
 			(effects
@@
 			(project "hoppen_fc"
 				(path "/abe950a1-9eef-4508-9fd4-31d3e723e029/c85454e5-a89e-41eb-a5ed-71b4fc4cf13a/93bd097e-cae3-4aaa-9718-ae37366bd59a"
-					(reference "R29")
+					(reference "R28")
 					(unit 1)
 				)
@@
 		(dnp no)
 		(fields_autoplaced yes)
-		(property "Reference" "R28"
+		(property "Reference" "R27"
 			(at 73.66 119.3799 0)
 			(effects
@@
 			(project ""
 				(path "/abe950a1-9eef-4508-9fd4-31d3e723e029/c85454e5-a89e-41eb-a5ed-71b4fc4cf13a/93bd097e-cae3-4aaa-9718-ae37366bd59a"
-					(reference "R28")
+					(reference "R27")
 					(unit 1)
 				)
@@
 		(on_board yes)
 		(dnp no)
-		(property "Reference" "R27"
+		(property "Reference" "R26"
 			(at 60.96 107.95 90)
 			(effects
@@
 			(project ""
 				(path "/abe950a1-9eef-4508-9fd4-31d3e723e029/c85454e5-a89e-41eb-a5ed-71b4fc4cf13a/93bd097e-cae3-4aaa-9718-ae37366bd59a"
-					(reference "R27")
+					(reference "R26")
 					(unit 1)
 				)
@@
 		(dnp no)
 		(fields_autoplaced yes)
-		(property "Reference" "R25"
+		(property "Reference" "R24"
 			(at 171.45 78.7399 0)
 			(effects
@@
 			(project "hoppen_fc"
 				(path "/abe950a1-9eef-4508-9fd4-31d3e723e029/c85454e5-a89e-41eb-a5ed-71b4fc4cf13a/93bd097e-cae3-4aaa-9718-ae37366bd59a"
-					(reference "R25")
+					(reference "R24")
 					(unit 1)
 				)
@@
 		(on_board yes)
 		(dnp no)
-		(property "Reference" "R26"
+		(property "Reference" "R25"
 			(at 186.69 106.68 90)
 			(effects
@@
 			(project "hoppen_fc"
 				(path "/abe950a1-9eef-4508-9fd4-31d3e723e029/c85454e5-a89e-41eb-a5ed-71b4fc4cf13a/93bd097e-cae3-4aaa-9718-ae37366bd59a"
-					(reference "R26")
-					(unit 1)
-				)
+					(reference "R25")
+					(unit 1)
+				)

Commit message: comments
Other:
- note added: "ADD TVS DIODES"
Changed lines of the file:
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@@
+		)
+	)
+	(text "ADD TVS DIODES\n"
+		(exclude_from_sim no)
+		(at 173.482 48.768 0)
+		(effects
+			(font
+				(face "KiCad Font")
+				(size 2.54 2.54)
+				(thickness 0.508)
+				(bold yes)
+				(color 255 0 0 1)
+			)
 		)
 	)

Commit message: bump
Parts:
- removed C63, C66: 1u, 0_capacitor_smd:C_0603_1608Metric, symbol Device:C
- removed C64: 100n, 0_capacitor_smd:C_0402_1005Metric, symbol Device:C
- added C52: 10u, 0_capacitor_smd:C_0805_2012Metric, symbol Device:C
- added C54: 100n, 0_capacitor_smd:C_0402_1005Metric, symbol Device:C
- added R30, R31: 10k, 0_resistor_smd:R_0402_1005Metric, symbol Device:R
- added TP20, TP21, TP22, TP23, TP24, TP25, TP26, TP27, TP28, TP29, TP30, TP31, TP32, TP33, TP34: TestPoint, TestPoint:TestPoint_Pad_1.0x1.0mm, symbol Connector:TestPoint
- added U13: FM24C64B, Package_SO:SOIC-8_3.9x4.9mm_P1.27mm, symbol Memory_NVRAM:FM24C64B
- R26: renamed from R25; LCSC C25092 -> C2929994
- R27: renamed from R26; LCSC C25092 -> C2929994
- renumbered C65 to C53, R24 to R25, R27 to R28, R28 to R29, U11 to U12
Connections:
- net +3V3: now also C52.1, C54.1, R30.2, R31.2, U13.8 (VDD)
- net GND: now also C52.2, C54.2, U13.1 (A0), U13.2 (A1), U13.3 (A2), U13.4 (VSS), U13.7 (WP)
- net QSPI_CLK_T: now also TP21.1
- net QSPI_IO0: now also TP20.1
- net QSPI_IO1: now also TP23.1
- net QSPI_IO2: now also TP26.1
- net QSPI_IO3: now also TP29.1
- net QSPI_nCS: now also TP24.1
- net SD_CLK: now also TP28.1
- net SD_CLK_T: now also TP31.1
- net SD_CMD: now also TP25.1
- net SD_D0: now also TP27.1
- net SD_D1: now also TP30.1
- net SD_D2: now also TP33.1
- net SD_D3: now also TP22.1
- new net I2C_SCL: R31.1, TP32.1, U13.6 (SCL)
- new net I2C_SDA: R30.1, TP34.1, U13.5 (SDA)
Other:
- note added: "EEPROM"
- note added: "PROBING"
- note removed: "ADD TVS DIODES"
- moved on the sheet: C53, J3, R25, R26, R27, R28, R29, U12

Commit message: bump
Parts:
- removed TP28: TestPoint, TestPoint:TestPoint_Pad_1.0x1.0mm, symbol Connector:TestPoint
- renumbered TP20 to TP36, TP21 to TP37, TP22 to TP38, TP23 to TP39, TP24 to TP40, TP25 to TP41, TP26 to TP42, TP27 to TP43, TP31 to TP44, TP29 to TP45, TP30 to TP46, TP34 to TP47, TP32 to TP48, TP33 to TP49
Other:
- moved on the sheet: TP44, TP47
Changed lines of the file:
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@@
 	(wire
 		(pts
-			(xy 137.16 148.59) (xy 148.59 148.59)
+			(xy 137.16 143.51) (xy 148.59 143.51)
 		)
 		(stroke
@@
 	(wire
 		(pts
-			(xy 137.16 143.51) (xy 148.59 143.51)
-		)
-		(stroke
-			(width 0)
-			(type default)
-		)
-	)
-	(wire
-		(pts
 			(xy 48.26 80.01) (xy 74.93 80.01)
 		)
@@
 	(wire
 		(pts
-			(xy 137.16 153.67) (xy 148.59 153.67)
+			(xy 137.16 148.59) (xy 148.59 148.59)
 		)
 		(stroke
@@
 	)
 	(label "I2C_SDA"
-		(at 148.59 153.67 180)
+		(at 148.59 148.59 180)
 		(effects
 			(font
@@
 	)
 	(label "SD_CLK_T"
-		(at 148.59 148.59 180)
+		(at 148.59 143.51 180)
 		(effects
 			(font
@@
 		)
 	)
-	(label "SD_CLK"
-		(at 148.59 143.51 180)
-		(effects
-			(font
-				(size 1.27 1.27)
-			)
-			(justify right bottom)
-		)
-	)
 	(label "QSPI_IO0"
 		(at 113.03 133.35 180)
@@
 		(dnp no)
 		(fields_autoplaced yes)
-		(property "Reference" "TP21"
+		(property "Reference" "TP37"
 			(at 116.078 130.81 90)
 			(effects
@@
 			(project "hoppen_fc"
 				(path "/abe950a1-9eef-4508-9fd4-31d3e723e029/c85454e5-a89e-41eb-a5ed-71b4fc4cf13a/93bd097e-cae3-4aaa-9718-ae37366bd59a"
-					(reference "TP21")
+					(reference "TP37")
 					(unit 1)
 				)
@@
 		(dnp no)
 		(fields_autoplaced yes)
-		(property "Reference" "TP24"
+		(property "Reference" "TP40"
 			(at 116.078 135.89 90)
 			(effects
@@
 			(project "hoppen_fc"
 				(path "/abe950a1-9eef-4508-9fd4-31d3e723e029/c85454e5-a89e-41eb-a5ed-71b4fc4cf13a/93bd097e-cae3-4aaa-9718-ae37366bd59a"
-					(reference "TP24")
+					(reference "TP40")
 					(unit 1)
 				)
@@
 		(dnp no)
 		(fields_autoplaced yes)
-		(property "Reference" "TP29"
+		(property "Reference" "TP45"
 			(at 98.298 146.05 90)
 			(effects
@@
 			(project "hoppen_fc"
 				(path "/abe950a1-9eef-4508-9fd4-31d3e723e029/c85454e5-a89e-41eb-a5ed-71b4fc4cf13a/93bd097e-cae3-4aaa-9718-ae37366bd59a"
-					(reference "TP29")
+					(reference "TP45")
 					(unit 1)
 				)
@@
 		(dnp no)
 		(fields_autoplaced yes)
-		(property "Reference" "TP25"
+		(property "Reference" "TP41"
 			(at 133.858 135.89 90)
 			(effects
@@
 			(project "hoppen_fc"
 				(path "/abe950a1-9eef-4508-9fd4-31d3e723e029/c85454e5-a89e-41eb-a5ed-71b4fc4cf13a/93bd097e-cae3-4aaa-9718-ae37366bd59a"
-					(reference "TP25")
+					(reference "TP41")
 					(unit 1)
 				)
@@
 		(dnp no)
 		(fields_autoplaced yes)
-		(property "Reference" "TP27"
+		(property "Reference" "TP43"
 			(at 116.078 140.97 90)
 			(effects
@@
 			(project "hoppen_fc"
 				(path "/abe950a1-9eef-4508-9fd4-31d3e723e029/c85454e5-a89e-41eb-a5ed-71b4fc4cf13a/93bd097e-cae3-4aaa-9718-ae37366bd59a"
-					(reference "TP27")
+					(reference "TP43")
 					(unit 1)
 				)
@@
 		(dnp no)
 		(fields_autoplaced yes)
-		(property "Reference" "TP23"
+		(property "Reference" "TP39"
 			(at 98.298 135.89 90)
 			(effects
@@
 			(project "hoppen_fc"
 				(path "/abe950a1-9eef-4508-9fd4-31d3e723e029/c85454e5-a89e-41eb-a5ed-71b4fc4cf13a/93bd097e-cae3-4aaa-9718-ae37366bd59a"
-					(reference "TP23")
+					(reference "TP39")
 					(unit 1)
 				)
@@
 		(dnp no)
 		(fields_autoplaced yes)
-		(property "Reference" "TP30"
+		(property "Reference" "TP46"
 			(at 116.078 146.05 90)
 			(effects
@@
 			(project "hoppen_fc"
 				(path "/abe950a1-9eef-4508-9fd4-31d3e723e029/c85454e5-a89e-41eb-a5ed-71b4fc4cf13a/93bd097e-cae3-4aaa-9718-ae37366bd59a"
-					(reference "TP30")
+					(reference "TP46")
 					(unit 1)
 				)
@@
 	(symbol
 		(lib_id "Connector:TestPoint")
-		(at 137.16 143.51 90)
-		(unit 1)
-		(exclude_from_sim no)
-		(in_bom yes)
-		(on_board yes)
-		(dnp no)
-		(fields_autoplaced yes)
-		(property "Reference" "TP28"
-			(at 133.858 140.97 90)
-			(effects
-				(font
-					(size 1.27 1.27)
-				)
-			)
-		)
-		(property "Value" "TestPoint"
-			(at 135.1279 140.97 0)
-			(effects
-				(font
-					(size 1.27 1.27)
-				)
-				(justify left)
-				(hide yes)
-			)
-		)
-		(property "Footprint" "TestPoint:TestPoint_Pad_1.0x1.0mm"
-			(at 137.16 138.43 0)
-			(effects
-				(font
-					(size 1.27 1.27)
-				)
-				(hide yes)
-			)
-		)
-		(property "Datasheet" "~"
-			(at 137.16 138.43 0)
-			(effects
-				(font
-					(size 1.27 1.27)
-				)
-				(hide yes)
-			)
-		)
-		(property "Description" "test point"
-			(at 137.16 143.51 0)
-			(effects
-				(font
-					(size 1.27 1.27)
-				)
-				(hide yes)
-			)
-		)
-		(pin "1"
-		)
-		(instances
-			(project "hoppen_fc"
-				(path "/abe950a1-9eef-4508-9fd4-31d3e723e029/c85454e5-a89e-41eb-a5ed-71b4fc4cf13a/93bd097e-cae3-4aaa-9718-ae37366bd59a"
-					(reference "TP28")
-					(unit 1)
-				)
-			)
-		)
-	)
-	(symbol
-		(lib_id "Connector:TestPoint")
 		(at 101.6 153.67 90)
 		(unit 1)
@@
 		(dnp no)
 		(fields_autoplaced yes)
-		(property "Reference" "TP32"
+		(property "Reference" "TP48"
 			(at 98.298 151.13 90)
 			(effects
@@
 			(project "hoppen_fc"
 				(path "/abe950a1-9eef-4508-9fd4-31d3e723e029/c85454e5-a89e-41eb-a5ed-71b4fc4cf13a/93bd097e-cae3-4aaa-9718-ae37366bd59a"
-					(reference "TP32")
+					(reference "TP48")
 					(unit 1)
 				)
@@
 		(dnp no)
 		(fields_autoplaced yes)
-		(property "Reference" "TP22"
+		(property "Reference" "TP38"
 			(at 133.858 130.81 90)
 			(effects
@@
 			(project "hoppen_fc"
 				(path "/abe950a1-9eef-4508-9fd4-31d3e723e029/c85454e5-a89e-41eb-a5ed-71b4fc4cf13a/93bd097e-cae3-4aaa-9718-ae37366bd59a"
-					(reference "TP22")
+					(reference "TP38")
 					(unit 1)
 				)
@@
 		(dnp no)
 		(fields_autoplaced yes)
-		(property "Reference" "TP20"
+		(property "Reference" "TP36"
 			(at 98.298 130.81 90)
 			(effects
@@
 			(project "hoppen_fc"
 				(path "/abe950a1-9eef-4508-9fd4-31d3e723e029/c85454e5-a89e-41eb-a5ed-71b4fc4cf13a/93bd097e-cae3-4aaa-9718-ae37366bd59a"
-					(reference "TP20")
+					(reference "TP36")
 					(unit 1)
 				)
@@
 		(dnp no)
 		(fields_autoplaced yes)
-		(property "Reference" "TP33"
+		(property "Reference" "TP49"
 			(at 116.078 151.13 90)
 			(effects
@@
 			(project "hoppen_fc"
 				(path "/abe950a1-9eef-4508-9fd4-31d3e723e029/c85454e5-a89e-41eb-a5ed-71b4fc4cf13a/93bd097e-cae3-4aaa-9718-ae37366bd59a"
-					(reference "TP33")
+					(reference "TP49")
 					(unit 1)
 				)
@@
 	(symbol
 		(lib_id "Connector:TestPoint")
-		(at 137.16 148.59 90)
+		(at 137.16 143.51 90)
 		(unit 1)
 		(exclude_from_sim no)
@@
 		(dnp no)
 		(fields_autoplaced yes)
-		(property "Reference" "TP31"
-			(at 133.858 146.05 90)
+		(property "Reference" "TP44"
+			(at 133.858 140.97 90)
 			(effects
 				(font
@@
 		)
 		(property "Value" "TestPoint"
-			(at 135.1279 146.05 0)
+			(at 135.1279 140.97 0)
 			(effects
 				(font
@@
 		)
 		(property "Footprint" "TestPoint:TestPoint_Pad_1.0x1.0mm"
-			(at 137.16 143.51 0)
+			(at 137.16 138.43 0)
 			(effects
 				(font
@@
 		)
 		(property "Datasheet" "~"
-			(at 137.16 143.51 0)
+			(at 137.16 138.43 0)
 			(effects
 				(font
@@
 		)
 		(property "Description" "test point"
-			(at 137.16 148.59 0)
+			(at 137.16 143.51 0)
 			(effects
 				(font
@@
 			(project "hoppen_fc"
 				(path "/abe950a1-9eef-4508-9fd4-31d3e723e029/c85454e5-a89e-41eb-a5ed-71b4fc4cf13a/93bd097e-cae3-4aaa-9718-ae37366bd59a"
-					(reference "TP31")
+					(reference "TP44")
 					(unit 1)
 				)
@@
 		(dnp no)
 		(fields_autoplaced yes)
-		(property "Reference" "TP26"
+		(property "Reference" "TP42"
 			(at 98.298 140.97 90)
 			(effects
@@
 			(project "hoppen_fc"
 				(path "/abe950a1-9eef-4508-9fd4-31d3e723e029/c85454e5-a89e-41eb-a5ed-71b4fc4cf13a/93bd097e-cae3-4aaa-9718-ae37366bd59a"
-					(reference "TP26")
+					(reference "TP42")
 					(unit 1)
 				)
@@
 	(symbol
 		(lib_id "Connector:TestPoint")
-		(at 137.16 153.67 90)
+		(at 137.16 148.59 90)
 		(unit 1)
 		(exclude_from_sim no)
@@
 		(dnp no)
 		(fields_autoplaced yes)
-		(property "Reference" "TP34"
-			(at 133.858 151.13 90)
+		(property "Reference" "TP47"
+			(at 133.858 146.05 90)
 			(effects
 				(font
@@
 		)
 		(property "Value" "TestPoint"
-			(at 135.1279 151.13 0)
+			(at 135.1279 146.05 0)
 			(effects
 				(font
@@
 		)
 		(property "Footprint" "TestPoint:TestPoint_Pad_1.0x1.0mm"
-			(at 137.16 148.59 0)
+			(at 137.16 143.51 0)
 			(effects
 				(font
@@
 		)
 		(property "Datasheet" "~"
-			(at 137.16 148.59 0)
+			(at 137.16 143.51 0)
 			(effects
 				(font
@@
 		)
 		(property "Description" "test point"
-			(at 137.16 153.67 0)
+			(at 137.16 148.59 0)
 			(effects
 				(font
@@
 			(project "hoppen_fc"
 				(path "/abe950a1-9eef-4508-9fd4-31d3e723e029/c85454e5-a89e-41eb-a5ed-71b4fc4cf13a/93bd097e-cae3-4aaa-9718-ae37366bd59a"
-					(reference "TP34")
+					(reference "TP47")
 					(unit 1)
 				)
