File: hoppen_fc/interfaces_comms.kicad_sch (KiCad schematic)
At the start: 26 parts, among them J12 GH1.25-4P, J13 GH1.25-4P, J14 GH1.25-2P, J15 GH1.25-2P, J16 GH1.25-4P, J17 GH1.25-5P, J18 GH1.25-2P, U16 LPW5209AB5F, U17 74AHCT1G125

Commit message: bump
Parts:
- removed C101, C102, C103, C98, C99: 100n, 0_capacitor_smd:C_0402_1005Metric, symbol Device:C
- removed J15: GH1.25-2P, 0_connectors:SM02B-GHS-TB-LF-SN, symbol 0_connectors:Conn_01x02_Mounting
- removed R52: 47k, 0_resistor_smd:R_0402_1005Metric, symbol Device:R
- removed U16: LPW5209AB5F, 0_power:SOT-23-5_L3.0-W1.7-P0.95-LS2.8-BL, symbol 0_power:LPW5209AB5F
- added C83, C84, C86: 22u, 0_capacitor_smd:C_0805_2012Metric, symbol Device:C
- added U22: PD4E1U, 0_transistors:SOT-363_SC-70-6, symbol 0_diodes:PD4E1U
- D13: footprint PCM_JLCPCB:D_SOD-123FL -> Diode_SMD:D_SOD-123
- J12, J13: value GH1.25-4P -> BM04B-GHS1.25; footprint 0_connectors:SM04B-GHS-TB-LF-SN -> 0_connectors:BM04B-GHS1.25; LCSC C189895 -> C161692
- J14: value GH1.25-2P -> BM02B-GHS1.25; footprint 0_connectors:SM02B-GHS-TB-LF-SN -> 0_connectors:BM02B-GHS1.25; LCSC C189893 -> C225118
- J15: renamed from J17; value GH1.25-5P -> BM05B-GHS1.25; footprint 0_connectors:SM05B-GHS-TB-LF-SN -> 0_connectors:BM05B-GHS1.25; LCSC C189896 -> C225121
- J16: renamed from J18; value GH1.25-2P -> BM02B-GHS1.25; footprint 0_connectors:SM02B-GHS-TB-LF-SN -> 0_connectors:BM02B-GHS1.25; LCSC C189893 -> C225118
- J17: renamed from J16; value GH1.25-4P -> BM04B-GHS1.25; footprint 0_connectors:SM04B-GHS-TB-LF-SN -> 0_connectors:BM04B-GHS1.25; LCSC C189895 -> C161692
- R57: renamed from R53; LCSC C25092 -> C2929994
- R58: renamed from R54; LCSC C25092 -> C2929994
- renumbered C100 to C85, R48 to R53, R49 to R54, R50 to R55, R51 to R56, U17 to U21
Connections:
- net +5V_EXT is gone; now on net +5V: J12.1 (Pin_1), J13.1 (Pin_1)
- net +5V: now also C83.1, C84.1
- net EXT_UART_PWR: now also C86.1
- net GND: now also C83.2, C84.2, C86.2, U22.2 (GND)
- net SWCLK: now also U22.6 (D1-)
- net SWDIO: now also U22.1 (D1+)
- no-connect marks 0 -> 2
Other:
- note added: "ESD PROTECTION"
- note removed: "5V OUTPUT @ 1000 mA"
- moved on the sheet: J15, J16, U21

Commit message: bump
Parts:
- removed D13: SMF18A, Diode_SMD:D_SOD-123, symbol PCM_JLCPCB-Diodes:TVS-Uni,SMF18A
- added D13: SMF28CA, PCM_JLCPCB:D_SOD-123FL, symbol PCM_JLCPCB-Diodes:TVS-Bi,SMF28CA
Connections:
- net EXT_BAT: now also D13.2
- net GND: now also D13.1
Changed lines of the file:
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@@
 	)
 	(junction
-		(at 247.65 118.11)
-		(diameter 0)
-		(color 0 0 0 0)
-	)
-	(junction
 		(at 260.35 163.83)
 		(diameter 0)
@@
 	)
 	(junction
+		(at 247.65 118.11)
+		(diameter 0)
+		(color 0 0 0 0)
+	)
+	(junction
 		(at 123.19 180.34)
 		(diameter 0)
@@
 	(wire
 		(pts
+			(xy 247.65 118.11) (xy 261.62 118.11)
+		)
+		(stroke
+			(width 0)
+			(type default)
+		)
+	)
+	(wire
+		(pts
 			(xy 120.65 58.42) (xy 124.46 58.42)
 		)
@@
 	(wire
 		(pts
-			(xy 260.35 172.72) (xy 260.35 171.45)
-		)
-		(stroke
-			(width 0)
-			(type default)
-		)
-	)
-	(wire
-		(pts
-			(xy 247.65 118.11) (xy 261.62 118.11)
+			(xy 241.3 118.11) (xy 247.65 118.11)
 		)
 		(stroke
@@
 	(wire
 		(pts
+			(xy 260.35 171.45) (xy 260.35 172.72)
+		)
+		(stroke
+			(width 0)
+			(type default)
+		)
+	)
+	(wire
+		(pts
 			(xy 232.41 58.42) (xy 236.22 58.42)
 		)
@@
 	(wire
 		(pts
-			(xy 241.3 118.11) (xy 247.65 118.11)
-		)
-		(stroke
-			(width 0)
-			(type default)
-		)
-	)
-	(wire
-		(pts
 			(xy 119.38 162.56) (xy 123.19 162.56)
 		)
@@
 	)
 	(symbol
+		(lib_id "PCM_JLCPCB-Diodes:TVS-Bi,SMF28CA")
+		(at 247.65 121.92 0)
+		(unit 1)
+		(exclude_from_sim no)
+		(in_bom yes)
+		(on_board yes)
+		(dnp no)
+		(fields_autoplaced yes)
+		(property "Reference" "D13"
+			(at 251.46 120.6499 0)
+			(effects
+				(font
+					(size 1.27 1.27)
+				)
+				(justify left)
+			)
+		)
+		(property "Value" "SMF28CA"
+			(at 251.46 123.19 0)
+			(effects
+				(font
+					(size 0.8 0.8)
+				)
+				(justify left)
+			)
+		)
+		(property "Footprint" "PCM_JLCPCB:D_SOD-123FL"
+			(at 245.872 121.92 90)
+			(effects
+				(font
+					(size 1.27 1.27)
+				)
+				(hide yes)
+			)
+		)
+		(property "Datasheet" "https://wmsc.lcsc.com/wmsc/upload/file/pdf/v2/lcsc/2312221742_hongjiacheng-SMF28CA_C19077517.pdf"
+			(at 247.65 121.92 0)
+			(effects
+				(font
+					(size 1.27 1.27)
+				)
+				(hide yes)
+			)
+		)
+		(property "Description" "4.4A 45.4V 200W 34.4V Bidirectional 28V SOD-123FL ESD and Surge Protection (TVS/ESD) ROHS"
+			(at 247.65 121.92 0)
+			(effects
+				(font
+					(size 1.27 1.27)
+				)
+				(hide yes)
+			)
+		)
+		(property "LCSC" "C19077517"
+			(at 247.65 121.92 0)
+			(effects
+				(font
+					(size 1.27 1.27)
+				)
+				(hide yes)
+			)
+		)
+		(property "Stock" "117291"
+			(at 247.65 121.92 0)
+			(effects
+				(font
+					(size 1.27 1.27)
+				)
+				(hide yes)
+			)
+		)
+		(property "Price" "0.028USD"
+			(at 247.65 121.92 0)
+			(effects
+				(font
+					(size 1.27 1.27)
+				)
+				(hide yes)
+			)
+		)
+		(property "Process" "SMT"
+			(at 247.65 121.92 0)
+			(effects
+				(font
+					(size 1.27 1.27)
+				)
+				(hide yes)
+			)
+		)
+		(property "Minimum Qty" "15"
+			(at 247.65 121.92 0)
+			(effects
+				(font
+					(size 1.27 1.27)
+				)
+				(hide yes)
+			)
+		)
+		(property "Attrition Qty" "4"
+			(at 247.65 121.92 0)
+			(effects
+				(font
+					(size 1.27 1.27)
+				)
+				(hide yes)
+			)
+		)
+		(property "Class" "Preferred Component"
+			(at 247.65 121.92 0)
+			(effects
+				(font
+					(size 1.27 1.27)
+				)
+				(hide yes)
+			)
+		)
+		(property "Category" "TVS/Fuse/Board Level Protection,Electrostatic And Surge Protection (TVS/ESD)"
+			(at 247.65 121.92 0)
+			(effects
+				(font
+					(size 1.27 1.27)
+				)
+				(hide yes)
+			)
+		)
+		(property "Manufacturer" "hongjiacheng"
+			(at 247.65 121.92 0)
+			(effects
+				(font
+					(size 1.27 1.27)
+				)
+				(hide yes)
+			)
+		)
+		(property "Part" "SMF28CA"
+			(at 247.65 121.92 0)
+			(effects
+				(font
+					(size 1.27 1.27)
+				)
+				(hide yes)
+			)
+		)
+		(pin "1"
+		)
+		(pin "2"
+		)
+		(instances
+			(project "hoppen_fc"
+				(path "/abe950a1-9eef-4508-9fd4-31d3e723e029/c85454e5-a89e-41eb-a5ed-71b4fc4cf13a/4ffe1006-14f1-46cf-875e-eefbb8c17932"
+					(reference "D13")
+					(unit 1)
+				)
+			)
+		)
+	)
+	(symbol
 		(lib_id "power:+3.3V")
 		(at 243.84 55.88 0)
@@
 					(unit 1)
 				)
-			)
-		)
-	)
-	(symbol
-		(lib_id "PCM_JLCPCB-Diodes:TVS-Uni,SMF18A")
-		(at 247.65 121.92 180)
-		(unit 1)
-		(exclude_from_sim no)
-		(in_bom yes)
-		(on_board yes)
-		(dnp no)
-		(fields_autoplaced yes)
-		(property "Reference" "D13"
-			(at 251.46 120.3324 0)
-			(effects
-				(font
-					(size 1.27 1.27)
-				)
-				(justify right)
-			)
-		)
-		(property "Value" "SMF18A"
-			(at 251.46 122.8725 0)
-			(effects
-				(font
-					(size 0.8 0.8)
-				)
-				(justify right)
-			)
-		)
-		(property "Footprint" "Diode_SMD:D_SOD-123"
-			(at 249.428 121.92 90)
-			(effects
-				(font
-					(size 1.27 1.27)
-				)
-				(hide yes)
-			)
-		)
-		(property "Datasheet" "https://wmsc.lcsc.com/wmsc/upload/file/pdf/v2/lcsc/2312280940_hongjiacheng-SMF18A_C19077512.pdf"
-			(at 247.65 121.92 0)
-			(effects
-				(font
-					(size 1.27 1.27)
-				)
-				(hide yes)
-			)
-		)
-		(property "Description" "6.8A 29.2V 200W 22.1V Unidirectional 18V SOD-123FL ESD and Surge Protection (TVS/ESD) ROHS"
-			(at 247.65 121.92 0)
-			(effects
-				(font
-					(size 1.27 1.27)
-				)
-				(hide yes)
-			)
-		)
-		(property "LCSC" "C19077512"
-			(at 247.65 121.92 0)
-			(effects
-				(font
-					(size 1.27 1.27)
-				)
-				(hide yes)
-			)
-		)
-		(property "Stock" "43774"
-			(at 247.65 121.92 0)
-			(effects
-				(font
-					(size 1.27 1.27)
-				)
-				(hide yes)
-			)
-		)
-		(property "Price" "0.027USD"
-			(at 247.65 121.92 0)
-			(effects
-				(font
-					(size 1.27 1.27)
-				)
-				(hide yes)
-			)
-		)
-		(property "Process" "SMT"
-			(at 247.65 121.92 0)
-			(effects
-				(font
-					(size 1.27 1.27)
-				)
-				(hide yes)
-			)
-		)
-		(property "Minimum Qty" "15"
-			(at 247.65 121.92 0)
-			(effects
-				(font
-					(size 1.27 1.27)
-				)
-				(hide yes)
-			)
-		)
-		(property "Attrition Qty" "4"
-			(at 247.65 121.92 0)
-			(effects
-				(font
-					(size 1.27 1.27)
-				)
-				(hide yes)
-			)
-		)
-		(property "Class" "Preferred Component"
-			(at 247.65 121.92 0)
-			(effects
-				(font
-					(size 1.27 1.27)
-				)
-				(hide yes)
-			)
-		)
-		(property "Category" "TVS/Fuse/Board Level Protection,Electrostatic And Surge Protection (TVS/ESD)"
-			(at 247.65 121.92 0)
-			(effects
-				(font
-					(size 1.27 1.27)
-				)
-				(hide yes)
-			)
-		)
-		(property "Manufacturer" "hongjiacheng"
-			(at 247.65 121.92 0)
-			(effects
-				(font
-					(size 1.27 1.27)
-				)
-				(hide yes)
-			)
-		)
-		(property "Part" "SMF18A"
-			(at 247.65 121.92 0)
-			(effects
-				(font
-					(size 1.27 1.27)
-				)
-				(hide yes)
-			)
-		)
-		(pin "1"
-		)
-		(pin "2"
-		)
-		(instances
-			(project "hoppen_fc"
-				(path "/abe950a1-9eef-4508-9fd4-31d3e723e029/c85454e5-a89e-41eb-a5ed-71b4fc4cf13a/4ffe1006-14f1-46cf-875e-eefbb8c17932"
-					(reference "D13")
-					(unit 1)
-				)

Commit message: production v1
Other:
- note added: "MAX 6S"
- note removed: "MAX 4S"
Changed lines of the file:
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@@
 		)
 	)
-	(text "MAX 4S"
+	(text "MAX 6S"
 		(exclude_from_sim no)
 		(at 223.266 138.176 0)
