File: hoppen_fc/mcu_io.kicad_sch (KiCad schematic)
At the start: 17 parts, among them SW1 SW_Push, SW2 SW_Push, SW3 SW_Push, U1 STM32H743ZITx, U2 PD4E1U, Y1 25 MHz Crystal, Y2 32.768 kHz

Commit message: production v1
Parts:
- R1: value 1k -> 10k; LCSC C106235 -> C25744
Connections:
- net ESC_TX_1: now also U1.58 (PE7); no longer U1.59 (PE8)
Changed lines of the file:
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@@
 	)
 	(no_connect
-		(at 191.77 83.82)
-	)
-	(no_connect
 		(at 116.84 86.36)
 	)
@@
 	)
 	(no_connect
+		(at 191.77 86.36)
+	)
+	(no_connect
 		(at 191.77 142.24)
 	)
@@
 	)
 	(label "ESC_TX_1"
-		(at 191.77 86.36 180)
+		(at 191.77 83.82 180)
 		(effects
 			(font
@@
 					(unit 2)
 				)
-				(path "/abe950a1-9eef-4508-9fd4-31d3e723e029/c85454e5-a89e-41eb-a5ed-71b4fc4cf13a/e8dec57f-fe0f-4242-be3c-094f4ce75313"
-					(reference "U1")
-					(unit 2)
-				)
 			)
 		)
@@
 			)
 		)
-		(property "Value" "1k"
+		(property "Value" "10k"
 			(at 163.83 270.5099 0)
 			(effects
@@
 			)
 		)
-		(property "LCSC" "C106235"
+		(property "LCSC" "C25744"
 			(at 161.29 269.24 0)
 			(effects
@@
 					(reference "U1")
 					(unit 3)
-				)
-				(path "/abe950a1-9eef-4508-9fd4-31d3e723e029/c85454e5-a89e-41eb-a5ed-71b4fc4cf13a/e8dec57f-fe0f-4242-be3c-094f4ce75313"
-					(reference "U1")
-					(unit 3)
